Commit message: kr6: fixup R900 sixx kinematic structure. Fix #51.

File: kuka_kr6_support/urdf/kr6r900sixx_macro.xacro (robot description, xacro)
@@ -118,5 +118,5 @@
     </joint>
     <joint name="${prefix}joint_a3" type="revolute">
-      <origin xyz="0 0 0.455" rpy="0 0 0"/>
+      <origin xyz="0.455 0 0" rpy="0 0 0"/>
       <parent link="${prefix}link_2"/>
       <child link="${prefix}link_3"/>
