Commit message: match KR6 R1820 filenames to other models

File: kuka_kr6_support/urdf/kr6_r1820_macro.xacro (robot description, xacro)
@@ -8,5 +8,5 @@
         <origin xyz="0 0 0" rpy="0 0 0" />
         <geometry>
-          <mesh filename="package://kuka_kr6_support/meshes/kuka_kr6_r1820/visual/base_link.stl" />
+          <mesh filename="package://kuka_kr6_support/meshes/kr6r1820/visual/base_link.stl" />
         </geometry>
         <xacro:material_kuka_pedestal />
@@ -15,5 +15,5 @@
         <origin xyz="0 0 0" rpy="0 0 0" />
         <geometry>
-          <mesh filename="package://kuka_kr6_support/meshes/kuka_kr6_r1820/collision/base_link.stl" />
+          <mesh filename="package://kuka_kr6_support/meshes/kr6r1820/collision/base_link.stl" />
         </geometry>
       </collision>
@@ -23,5 +23,5 @@
         <origin xyz="0 0 0" rpy="0 0 0" />
         <geometry>
-          <mesh filename="package://kuka_kr6_support/meshes/kuka_kr6_r1820/visual/link_1.stl" />
+          <mesh filename="package://kuka_kr6_support/meshes/kr6r1820/visual/link_1.stl" />
         </geometry>
         <xacro:material_kuka_orange />
@@ -30,5 +30,5 @@
         <origin xyz="0 0 0" rpy="0 0 0" />
         <geometry>
-          <mesh filename="package://kuka_kr6_support/meshes/kuka_kr6_r1820/collision/link_1.stl" />
+          <mesh filename="package://kuka_kr6_support/meshes/kr6r1820/collision/link_1.stl" />
         </geometry>
       </collision>
@@ -38,5 +38,5 @@
         <origin xyz="0 0 0" rpy="0 0 0" />
         <geometry>
-          <mesh filename="package://kuka_kr6_support/meshes/kuka_kr6_r1820/visual/link_2.stl" />
+          <mesh filename="package://kuka_kr6_support/meshes/kr6r1820/visual/link_2.stl" />
         </geometry>
         <xacro:material_kuka_orange />
@@ -45,5 +45,5 @@
         <origin xyz="0 0 0" rpy="0 0 0" />
         <geometry>
-          <mesh filename="package://kuka_kr6_support/meshes/kuka_kr6_r1820/collision/link_2.stl" />
+          <mesh filename="package://kuka_kr6_support/meshes/kr6r1820/collision/link_2.stl" />
         </geometry>
       </collision>
@@ -53,5 +53,5 @@
         <origin xyz="0 0 0" rpy="0 0 0" />
         <geometry>
-          <mesh filename="package://kuka_kr6_support/meshes/kuka_kr6_r1820/visual/link_3.stl" />
+          <mesh filename="package://kuka_kr6_support/meshes/kr6r1820/visual/link_3.stl" />
         </geometry>
         <xacro:material_kuka_orange />
@@ -60,5 +60,5 @@
         <origin xyz="0 0 0" rpy="0 0 0" />
         <geometry>
-          <mesh filename="package://kuka_kr6_support/meshes/kuka_kr6_r1820/collision/link_3.stl" />
+          <mesh filename="package://kuka_kr6_support/meshes/kr6r1820/collision/link_3.stl" />
         </geometry>
       </collision>
@@ -68,5 +68,5 @@
         <origin xyz="0 0 0" rpy="0 0 0" />
         <geometry>
-          <mesh filename="package://kuka_kr6_support/meshes/kuka_kr6_r1820/visual/link_4.stl" />
+          <mesh filename="package://kuka_kr6_support/meshes/kr6r1820/visual/link_4.stl" />
         </geometry>
         <xacro:material_kuka_orange />
@@ -75,5 +75,5 @@
         <origin xyz="0 0 0" rpy="0 0 0" />
         <geometry>
-          <mesh filename="package://kuka_kr6_support/meshes/kuka_kr6_r1820/collision/link_4.stl" />
+          <mesh filename="package://kuka_kr6_support/meshes/kr6r1820/collision/link_4.stl" />
         </geometry>
       </collision>
@@ -83,5 +83,5 @@
         <origin xyz="0 0 0" rpy="0 0 0" />
         <geometry>
-          <mesh filename="package://kuka_kr6_support/meshes/kuka_kr6_r1820/visual/link_5.stl" />
+          <mesh filename="package://kuka_kr6_support/meshes/kr6r1820/visual/link_5.stl" />
         </geometry>
         <xacro:material_kuka_orange />
@@ -90,5 +90,5 @@
         <origin xyz="0 0 0" rpy="0 0 0" />
         <geometry>
-          <mesh filename="package://kuka_kr6_support/meshes/kuka_kr6_r1820/collision/link_5.stl" />
+          <mesh filename="package://kuka_kr6_support/meshes/kr6r1820/collision/link_5.stl" />
         </geometry>
       </collision>
@@ -98,5 +98,5 @@
         <origin xyz="0 0 0" rpy="0 0 0" />
         <geometry>
-          <mesh filename="package://kuka_kr6_support/meshes/kuka_kr6_r1820/visual/link_6.stl" />
+          <mesh filename="package://kuka_kr6_support/meshes/kr6r1820/visual/link_6.stl" />
         </geometry>
         <xacro:material_kuka_pedestal />
@@ -105,5 +105,5 @@
         <origin xyz="0 0 0" rpy="0 0 0" />
         <geometry>
-          <mesh filename="package://kuka_kr6_support/meshes/kuka_kr6_r1820/collision/link_6.stl" />
+          <mesh filename="package://kuka_kr6_support/meshes/kr6r1820/collision/link_6.stl" />
         </geometry>
       </collision>
