Commit message: Changed link names within macro.xacro to follow lower case and under score conventions. Changed link 1 and 6 collision stl's to have correct origin.

File: kuka_kr210_support/urdf/kr210l150.urdf (robot description, URDF)
Before this commit: robot kuka_kr210, 8 links, 7 joints
Links:
- removed link Link1
- removed link Link2
- removed link Link3
- removed link Link4
- removed link Link5
- removed link Link6
- added link link_1, mass 1385.5; collision mesh filename=package://kuka_kr210_support/meshes/kr210l150/collision/lin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; visual mesh filename=package://kuka_kr210_support/meshes/kr210l150/visual/link_1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
- added link link_2, mass 958.62; collision mesh filename=package://kuka_kr210_support/meshes/kr210l150/collision/lin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; visual mesh filename=package://kuka_kr210_support/meshes/kr210l150/visual/link_2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
- added link link_3, mass 710.03; collision mesh filename=package://kuka_kr210_support/meshes/kr210l150/collision/lin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; visual mesh filename=package://kuka_kr210_support/meshes/kr210l150/visual/link_3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
- added link link_4, mass 173.73; collision mesh filename=package://kuka_kr210_support/meshes/kr210l150/collision/lin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; visual mesh filename=package://kuka_kr210_support/meshes/kr210l150/visual/link_4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
- added link link_5, mass 72.17; collision mesh filename=package://kuka_kr210_support/meshes/kr210l150/collision/lin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; visual mesh filename=package://kuka_kr210_support/meshes/kr210l150/visual/link_5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
- added link link_6, mass 6.3154; collision mesh filename=package://kuka_kr210_support/meshes/kr210l150/collision/lin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; visual mesh filename=package://kuka_kr210_support/meshes/kr210l150/visual/link_6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
- link base_link: geometry collision mesh filename=package://kuka_kr210_support/meshes/kr210l150/collision/bas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; visual mesh filename=package://kuka_kr210_support/meshes/kr210l150/visual/base_l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
Joints:
- removed joint J1
- removed joint J2
- removed joint J3
- removed joint J4
- removed joint J5
- removed joint J6
- added joint joint_1: type revolute, parent base_link, child link_1, origin xyz=-0.00262 0.00097586 0.33099 rpy=0 0 0, axis 0 0 1, limit lower=-3.228859205 upper=3.228859205 effort=0 velocity=2.146755039
- added joint joint_2: type revolute, parent link_1, child link_2, origin xyz=0.35277 -0.037476 0.4192 rpy=0 0 0, axis 0 1 0, limit lower=-0.785398185 upper=1.483529905 effort=0 velocity=2.007128695
- added joint joint_3: type revolute, parent link_2, child link_3, origin xyz=-9.8483E-05 -0.1475 1.2499 rpy=0 0 0, axis 0 1 0, limit lower=-3.66519153 upper=1.134464045 effort=0 velocity=1.954768816
- added joint joint_4: type revolute, parent link_3, child link_4, origin xyz=0.95795 0.184 -0.055059 rpy=0 0 0, axis 1 0 0, limit lower=-6.10865255 upper=6.10865255 effort=0 velocity=3.124139447
- added joint joint_5: type revolute, parent link_4, child link_5, origin xyz=0.542 0 0 rpy=0 0 0, axis 0 1 0, limit lower=-2.181661625 upper=2.181661625 effort=0 velocity=3.001966396
- added joint joint_6: type revolute, parent link_5, child link_6, origin xyz=0.1925 0 0 rpy=0 0 0, axis 1 0 0, limit lower=-6.10865255 upper=6.10865255 effort=0 velocity=3.822271167
- joint link_6-tool0: parent Link6 -> link_6

File: kuka_kr210_support/urdf/kr210l150.xacro (robot description, xacro)
@@ -2,5 +2,5 @@
 <!--Generates a urdf from the macro in kr210_macro.xacro -->
 <robot name="kuka_kr210" xmlns:xacro="http://ros.org/wiki/xacro">
-	<xacro:include filename="$(find kuka_kr210_support)/urdf/kr210_macro.xacro"/>
-	<xacro:kuka_kr210 prefix=""/>
+	<xacro:include filename="$(find kuka_kr210_support)/urdf/kr210l150_macro.xacro"/>
+	<xacro:kuka_kr210l150 prefix=""/>
 </robot>

File: kuka_kr210_support/urdf/kr210l150_macro.xacro (robot description, xacro)
@@ -2,5 +2,5 @@
 	<property name="pi" value="3.141592654" />
 	<property name="deg" value="0.017453293" /> <!--degrees to radians-->
-	<xacro:macro name="kuka_kr210" params="prefix">
+	<xacro:macro name="kuka_kr210l150" params="prefix">
   <link
     name="${prefix}base_link">
@@ -25,19 +25,19 @@
       <geometry>
         <mesh
-          filename="package://kuka_kr210_support/meshes/visual/base_link.dae" />
-      </geometry>
-      <material
-        name="">
-        <color
-          rgba="0.75294 0.75294 0.75294 1" />
-      </material>
-    </visual>
-    <collision>
-      <origin
-        xyz="0 0 0"
-        rpy="${-pi/2} 0 0" />
-      <geometry>
-        <mesh
-          filename="package://kuka_kr210_support/meshes/collision/base_link.stl" />
+          filename="package://kuka_kr210_support/meshes/kr210l150/visual/base_link.dae" />
+      </geometry>
+      <material
+        name="">
+        <color
+          rgba="0.75294 0.75294 0.75294 1" />
+      </material>
+    </visual>
+    <collision>
+      <origin
+        xyz="0 0 0"
+        rpy="${-pi/2} 0 0" />
+      <geometry>
+        <mesh
+          filename="package://kuka_kr210_support/meshes/kr210l150/collision/base_link.stl" />
       </geometry>
     </collision>
@@ -65,24 +65,24 @@
       <geometry>
         <mesh
-          filename="package://kuka_kr210_support/meshes/visual/Link1.dae" />
-      </geometry>
-      <material
-        name="">
-        <color
-          rgba="0.75294 0.75294 0.75294 1" />
-      </material>
-    </visual>
-    <collision>
-      <origin
-        xyz="0 0 0"
-        rpy="0 0 0" />
-      <geometry>
-        <mesh
-          filename="package://kuka_kr210_support/meshes/collision/Link1.stl" />
-      </geometry>
-    </collision>
-  </link>
-  <joint
-    name="${prefix}J1"
+          filename="package://kuka_kr210_support/meshes/kr210l150/visual/link_1.dae" />
+      </geometry>
+      <material
+        name="">
+        <color
+          rgba="0.75294 0.75294 0.75294 1" />
+      </material>
+    </visual>
+    <collision>
+      <origin
+        xyz="0 0 0"
+        rpy="0 0 0" />
+      <geometry>
+        <mesh
+          filename="package://kuka_kr210_support/meshes/kr210l150/collision/link_1.stl" />
+      </geometry>
+    </collision>
+  </link>
+  <joint
+    name="${prefix}joint_1"
     type="revolute">
     <origin
@@ -98,5 +98,5 @@
   </joint>
   <link
-    name="${prefix}Link2">
+    name="${prefix}link_2">
     <inertial>
       <origin
@@ -119,24 +119,24 @@
       <geometry>
         <mesh
-          filename="package://kuka_kr210_support/meshes/visual/Link2.dae" />
-      </geometry>
-      <material
-        name="">
-        <color
-          rgba="0.75294 0.75294 0.75294 1" />
-      </material>
-    </visual>
-    <collision>
-      <origin
-        xyz="0 0 0"
-        rpy="0 0 0" />
-      <geometry>
-        <mesh
-          filename="package://kuka_kr210_support/meshes/collision/Link2.stl" />
-      </geometry>
-    </collision>
-  </link>
-  <joint
-    name="${prefix}J2"
+          filename="package://kuka_kr210_support/meshes/kr210l150/visual/link_2.dae" />
+      </geometry>
+      <material
+        name="">
+        <color
+          rgba="0.75294 0.75294 0.75294 1" />
+      </material>
+    </visual>
+    <collision>
+      <origin
+        xyz="0 0 0"
+        rpy="0 0 0" />
+      <geometry>
+        <mesh
+          filename="package://kuka_kr210_support/meshes/kr210l150/collision/link_2.stl" />
+      </geometry>
+    </collision>
+  </link>
+  <joint
+    name="${prefix}joint_2"
     type="revolute">
     <origin
@@ -146,5 +146,5 @@
       link="${prefix}Link1" />
     <child
-      link="${prefix}Link2" />
+      link="${prefix}link_2" />
     <axis
       xyz="0 1 0" />
@@ -152,5 +152,5 @@
   </joint>
   <link
-    name="${prefix}Link3">
+    name="${prefix}link_3">
     <inertial>
       <origin
@@ -173,24 +173,24 @@
       <geometry>
         <mesh
-          filename="package://kuka_kr210_support/meshes/visual/Link3.dae" />
-      </geometry>
-      <material
-        name="">
-        <color
-          rgba="0.75294 0.75294 0.75294 1" />
-      </material>
-    </visual>
-    <collision>
-      <origin
-        xyz="0 0 0"
-        rpy="0 0 0" />
-      <geometry>
-        <mesh
-          filename="package://kuka_kr210_support/meshes/collision/Link3.stl" />
-      </geometry>
-    </collision>
-  </link>
-  <joint
-    name="${prefix}J3"
+          filename="package://kuka_kr210_support/meshes/kr210l150/visual/link_3.dae" />
+      </geometry>
+      <material
+        name="">
+        <color
+          rgba="0.75294 0.75294 0.75294 1" />
+      </material>
+    </visual>
+    <collision>
+      <origin
+        xyz="0 0 0"
+        rpy="0 0 0" />
+      <geometry>
+        <mesh
+          filename="package://kuka_kr210_support/meshes/kr210l150/collision/link_3.stl" />
+      </geometry>
+    </collision>
+  </link>
+  <joint
+    name="${prefix}joint_3"
     type="revolute">
     <origin
@@ -198,7 +198,7 @@
       rpy="0 0 0" />
     <parent
-      link="${prefix}Link2" />
-    <child
-      link="${prefix}Link3" />
+      link="${prefix}link_2" />
+    <child
+      link="${prefix}link_3" />
     <axis
       xyz="0 1 0" />
@@ -206,5 +206,5 @@
   </joint>
   <link
-    name="${prefix}Link4">
+    name="${prefix}link_4">
     <inertial>
       <origin
@@ -227,24 +227,24 @@
       <geometry>
         <mesh
-          filename="package://kuka_kr210_support/meshes/visual/Link4.dae" />
-      </geometry>
-      <material
-        name="">
-        <color
-          rgba="0.75294 0.75294 0.75294 1" />
-      </material>
-    </visual>
-    <collision>
-      <origin
-        xyz="0 0 0"
-        rpy="0 0 0" />
-      <geometry>
-        <mesh
-          filename="package://kuka_kr210_support/meshes/collision/Link4.stl" />
-      </geometry>
-    </collision>
-  </link>
-  <joint
-    name="${prefix}J4"
+          filename="package://kuka_kr210_support/meshes/kr210l150/visual/link_4.dae" />
+      </geometry>
+      <material
+        name="">
+        <color
+          rgba="0.75294 0.75294 0.75294 1" />
+      </material>
+    </visual>
+    <collision>
+      <origin
+        xyz="0 0 0"
+        rpy="0 0 0" />
+      <geometry>
+        <mesh
+          filename="package://kuka_kr210_support/meshes/kr210l150/collision/link_4.stl" />
+      </geometry>
+    </collision>
+  </link>
+  <joint
+    name="${prefix}joint_4"
     type="revolute">
     <origin
@@ -252,7 +252,7 @@
       rpy="0 0 0" />
     <parent
-      link="${prefix}Link3" />
-    <child
-      link="${prefix}Link4" />
+      link="${prefix}link_3" />
+    <child
+      link="${prefix}link_4" />
     <axis
       xyz="1 0 0" />
@@ -260,5 +260,5 @@
   </joint>
   <link
-    name="${prefix}Link5">
+    name="${prefix}link_5">
     <inertial>
       <origin
@@ -281,24 +281,24 @@
       <geometry>
         <mesh
-          filename="package://kuka_kr210_support/meshes/visual/Link5.dae" />
-      </geometry>
-      <material
-        name="">
-        <color
-          rgba="0.75294 0.75294 0.75294 1" />
-      </material>
-    </visual>
-    <collision>
-      <origin
-        xyz="0 0 0"
-        rpy="0 0 0" />
-      <geometry>
-        <mesh
-          filename="package://kuka_kr210_support/meshes/collision/Link5.stl" />
-      </geometry>
-    </collision>
-  </link>
-  <joint
-    name="${prefix}J5"
+          filename="package://kuka_kr210_support/meshes/kr210l150/visual/link_5.dae" />
+      </geometry>
+      <material
+        name="">
+        <color
+          rgba="0.75294 0.75294 0.75294 1" />
+      </material>
+    </visual>
+    <collision>
+      <origin
+        xyz="0 0 0"
+        rpy="0 0 0" />
+      <geometry>
+        <mesh
+          filename="package://kuka_kr210_support/meshes/kr210l150/collision/link_5.stl" />
+      </geometry>
+    </collision>
+  </link>
+  <joint
+    name="${prefix}joint_5"
     type="revolute">
     <origin
@@ -306,7 +306,7 @@
       rpy="0 0 0" />
     <parent
-      link="${prefix}Link4" />
-    <child
-      link="${prefix}Link5" />
+      link="${prefix}link_4" />
+    <child
+      link="${prefix}link_5" />
     <axis
       xyz="0 1 0" />
@@ -314,5 +314,5 @@
   </joint>
   <link
-    name="${prefix}Link6">
+    name="${prefix}link_6">
     <inertial>
       <origin
@@ -335,24 +335,24 @@
       <geometry>
         <mesh
-          filename="package://kuka_kr210_support/meshes/visual/Link6.dae" />
-      </geometry>
-      <material
-        name="">
-        <color
-          rgba="0.75294 0.75294 0.75294 1" />
-      </material>
-    </visual>
-    <collision>
-      <origin
-        xyz="0 0 0"
-        rpy="0 0 0" />
-      <geometry>
-        <mesh
-          filename="package://kuka_kr210_support/meshes/collision/Link6.stl" />
-      </geometry>
-    </collision>
-  </link>
-  <joint
-    name="${prefix}J6"
+          filename="package://kuka_kr210_support/meshes/kr210l150/visual/link_6.dae" />
+      </geometry>
+      <material
+        name="">
+        <color
+          rgba="0.75294 0.75294 0.75294 1" />
+      </material>
+    </visual>
+    <collision>
+      <origin
+        xyz="0 0 0"
+        rpy="0 0 0" />
+      <geometry>
+        <mesh
+          filename="package://kuka_kr210_support/meshes/kr210l150/collision/link_6.stl" />
+      </geometry>
+    </collision>
+  </link>
+  <joint
+    name="${prefix}joint_6"
     type="revolute">
     <origin
@@ -360,7 +360,7 @@
       rpy="0 0 0" />
     <parent
-      link="${prefix}Link5" />
-    <child
-      link="${prefix}Link6" />
+      link="${prefix}link_5" />
+    <child
+      link="${prefix}link_6" />
     <axis
       xyz="1 0 0" />
@@ -369,5 +369,5 @@
   <link name="${prefix}tool0" />
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
Commit message: kr210l150: rename 'Link1' to 'link_1'.
Brings link name in-line with other links in xacro macro. A fixed joint
linking 'Link1' with 'link_1' is added to preserve bw-compatibility.

File: kuka_kr210_support/urdf/kr210l150.urdf (robot description, URDF)
Before this commit: robot kuka_kr210, 8 links, 7 joints
Links:
- added link Link1
Joints:
- added joint Link1-link_1: type fixed, parent link_1, child Link1, origin xyz=0 0 0 rpy=0 0 0

File: kuka_kr210_support/urdf/kr210l150_macro.xacro (robot description, xacro)
@@ -28,5 +28,5 @@
       </collision>
     </link>
-    <link name="${prefix}Link1">
+    <link name="${prefix}link_1">
       <inertial>
         <origin xyz="-0.036811 -0.024697 0.56577" rpy="0 0 0"/>
@@ -166,5 +166,5 @@
       <origin xyz="-0.00262 0.00097586 0.33099" rpy="0 0 0"/>
       <parent link="${prefix}base_link"/>
-      <child link="${prefix}Link1"/>
+      <child link="${prefix}link_1"/>
       <axis xyz="0 0 1"/>
       <limit lower="${-185*deg}" upper="${185*deg}" effort="0" velocity="${123*deg}"/>
@@ -172,5 +172,5 @@
     <joint name="${prefix}joint_2" type="revolute">
       <origin xyz="0.35277 -0.037476 0.4192" rpy="0 0 0"/>
-      <parent link="${prefix}Link1"/>
+      <parent link="${prefix}link_1"/>
       <child link="${prefix}link_2"/>
       <axis xyz="0 1 0"/>
@@ -210,4 +210,11 @@
       <origin xyz="0.0375 0 -0.00023924" rpy="0 0 0"/>
     </joint>
+    <!-- rename 'Link1' to 'link_1', maintain bw-compatibility -->
+    <link name="${prefix}Link1"/>
+    <joint name="${prefix}Link1-link_1" type="fixed">
+      <parent link="${prefix}link_1"/>
+      <child link="${prefix}Link1"/>
+      <origin xyz="0 0 0" rpy="0 0 0"/>
+    </joint>
   </xacro:macro>
 </robot>

Commit message: kr210: update joint names of L150 to follow conventions. Fix #37

File: kuka_kr210_support/urdf/kr210l150.urdf (robot description, URDF)
Before this commit: robot kuka_kr210, 9 links, 8 joints
Joints:
- removed joint joint_1
- removed joint joint_2
- removed joint joint_3
- removed joint joint_4
- removed joint joint_5
- removed joint joint_6
- added joint joint_a1: type revolute, parent base_link, child link_1, origin xyz=-0.00262 0.00097586 0.33099 rpy=0 0 0, axis 0 0 1, limit lower=-3.228859205 upper=3.228859205 effort=0 velocity=2.146755039
- added joint joint_a2: type revolute, parent link_1, child link_2, origin xyz=0.35277 -0.037476 0.4192 rpy=0 0 0, axis 0 1 0, limit lower=-0.785398185 upper=1.483529905 effort=0 velocity=2.007128695
- added joint joint_a3: type revolute, parent link_2, child link_3, origin xyz=-9.8483E-05 -0.1475 1.2499 rpy=0 0 0, axis 0 1 0, limit lower=-3.66519153 upper=1.134464045 effort=0 velocity=1.954768816
- added joint joint_a4: type revolute, parent link_3, child link_4, origin xyz=0.95795 0.184 -0.055059 rpy=0 0 0, axis 1 0 0, limit lower=-6.10865255 upper=6.10865255 effort=0 velocity=3.124139447
- added joint joint_a5: type revolute, parent link_4, child link_5, origin xyz=0.542 0 0 rpy=0 0 0, axis 0 1 0, limit lower=-2.181661625 upper=2.181661625 effort=0 velocity=3.001966396
- added joint joint_a6: type revolute, parent link_5, child link_6, origin xyz=0.1925 0 0 rpy=0 0 0, axis 1 0 0, limit lower=-6.10865255 upper=6.10865255 effort=0 velocity=3.822271167

File: kuka_kr210_support/urdf/kr210l150_macro.xacro (robot description, xacro)
@@ -163,5 +163,5 @@
     <link name="${prefix}tool0"/>
     <!-- joints -->
-    <joint name="${prefix}joint_1" type="revolute">
+    <joint name="${prefix}joint_a1" type="revolute">
       <origin xyz="-0.00262 0.00097586 0.33099" rpy="0 0 0"/>
       <parent link="${prefix}base_link"/>
@@ -170,5 +170,5 @@
       <limit lower="${-185*deg}" upper="${185*deg}" effort="0" velocity="${123*deg}"/>
     </joint>
-    <joint name="${prefix}joint_2" type="revolute">
+    <joint name="${prefix}joint_a2" type="revolute">
       <origin xyz="0.35277 -0.037476 0.4192" rpy="0 0 0"/>
       <parent link="${prefix}link_1"/>
@@ -177,5 +177,5 @@
       <limit lower="${-45*deg}" upper="${85*deg}" effort="0" velocity="${115*deg}"/>
     </joint>
-    <joint name="${prefix}joint_3" type="revolute">
+    <joint name="${prefix}joint_a3" type="revolute">
       <origin xyz="-9.8483E-05 -0.1475 1.2499" rpy="0 0 0"/>
       <parent link="${prefix}link_2"/>
@@ -184,5 +184,5 @@
       <limit lower="${-210*deg}" upper="${(155-90)*deg}" effort="0" velocity="${112*deg}"/>
     </joint>
-    <joint name="${prefix}joint_4" type="revolute">
+    <joint name="${prefix}joint_a4" type="revolute">
       <origin xyz="0.95795 0.184 -0.055059" rpy="0 0 0"/>
       <parent link="${prefix}link_3"/>
@@ -191,5 +191,5 @@
       <limit lower="${-350*deg}" upper="${350*deg}" effort="0" velocity="${179*deg}"/>
     </joint>
-    <joint name="${prefix}joint_5" type="revolute">
+    <joint name="${prefix}joint_a5" type="revolute">
       <origin xyz="0.542 0 0" rpy="0 0 0"/>
       <parent link="${prefix}link_4"/>
@@ -198,5 +198,5 @@
       <limit lower="${-125*deg}" upper="${125*deg}" effort="0" velocity="${172*deg}"/>
     </joint>
-    <joint name="${prefix}joint_6" type="revolute">
+    <joint name="${prefix}joint_a6" type="revolute">
       <origin xyz="0.1925 0 0" rpy="0 0 0"/>
       <parent link="${prefix}link_5"/>
