Commit message: split L150 and L150-2 into separate xacro/launch files

File: kuka_kr210_support/urdf/kr210l150-2.xacro (robot description, xacro)
@@ -1,5 +1,5 @@
 <?xml version="1.0" ?>
-<robot name="kuka_kr210" xmlns:xacro="http://wiki.ros.org/xacro">
-  <xacro:include filename="$(find kuka_kr210_support)/urdf/kr210l150_macro.xacro"/>
-  <xacro:kuka_kr210l150 prefix="" model="2"/>
+<robot name="kuka_kr210-2" xmlns:xacro="http://wiki.ros.org/xacro">
+  <xacro:include filename="$(find kuka_kr210_support)/urdf/kr210l150-2_macro.xacro"/>
+  <xacro:kuka_kr210l150-2 prefix=""/>
 </robot>

File: kuka_kr210_support/urdf/kr210l150-2_macro.xacro (robot description, xacro)
@@ -3,5 +3,5 @@
   <xacro:include filename="$(find kuka_resources)/urdf/common_constants.xacro"/>
   <xacro:include filename="$(find kuka_resources)/urdf/common_materials.xacro"/>
-  <xacro:macro name="kuka_kr210l150" params="prefix">
+  <xacro:macro name="kuka_kr210l150-2" params="prefix">
     <!-- links -->
     <link name="${prefix}base_link">
@@ -128,9 +128,9 @@
     </joint>
     <joint name="${prefix}joint_a3" type="revolute">
-      <origin xyz="0 0 1.25" rpy="0 ${radians(90)} 0"/>
+      <origin xyz="0 0 1.25" rpy="0 0 0"/>
       <parent link="${prefix}link_2"/>
       <child link="${prefix}link_3"/>
       <axis xyz="0 1 0"/>
-      <limit lower="${radians(-219)}" upper="${radians(65)}" effort="0" velocity="${radians(81)}"/>
+      <limit lower="${radians(-119)}" upper="${radians(155)}" effort="0" velocity="${radians(81)}"/>
     </joint>
     <joint name="${prefix}joint_a4" type="revolute">

File: kuka_kr210_support/urdf/kr210l150.xacro (robot description, xacro)
@@ -1,5 +1,5 @@
 <?xml version="1.0" ?>
-<robot name="kuka_kr210" xmlns:xacro="http://wiki.ros.org/xacro">
+<robot name="kuka_kr210l150" xmlns:xacro="http://wiki.ros.org/xacro">
   <xacro:include filename="$(find kuka_kr210_support)/urdf/kr210l150_macro.xacro"/>
-  <xacro:kuka_kr210l150 prefix="" model=""/>
+  <xacro:kuka_kr210l150 prefix=""/>
 </robot>
