Commit message: added support for R900

File: kuka_kr10_support/urdf/kr10r900sixx.xacro (robot description, xacro)
@@ -1,4 +1,4 @@
 <?xml version="1.0"?>
-<robot name="kuka_kr6r900sixx" xmlns:xacro="http://wiki.ros.org/xacro">
+<robot name="kuka_kr10r900sixx" xmlns:xacro="http://wiki.ros.org/xacro">
   <xacro:include filename="$(find kuka_kr6_support)/urdf/krXr900sixx_macro.xacro" />
   <xacro:kuka_krXr900sixx prefix=""/>

File: kuka_kr6_support/urdf/krXr900sixx_macro.xacro (robot description, xacro)
@@ -1,7 +1,6 @@
 <?xml version="1.0"?>
 <robot xmlns:xacro="http://wiki.ros.org/xacro">
-  <xacro:include filename="$(find kuka_resources)/urdf/common_constants.xacro"/>
   <xacro:include filename="$(find kuka_resources)/urdf/common_materials.xacro"/>
-  <xacro:macro name="kuka_kr6r900sixx" params="prefix">
+  <xacro:macro name="kuka_krXr900sixx" params="prefix">
     <link name="${prefix}base_link">
       <visual>
@@ -116,5 +115,5 @@
       <child link="${prefix}link_1"/>
       <axis xyz="0 0 -1"/>
-      <limit effort="0" lower="${-DEG2RAD * 170}" upper="${DEG2RAD * 170}" velocity="${DEG2RAD * 360}"/>
+      <limit effort="0" lower="${radians(-170)}" upper="${radians(170)}" velocity="${radians(360)}"/>
     </joint>
     <joint name="${prefix}joint_a2" type="revolute">
@@ -123,5 +122,5 @@
       <child link="${prefix}link_2"/>
       <axis xyz="0 1 0"/>
-      <limit effort="0" lower="${-DEG2RAD * 190}" upper="${DEG2RAD * 45}" velocity="${DEG2RAD * 300}"/>
+      <limit effort="0" lower="${radians(-190)}" upper="${radians(45)}" velocity="${radians(300)}"/>
     </joint>
     <joint name="${prefix}joint_a3" type="revolute">
@@ -130,5 +129,5 @@
       <child link="${prefix}link_3"/>
       <axis xyz="0 1 0"/>
-      <limit effort="0" lower="${-DEG2RAD * 120}" upper="${DEG2RAD * 156}" velocity="${DEG2RAD * 360}"/>
+      <limit effort="0" lower="${radians(-120)}" upper="${radians(156)}" velocity="${radians(360)}"/>
     </joint>
     <joint name="${prefix}joint_a4" type="revolute">
@@ -137,5 +136,5 @@
       <child link="${prefix}link_4"/>
       <axis xyz="-1 0 0"/>
-      <limit effort="0" lower="${-DEG2RAD * 185}" upper="${DEG2RAD * 185}" velocity="${DEG2RAD * 381}"/>
+      <limit effort="0" lower="${radians(-185)}" upper="${radians(185)}" velocity="${radians(381)}"/>
     </joint>
     <joint name="${prefix}joint_a5" type="revolute">
@@ -144,5 +143,5 @@
       <child link="${prefix}link_5"/>
       <axis xyz="0 1 0"/>
-      <limit effort="0" lower="${-DEG2RAD * 120}" upper="${DEG2RAD * 120}" velocity="${DEG2RAD * 388}"/>
+      <limit effort="0" lower="${radians(-120)}" upper="${radians(120)}" velocity="${radians(388)}"/>
     </joint>
     <joint name="${prefix}joint_a6" type="revolute">
@@ -151,10 +150,10 @@
       <child link="${prefix}link_6"/>
       <axis xyz="-1 0 0"/>
-      <limit effort="0" lower="${-DEG2RAD * 350}" upper="${DEG2RAD * 350}" velocity="${DEG2RAD * 615}"/>
+      <limit effort="0" lower="${radians(-350)}" upper="${radians(350)}" velocity="${radians(615)}"/>
     </joint>
     <joint name="${prefix}joint_a6-tool0" type="fixed">
       <parent link="${prefix}link_6"/>
       <child link="${prefix}tool0"/>
-      <origin xyz="0 0 0" rpy="0 ${DEG2RAD * 90} 0"/>
+      <origin xyz="0 0 0" rpy="0 ${radians(90)} 0"/>
     </joint>
     <!-- ROS base_link to KUKA $ROBROOT coordinate system transform -->
