Commit message: Proxon modify

File: kuka_kr10_support/urdf/proxxon_drill_macro.xacro (robot description, xacro)
@@ -6,5 +6,5 @@
     <link name="${prefix}drilling_tool_link">
       <visual>
-        <origin xyz="0 0 0" rpy="0 0 0"/>
+        <origin xyz="-0.15 0 -0.1035" rpy="-${DEG2RAD * 90} -${DEG2RAD * 0} ${DEG2RAD * 90}"/>
         <geometry>
           <mesh filename="package://kuka_kr10_support/meshes/kr10r1100sixx/visual/proxxon_drilling.stl" scale="0.001 0.001 0.001" />
@@ -13,5 +13,5 @@
       </visual>
       <collision>
-        <origin xyz="0 0 0" rpy="0 0 0"/>
+        <origin xyz="-0.15 0 -0.1035" rpy="-${DEG2RAD * 90} -${DEG2RAD * 0} ${DEG2RAD * 90}"/>
         <geometry>
           <mesh filename="package://kuka_kr10_support/meshes/kr10r1100sixx/collision/proxxon_drilling.stl" scale="0.001 0.001 0.001" />
@@ -20,5 +20,5 @@
       <inertial>
         <mass value="50" />
-        <origin xyz="0.05 0.00 -0.00" rpy="0 0 0" />
+        <origin xyz="-0.15 0 -0.1035" rpy="-${DEG2RAD * 90} -${DEG2RAD * 0} ${DEG2RAD * 90}" />
         <inertia ixx="0.00402901710341" ixy="0.000210543968708" ixz="4.6068390983e-05" iyy="0.00668778512296" iyz="1.26910167997e-06" izz="0.00711775677213" />
       </inertial>
@@ -26,5 +26,5 @@
     <!-- joint between arm_6_link and drilling_tool_link -->
     <joint name="${prefix}joint_drilling_tool_link" type="fixed">
-      <origin xyz="0.0375 0 0" rpy="${DEG2RAD * 0} ${DEG2RAD * 0} ${DEG2RAD * 90}" />
+      <origin xyz="0.1035 0 -0.15" rpy="${DEG2RAD * 0} ${DEG2RAD * 90} ${DEG2RAD * 0}" />
       <parent link="${prefix}link_6"/>
       <child link="${prefix}drilling_tool_link"/>

Commit message: Modify x position

File: kuka_kr10_support/urdf/proxxon_drill_macro.xacro (robot description, xacro)
@@ -6,5 +6,5 @@
     <link name="${prefix}drilling_tool_link">
       <visual>
-        <origin xyz="-0.15 0 -0.1035" rpy="-${DEG2RAD * 90} -${DEG2RAD * 0} ${DEG2RAD * 90}"/>
+        <origin xyz="-0.157 0 -0.066" rpy="-${DEG2RAD * 90} -${DEG2RAD * 0} ${DEG2RAD * 90}"/>
         <geometry>
           <mesh filename="package://kuka_kr10_support/meshes/kr10r1100sixx/visual/proxxon_drilling.stl" scale="0.001 0.001 0.001" />
@@ -13,5 +13,5 @@
       </visual>
       <collision>
-        <origin xyz="-0.15 0 -0.1035" rpy="-${DEG2RAD * 90} -${DEG2RAD * 0} ${DEG2RAD * 90}"/>
+        <origin xyz="-0.157 0 -0.066" rpy="-${DEG2RAD * 90} -${DEG2RAD * 0} ${DEG2RAD * 90}"/>
         <geometry>
           <mesh filename="package://kuka_kr10_support/meshes/kr10r1100sixx/collision/proxxon_drilling.stl" scale="0.001 0.001 0.001" />
@@ -20,5 +20,5 @@
       <inertial>
         <mass value="50" />
-        <origin xyz="-0.15 0 -0.1035" rpy="-${DEG2RAD * 90} -${DEG2RAD * 0} ${DEG2RAD * 90}" />
+        <origin xyz="-0.157 0 -0.066" rpy="-${DEG2RAD * 90} -${DEG2RAD * 0} ${DEG2RAD * 90}" />
         <inertia ixx="0.00402901710341" ixy="0.000210543968708" ixz="4.6068390983e-05" iyy="0.00668778512296" iyz="1.26910167997e-06" izz="0.00711775677213" />
       </inertial>
@@ -26,5 +26,5 @@
     <!-- joint between arm_6_link and drilling_tool_link -->
     <joint name="${prefix}joint_drilling_tool_link" type="fixed">
-      <origin xyz="0.1035 0 -0.15" rpy="${DEG2RAD * 0} ${DEG2RAD * 90} ${DEG2RAD * 0}" />
+      <origin xyz="0.1035 0 -0.157" rpy="${DEG2RAD * 0} ${DEG2RAD * 90} ${DEG2RAD * 0}" />
       <parent link="${prefix}link_6"/>
       <child link="${prefix}drilling_tool_link"/>

Commit message: Minor changes in xacro

File: kuka_kr10_support/urdf/proxxon_drill_macro.xacro (robot description, xacro)
@@ -6,19 +6,19 @@
     <link name="${prefix}drilling_tool_link">
       <visual>
-        <origin xyz="-0.157 0 -0.066" rpy="-${DEG2RAD * 90} -${DEG2RAD * 0} ${DEG2RAD * 90}"/>
+        <origin xyz="-0.1564 0 -0.066" rpy="-${DEG2RAD * 90} -${DEG2RAD * 0} ${DEG2RAD * 90}"/>
         <geometry>
-          <mesh filename="package://kuka_kr10_support/meshes/kr10r1100sixx/visual/proxxon_drilling.stl" scale="0.001 0.001 0.001" />
+          <mesh filename="package://kuka_kr10_support/meshes/kr10r1100sixx/visual/proxxon_drilling_v2.stl" scale="0.001 0.001 0.001" />
         </geometry>
         <xacro:material_kuka_orange />
       </visual>
       <collision>
-        <origin xyz="-0.157 0 -0.066" rpy="-${DEG2RAD * 90} -${DEG2RAD * 0} ${DEG2RAD * 90}"/>
+        <origin xyz="-0.1564 0 -0.066" rpy="-${DEG2RAD * 90} -${DEG2RAD * 0} ${DEG2RAD * 90}"/>
         <geometry>
-          <mesh filename="package://kuka_kr10_support/meshes/kr10r1100sixx/collision/proxxon_drilling.stl" scale="0.001 0.001 0.001" />
+          <mesh filename="package://kuka_kr10_support/meshes/kr10r1100sixx/collision/proxxon_drilling_v2.stl" scale="0.001 0.001 0.001" />
         </geometry>
       </collision>
       <inertial>
         <mass value="50" />
-        <origin xyz="-0.157 0 -0.066" rpy="-${DEG2RAD * 90} -${DEG2RAD * 0} ${DEG2RAD * 90}" />
+        <origin xyz="-0.1564 0 -0.066" rpy="-${DEG2RAD * 90} -${DEG2RAD * 0} ${DEG2RAD * 90}" />
         <inertia ixx="0.00402901710341" ixy="0.000210543968708" ixz="4.6068390983e-05" iyy="0.00668778512296" iyz="1.26910167997e-06" izz="0.00711775677213" />
       </inertial>
