Commit message: kr10r1100sixx: changing visual meshes from stl to collada
Adopting colors from existing models:
Kuka orange - RAL2003
Base/flange - RAL9005

File: kuka_kr10_support/urdf/kr10r1100sixx_macro.xacro (robot description, xacro)
@@ -8,5 +8,5 @@
         <origin xyz="0 0 0" rpy="0 0 0"/>
         <geometry>
-          <mesh filename="package://kuka_kr10_support/meshes/kr10r1100sixx/visual/base.stl" />
+          <mesh filename="package://kuka_kr10_support/meshes/kr10r1100sixx/visual/base.dae" />
         </geometry>
         <xacro:material_kuka_black />
@@ -23,5 +23,5 @@
         <origin xyz="0 0 0" rpy="0 0 0"/>
         <geometry>
-          <mesh filename="package://kuka_kr10_support/meshes/kr10r1100sixx/visual/link_1.stl" />
+          <mesh filename="package://kuka_kr10_support/meshes/kr10r1100sixx/visual/link_1.dae" />
         </geometry>
         <xacro:material_kuka_orange />
@@ -38,5 +38,5 @@
         <origin xyz="0 0 0" rpy="0 0 0"/>
         <geometry>
-          <mesh filename="package://kuka_kr10_support/meshes/kr10r1100sixx/visual/link_2.stl"/>
+          <mesh filename="package://kuka_kr10_support/meshes/kr10r1100sixx/visual/link_2.dae"/>
         </geometry>
         <xacro:material_kuka_orange />
@@ -53,5 +53,5 @@
         <origin xyz="0 0 0" rpy="0 0 0"/>
         <geometry>
-          <mesh filename="package://kuka_kr10_support/meshes/kr10r1100sixx/visual/link_3.stl" />
+          <mesh filename="package://kuka_kr10_support/meshes/kr10r1100sixx/visual/link_3.dae" />
         </geometry>
         <xacro:material_kuka_orange />
@@ -68,5 +68,5 @@
         <origin xyz="0 0 0" rpy="0 0 0"/>
         <geometry>
-          <mesh filename="package://kuka_kr10_support/meshes/kr10r1100sixx/visual/link_4.stl" />
+          <mesh filename="package://kuka_kr10_support/meshes/kr10r1100sixx/visual/link_4.dae" />
         </geometry>
         <xacro:material_kuka_orange />
@@ -83,5 +83,5 @@
         <origin xyz="0 0 0" rpy="0 0 0"/>
         <geometry>
-          <mesh filename="package://kuka_kr10_support/meshes/kr10r1100sixx/visual/link_5.stl" />
+          <mesh filename="package://kuka_kr10_support/meshes/kr10r1100sixx/visual/link_5.dae" />
         </geometry>
         <xacro:material_kuka_orange />
@@ -98,5 +98,5 @@
         <origin xyz="0 0 0" rpy="0 0 0"/>
         <geometry>
-          <mesh filename="package://kuka_kr10_support/meshes/kr10r1100sixx/visual/link_6.stl" />
+          <mesh filename="package://kuka_kr10_support/meshes/kr10r1100sixx/visual/link_6.dae" />
         </geometry>
         <xacro:material_kuka_pedestal />

Commit message: Fix: base -> base_link.(stl,dae)

File: kuka_kr10_support/urdf/kr10r1100sixx_macro.xacro (robot description, xacro)
@@ -8,5 +8,5 @@
         <origin xyz="0 0 0" rpy="0 0 0"/>
         <geometry>
-          <mesh filename="package://kuka_kr10_support/meshes/kr10r1100sixx/visual/base.dae" />
+          <mesh filename="package://kuka_kr10_support/meshes/kr10r1100sixx/visual/base_link.dae" />
         </geometry>
         <xacro:material_kuka_black />
@@ -15,5 +15,5 @@
         <origin xyz="0 0 0" rpy="0 0 0"/>
         <geometry>
-          <mesh filename="package://kuka_kr10_support/meshes/kr10r1100sixx/collision/base.stl" />
+          <mesh filename="package://kuka_kr10_support/meshes/kr10r1100sixx/collision/base_link.stl" />
         </geometry>
       </collision>

Commit message: Revert "kr10r1100sixx: changing visual meshes from stl to collada"
This reverts commit 45da9182eee46bc202042aa0e039f1d7689302bb.

File: kuka_kr10_support/urdf/kr10r1100sixx_macro.xacro (robot description, xacro)
@@ -8,5 +8,5 @@
         <origin xyz="0 0 0" rpy="0 0 0"/>
         <geometry>
-          <mesh filename="package://kuka_kr10_support/meshes/kr10r1100sixx/visual/base_link.dae" />
+          <mesh filename="package://kuka_kr10_support/meshes/kr10r1100sixx/visual/base_link.stl" />
         </geometry>
         <xacro:material_kuka_black />
@@ -23,5 +23,5 @@
         <origin xyz="0 0 0" rpy="0 0 0"/>
         <geometry>
-          <mesh filename="package://kuka_kr10_support/meshes/kr10r1100sixx/visual/link_1.dae" />
+          <mesh filename="package://kuka_kr10_support/meshes/kr10r1100sixx/visual/link_1.stl" />
         </geometry>
         <xacro:material_kuka_orange />
@@ -38,5 +38,5 @@
         <origin xyz="0 0 0" rpy="0 0 0"/>
         <geometry>
-          <mesh filename="package://kuka_kr10_support/meshes/kr10r1100sixx/visual/link_2.dae"/>
+          <mesh filename="package://kuka_kr10_support/meshes/kr10r1100sixx/visual/link_2.stl"/>
         </geometry>
         <xacro:material_kuka_orange />
@@ -53,5 +53,5 @@
         <origin xyz="0 0 0" rpy="0 0 0"/>
         <geometry>
-          <mesh filename="package://kuka_kr10_support/meshes/kr10r1100sixx/visual/link_3.dae" />
+          <mesh filename="package://kuka_kr10_support/meshes/kr10r1100sixx/visual/link_3.stl" />
         </geometry>
         <xacro:material_kuka_orange />
@@ -68,5 +68,5 @@
         <origin xyz="0 0 0" rpy="0 0 0"/>
         <geometry>
-          <mesh filename="package://kuka_kr10_support/meshes/kr10r1100sixx/visual/link_4.dae" />
+          <mesh filename="package://kuka_kr10_support/meshes/kr10r1100sixx/visual/link_4.stl" />
         </geometry>
         <xacro:material_kuka_orange />
@@ -83,5 +83,5 @@
         <origin xyz="0 0 0" rpy="0 0 0"/>
         <geometry>
-          <mesh filename="package://kuka_kr10_support/meshes/kr10r1100sixx/visual/link_5.dae" />
+          <mesh filename="package://kuka_kr10_support/meshes/kr10r1100sixx/visual/link_5.stl" />
         </geometry>
         <xacro:material_kuka_orange />
@@ -98,5 +98,5 @@
         <origin xyz="0 0 0" rpy="0 0 0"/>
         <geometry>
-          <mesh filename="package://kuka_kr10_support/meshes/kr10r1100sixx/visual/link_6.dae" />
+          <mesh filename="package://kuka_kr10_support/meshes/kr10r1100sixx/visual/link_6.stl" />
         </geometry>
         <xacro:material_kuka_pedestal />

Commit message: Added dummy inertial values in kr10 for gazebo

File: kuka_kr10_support/urdf/kr10r1100sixx_macro.xacro (robot description, xacro)
@@ -18,4 +18,11 @@
         </geometry>
       </collision>
+      <inertial> <!-- DUMMY VALUES -->
+        <mass value="10.733459"/>
+        <origin xyz="0.014288 0.000001 0.122264" rpy="0.0 0.0 0.0"/>
+        <inertia ixx="0.096590" ixy="-0.000005" ixz="-0.003803"
+                                iyy="0.087591"  iyz="-0.000001"
+                                                izz="0.081632"/>
+      </inertial>
     </link>
     <link name="${prefix}link_1">
@@ -33,4 +40,11 @@
         </geometry>
       </collision>
+      <inertial> <!-- DUMMY VALUES -->
+        <mass value="10.733459"/>
+        <origin xyz="0.014288 0.000001 0.122264" rpy="0.0 0.0 0.0"/>
+        <inertia ixx="0.096590" ixy="-0.000005" ixz="-0.003803"
+                                iyy="0.087591"  iyz="-0.000001"
+                                                izz="0.081632"/>
+      </inertial>
     </link>
     <link name="${prefix}link_2">
@@ -48,4 +62,11 @@
         </geometry>
       </collision>
+      <inertial> <!-- DUMMY VALUES -->
+        <mass value="10.733459"/>
+        <origin xyz="0.014288 0.000001 0.122264" rpy="0.0 0.0 0.0"/>
+        <inertia ixx="0.096590" ixy="-0.000005" ixz="-0.003803"
+                                iyy="0.087591"  iyz="-0.000001"
+                                                izz="0.081632"/>
+      </inertial>
     </link>
     <link name="${prefix}link_3">
@@ -63,4 +84,11 @@
         </geometry>
       </collision>
+      <inertial> <!-- DUMMY VALUES -->
+        <mass value="10.733459"/>
+        <origin xyz="0.014288 0.000001 0.122264" rpy="0.0 0.0 0.0"/>
+        <inertia ixx="0.096590" ixy="-0.000005" ixz="-0.003803"
+                                iyy="0.087591"  iyz="-0.000001"
+                                                izz="0.081632"/>
+      </inertial>
     </link>
     <link name="${prefix}link_4">
@@ -78,4 +106,11 @@
         </geometry>
       </collision>
+      <inertial> <!-- DUMMY VALUES -->
+        <mass value="10.733459"/>
+        <origin xyz="0.014288 0.000001 0.122264" rpy="0.0 0.0 0.0"/>
+        <inertia ixx="0.096590" ixy="-0.000005" ixz="-0.003803"
+                                iyy="0.087591"  iyz="-0.000001"
+                                                izz="0.081632"/>
+      </inertial>
     </link>
     <link name="${prefix}link_5">
@@ -93,4 +128,11 @@
         </geometry>
       </collision>
+      <inertial> <!-- DUMMY VALUES -->
+        <mass value="10.733459"/>
+        <origin xyz="0.014288 0.000001 0.122264" rpy="0.0 0.0 0.0"/>
+        <inertia ixx="0.096590" ixy="-0.000005" ixz="-0.003803"
+                                iyy="0.087591"  iyz="-0.000001"
+                                                izz="0.081632"/>
+      </inertial>
     </link>
     <link name="${prefix}link_6">
@@ -108,4 +150,11 @@
         </geometry>
       </collision>
+      <inertial> <!-- DUMMY VALUES -->
+        <mass value="10.733459"/>
+        <origin xyz="0.014288 0.000001 0.122264" rpy="0.0 0.0 0.0"/>
+        <inertia ixx="0.096590" ixy="-0.000005" ixz="-0.003803"
+                                iyy="0.087591"  iyz="-0.000001"
+                                                izz="0.081632"/>
+      </inertial>
     </link>
     <!-- This frame corresponds to the $FLANGE coordinate system in KUKA KRC controllers. -->

Commit message: Added link and mass macros to common_parameters and replaced corresponding data in xacro

File: kuka_kr10_support/urdf/kr10r1100sixx_macro.xacro (robot description, xacro)
@@ -3,4 +3,5 @@
   <xacro:include filename="$(find kuka_resources)/urdf/common_constants.xacro"/>
   <xacro:include filename="$(find kuka_resources)/urdf/common_materials.xacro"/>
+  <xacro:include filename="$(find kuka_resources)/urdf/common_robotparameters.xacro"/>
   <xacro:macro name="kuka_kr10r1100sixx" params="prefix">
     <link name="${prefix}base_link">
@@ -18,11 +19,7 @@
         </geometry>
       </collision>
-      <inertial> <!-- DUMMY VALUES -->
-        <mass value="10.733459"/>
-        <origin xyz="0.014288 0.000001 0.122264" rpy="0.0 0.0 0.0"/>
-        <inertia ixx="0.096590" ixy="-0.000005" ixz="-0.003803"
-                                iyy="0.087591"  iyz="-0.000001"
-                                                izz="0.081632"/>
-      </inertial>
+      <xacro:cylinder_inertial radius="${kuka_kr10r1100sixx_d1/4}" length="${kuka_kr10r1100sixx_d1/2}" mass="${kuka_kr10r1100sixx_base_link_mass}">
+        <origin xyz="0.0 0.0 0.0" rpy="0 0 0" />
+      </xacro:cylinder_inertial>
     </link>
     <link name="${prefix}link_1">
@@ -40,11 +37,7 @@
         </geometry>
       </collision>
-      <inertial> <!-- DUMMY VALUES -->
-        <mass value="10.733459"/>
-        <origin xyz="0.014288 0.000001 0.122264" rpy="0.0 0.0 0.0"/>
-        <inertia ixx="0.096590" ixy="-0.000005" ixz="-0.003803"
-                                iyy="0.087591"  iyz="-0.000001"
-                                                izz="0.081632"/>
-      </inertial>
+      <xacro:cylinder_inertial radius="${kuka_kr10r1100sixx_d1/4}" length="${kuka_kr10r1100sixx_d1/2}" mass="${kuka_kr10r1100sixx_link_1_mass}">
+        <origin xyz="0.0 0.0 0.0" rpy="0 0 0" />
+      </xacro:cylinder_inertial>
     </link>
     <link name="${prefix}link_2">
@@ -62,11 +55,7 @@
         </geometry>
       </collision>
-      <inertial> <!-- DUMMY VALUES -->
-        <mass value="10.733459"/>
-        <origin xyz="0.014288 0.000001 0.122264" rpy="0.0 0.0 0.0"/>
-        <inertia ixx="0.096590" ixy="-0.000005" ixz="-0.003803"
-                                iyy="0.087591"  iyz="-0.000001"
-                                                izz="0.081632"/>
-      </inertial>
+      <xacro:cylinder_inertial radius="${kuka_kr10r1100sixx_d1/4}" length="${kuka_kr10r1100sixx_a2}" mass="${kuka_kr10r1100sixx_link_2_mass}">
+        <origin xyz="0.0 0.0 0.0" rpy="0 0 0" />
+      </xacro:cylinder_inertial>
     </link>
     <link name="${prefix}link_3">
@@ -84,11 +73,7 @@
         </geometry>
       </collision>
-      <inertial> <!-- DUMMY VALUES -->
-        <mass value="10.733459"/>
-        <origin xyz="0.014288 0.000001 0.122264" rpy="0.0 0.0 0.0"/>
-        <inertia ixx="0.096590" ixy="-0.000005" ixz="-0.003803"
-                                iyy="0.087591"  iyz="-0.000001"
-                                                izz="0.081632"/>
-      </inertial>
+      <xacro:cylinder_inertial radius="${kuka_kr10r1100sixx_a3}" length="${kuka_kr10r1100sixx_a3*10}" mass="${kuka_kr10r1100sixx_link_3_mass}">
+        <origin xyz="0.0 0.0 0.0" rpy="0 0 0" />
+      </xacro:cylinder_inertial>
     </link>
     <link name="${prefix}link_4">
@@ -106,11 +91,7 @@
         </geometry>
       </collision>
-      <inertial> <!-- DUMMY VALUES -->
-        <mass value="10.733459"/>
-        <origin xyz="0.014288 0.000001 0.122264" rpy="0.0 0.0 0.0"/>
-        <inertia ixx="0.096590" ixy="-0.000005" ixz="-0.003803"
-                                iyy="0.087591"  iyz="-0.000001"
-                                                izz="0.081632"/>
-      </inertial>
+      <xacro:cylinder_inertial radius="${kuka_kr10r1100sixx_d1/4}" length="${kuka_kr10r1100sixx_d4}" mass="${kuka_kr10r1100sixx_link_4_mass}">
+        <origin xyz="0.0 0.0 0.0" rpy="0 0 0" />
+      </xacro:cylinder_inertial>
     </link>
     <link name="${prefix}link_5">
@@ -128,11 +109,7 @@
         </geometry>
       </collision>
-      <inertial> <!-- DUMMY VALUES -->
-        <mass value="10.733459"/>
-        <origin xyz="0.014288 0.000001 0.122264" rpy="0.0 0.0 0.0"/>
-        <inertia ixx="0.096590" ixy="-0.000005" ixz="-0.003803"
-                                iyy="0.087591"  iyz="-0.000001"
-                                                izz="0.081632"/>
-      </inertial>
+      <xacro:cylinder_inertial radius="${kuka_kr10r1100sixx_a5/2}" length="${kuka_kr10r1100sixx_a5}" mass="${kuka_kr10r1100sixx_link_5_mass}">
+        <origin xyz="0.0 0.0 0.0" rpy="0 0 0" />
+      </xacro:cylinder_inertial>
     </link>
     <link name="${prefix}link_6">
@@ -150,16 +127,12 @@
         </geometry>
       </collision>
-      <inertial> <!-- DUMMY VALUES -->
-        <mass value="10.733459"/>
-        <origin xyz="0.014288 0.000001 0.122264" rpy="0.0 0.0 0.0"/>
-        <inertia ixx="0.096590" ixy="-0.000005" ixz="-0.003803"
-                                iyy="0.087591"  iyz="-0.000001"
-                                                izz="0.081632"/>
-      </inertial>
+      <xacro:cylinder_inertial radius="${kuka_kr10r1100sixx_a5/2}" length="${kuka_kr10r1100sixx_a5/10}" mass="${kuka_kr10r1100sixx_link_6_mass}">
+        <origin xyz="0.0 0.0 0.0" rpy="0 0 0" />
+      </xacro:cylinder_inertial>
     </link>
     <!-- This frame corresponds to the $FLANGE coordinate system in KUKA KRC controllers. -->
     <link name="${prefix}tool0"/>
     <joint name="${prefix}joint_a1" type="revolute">
-      <origin xyz="0 0 0.400" rpy="0 0 0"/>
+      <origin xyz="0 0 ${kuka_kr10r1100sixx_d1}" rpy="0 0 0"/>
       <parent link="${prefix}base_link"/>
       <child link="${prefix}link_1"/>
@@ -168,5 +141,5 @@
     </joint>
     <joint name="${prefix}joint_a2" type="revolute">
-      <origin xyz="0.025 0 0" rpy="0 0 0"/>
+      <origin xyz="${kuka_kr10r1100sixx_a1} 0 0" rpy="0 0 0"/>
       <parent link="${prefix}link_1"/>
       <child link="${prefix}link_2"/>
@@ -175,5 +148,5 @@
     </joint>
     <joint name="${prefix}joint_a3" type="revolute">
-      <origin xyz="0.560 0 0" rpy="0 0 0"/>
+      <origin xyz="${kuka_kr10r1100sixx_a2} 0 0" rpy="0 0 0"/>
       <parent link="${prefix}link_2"/>
       <child link="${prefix}link_3"/>
@@ -182,5 +155,5 @@
     </joint>
     <joint name="${prefix}joint_a4" type="revolute">
-      <origin xyz="0 0 0.035" rpy="0 0 0"/>
+      <origin xyz="0 0 ${kuka_kr10r1100sixx_a3}" rpy="0 0 0"/>
       <parent link="${prefix}link_3"/>
       <child link="${prefix}link_4"/>
@@ -189,5 +162,5 @@
     </joint>
     <joint name="${prefix}joint_a5" type="revolute">
-      <origin xyz="0.515 0 0" rpy="0 0 0"/>
+      <origin xyz="${kuka_kr10r1100sixx_d4} 0 0" rpy="0 0 0"/>
       <parent link="${prefix}link_4"/>
       <child link="${prefix}link_5"/>
@@ -196,5 +169,5 @@
     </joint>
     <joint name="${prefix}joint_a6" type="revolute">
-      <origin xyz="0.080 0 0" rpy="0 0 0"/>
+      <origin xyz="${kuka_kr10r1100sixx_a5} 0 0" rpy="0 0 0"/>
       <parent link="${prefix}link_5"/>
       <child link="${prefix}link_6"/>

Commit message: Integrated robotparameters to kr10r1100sixx_macro.xacro

File: kuka_kr10_support/urdf/kr10r1100sixx_macro.xacro (robot description, xacro)
@@ -3,5 +3,29 @@
   <xacro:include filename="$(find kuka_resources)/urdf/common_constants.xacro"/>
   <xacro:include filename="$(find kuka_resources)/urdf/common_materials.xacro"/>
-  <xacro:include filename="$(find kuka_resources)/urdf/common_robotparameters.xacro"/>
+  <!-- Mass parameters (guessed), total mass should be 55 kg -->
+  <xacro:property name="kuka_kr10r1100sixx_base_link_mass" value="4.0" />
+  <xacro:property name="kuka_kr10r1100sixx_link_1_mass" value="4.0" />
+  <xacro:property name="kuka_kr10r1100sixx_link_2_mass" value="19.0" />
+  <xacro:property name="kuka_kr10r1100sixx_link_3_mass" value="10.0" />
+  <xacro:property name="kuka_kr10r1100sixx_link_4_mass" value="15.0" />
+  <xacro:property name="kuka_kr10r1100sixx_link_5_mass" value="2.8" />
+  <xacro:property name="kuka_kr10r1100sixx_link_6_mass" value="0.2" />
+  <!-- Kinematic parameters -->
+  <xacro:property name="kuka_kr10r1100sixx_d1" value="0.400" />
+  <xacro:property name="kuka_kr10r1100sixx_d4" value="0.515" />
+  <xacro:property name="kuka_kr10r1100sixx_a1" value="0.025" />
+  <xacro:property name="kuka_kr10r1100sixx_a2" value="0.560" />
+  <xacro:property name="kuka_kr10r1100sixx_a3" value="0.035" />
+  <xacro:property name="kuka_kr10r1100sixx_a5" value="0.080" />
+  <!-- Cylindrical inertia tensor -->
+  <xacro:macro name="cylinder_inertial" params="radius length mass *origin">
+   <inertial>
+     <mass value="${mass}" />
+     <xacro:insert_block name="origin" />
+     <inertia ixx="${0.0833333 * mass * (3 * radius * radius + length * length)}" ixy="0.0" ixz="0.0"
+       iyy="${0.0833333 * mass * (3 * radius * radius + length * length)}" iyz="0.0"
+       izz="${0.5 * mass * radius * radius}" />
+   </inertial>
+ </xacro:macro>
   <xacro:macro name="kuka_kr10r1100sixx" params="prefix">
     <link name="${prefix}base_link">
