Commit message: More descriptive parameter names

File: kuka_kr10_support/urdf/kr10r1100sixx_macro.xacro (robot description, xacro)
@@ -4,18 +4,18 @@
   <xacro:include filename="$(find kuka_resources)/urdf/common_materials.xacro"/>
   <!-- Mass parameters (guessed), total mass should be 55 kg -->
-  <xacro:property name="kuka_kr10r1100sixx_base_link_mass" value="4.0" />
-  <xacro:property name="kuka_kr10r1100sixx_link_1_mass" value="4.0" />
-  <xacro:property name="kuka_kr10r1100sixx_link_2_mass" value="19.0" />
-  <xacro:property name="kuka_kr10r1100sixx_link_3_mass" value="10.0" />
-  <xacro:property name="kuka_kr10r1100sixx_link_4_mass" value="15.0" />
-  <xacro:property name="kuka_kr10r1100sixx_link_5_mass" value="2.8" />
-  <xacro:property name="kuka_kr10r1100sixx_link_6_mass" value="0.2" />
+  <xacro:property name="base_mass" value="4.0" />
+  <xacro:property name="link1_mass" value="4.0" />
+  <xacro:property name="link2_mass" value="19.0" />
+  <xacro:property name="link3_mass" value="10.0" />
+  <xacro:property name="link4_mass" value="15.0" />
+  <xacro:property name="link5_mass" value="2.8" />
+  <xacro:property name="link6_mass" value="0.2" />
   <!-- Kinematic parameters -->
-  <xacro:property name="kuka_kr10r1100sixx_d1" value="0.400" />
-  <xacro:property name="kuka_kr10r1100sixx_d4" value="0.515" />
-  <xacro:property name="kuka_kr10r1100sixx_a1" value="0.025" />
-  <xacro:property name="kuka_kr10r1100sixx_a2" value="0.560" />
-  <xacro:property name="kuka_kr10r1100sixx_a3" value="0.035" />
-  <xacro:property name="kuka_kr10r1100sixx_a5" value="0.080" />
+  <xacro:property name="base_link1_length" value="0.400" />
+  <xacro:property name="link1_link2_offset" value="0.025" />
+  <xacro:property name="link2_length" value="0.560" />
+  <xacro:property name="link2_link3_offset" value="0.035" />
+  <xacro:property name="link3_link4_length" value="0.515" />
+  <xacro:property name="link5_link6_length" value="0.080" />
   <!-- Cylindrical inertia tensor -->
   <xacro:macro name="cylinder_inertial" params="radius length mass *origin">
@@ -43,5 +43,5 @@
         </geometry>
       </collision>
-      <xacro:cylinder_inertial radius="${kuka_kr10r1100sixx_d1/4}" length="${kuka_kr10r1100sixx_d1/2}" mass="${kuka_kr10r1100sixx_base_link_mass}">
+      <xacro:cylinder_inertial radius="${base_link1_length/4}" length="${base_link1_length/2}" mass="${base_mass}">
         <origin xyz="0.0 0.0 0.0" rpy="0 0 0" />
       </xacro:cylinder_inertial>
@@ -61,5 +61,5 @@
         </geometry>
       </collision>
-      <xacro:cylinder_inertial radius="${kuka_kr10r1100sixx_d1/4}" length="${kuka_kr10r1100sixx_d1/2}" mass="${kuka_kr10r1100sixx_link_1_mass}">
+      <xacro:cylinder_inertial radius="${base_link1_length/4}" length="${base_link1_length/2}" mass="${link1_mass}">
         <origin xyz="0.0 0.0 0.0" rpy="0 0 0" />
       </xacro:cylinder_inertial>
@@ -79,5 +79,5 @@
         </geometry>
       </collision>
-      <xacro:cylinder_inertial radius="${kuka_kr10r1100sixx_d1/4}" length="${kuka_kr10r1100sixx_a2}" mass="${kuka_kr10r1100sixx_link_2_mass}">
+      <xacro:cylinder_inertial radius="${base_link1_length/4}" length="${link2_length}" mass="${link2_mass}">
         <origin xyz="0.0 0.0 0.0" rpy="0 0 0" />
       </xacro:cylinder_inertial>
@@ -97,5 +97,5 @@
         </geometry>
       </collision>
-      <xacro:cylinder_inertial radius="${kuka_kr10r1100sixx_a3}" length="${kuka_kr10r1100sixx_a3*10}" mass="${kuka_kr10r1100sixx_link_3_mass}">
+      <xacro:cylinder_inertial radius="${link2_link3_offset}" length="${link2_link3_offset*10}" mass="${link3_mass}">
         <origin xyz="0.0 0.0 0.0" rpy="0 0 0" />
       </xacro:cylinder_inertial>
@@ -115,5 +115,5 @@
         </geometry>
       </collision>
-      <xacro:cylinder_inertial radius="${kuka_kr10r1100sixx_d1/4}" length="${kuka_kr10r1100sixx_d4}" mass="${kuka_kr10r1100sixx_link_4_mass}">
+      <xacro:cylinder_inertial radius="${base_link1_length/4}" length="${link3_link4_length}" mass="${link4_mass}">
         <origin xyz="0.0 0.0 0.0" rpy="0 0 0" />
       </xacro:cylinder_inertial>
@@ -133,5 +133,5 @@
         </geometry>
       </collision>
-      <xacro:cylinder_inertial radius="${kuka_kr10r1100sixx_a5/2}" length="${kuka_kr10r1100sixx_a5}" mass="${kuka_kr10r1100sixx_link_5_mass}">
+      <xacro:cylinder_inertial radius="${link5_link6_length/2}" length="${link5_link6_length}" mass="${link5_mass}">
         <origin xyz="0.0 0.0 0.0" rpy="0 0 0" />
       </xacro:cylinder_inertial>
@@ -151,5 +151,5 @@
         </geometry>
       </collision>
-      <xacro:cylinder_inertial radius="${kuka_kr10r1100sixx_a5/2}" length="${kuka_kr10r1100sixx_a5/10}" mass="${kuka_kr10r1100sixx_link_6_mass}">
+      <xacro:cylinder_inertial radius="${link5_link6_length/2}" length="${link5_link6_length/10}" mass="${link6_mass}">
         <origin xyz="0.0 0.0 0.0" rpy="0 0 0" />
       </xacro:cylinder_inertial>
@@ -158,5 +158,5 @@
     <link name="${prefix}tool0"/>
     <joint name="${prefix}joint_a1" type="revolute">
-      <origin xyz="0 0 ${kuka_kr10r1100sixx_d1}" rpy="0 0 0"/>
+      <origin xyz="0 0 ${base_link1_length}" rpy="0 0 0"/>
       <parent link="${prefix}base_link"/>
       <child link="${prefix}link_1"/>
@@ -165,5 +165,5 @@
     </joint>
     <joint name="${prefix}joint_a2" type="revolute">
-      <origin xyz="${kuka_kr10r1100sixx_a1} 0 0" rpy="0 0 0"/>
+      <origin xyz="${link1_link2_offset} 0 0" rpy="0 0 0"/>
       <parent link="${prefix}link_1"/>
       <child link="${prefix}link_2"/>
@@ -172,5 +172,5 @@
     </joint>
     <joint name="${prefix}joint_a3" type="revolute">
-      <origin xyz="${kuka_kr10r1100sixx_a2} 0 0" rpy="0 0 0"/>
+      <origin xyz="${link2_length} 0 0" rpy="0 0 0"/>
       <parent link="${prefix}link_2"/>
       <child link="${prefix}link_3"/>
@@ -179,5 +179,5 @@
     </joint>
     <joint name="${prefix}joint_a4" type="revolute">
-      <origin xyz="0 0 ${kuka_kr10r1100sixx_a3}" rpy="0 0 0"/>
+      <origin xyz="0 0 ${link2_link3_offset}" rpy="0 0 0"/>
       <parent link="${prefix}link_3"/>
       <child link="${prefix}link_4"/>
@@ -186,5 +186,5 @@
     </joint>
     <joint name="${prefix}joint_a5" type="revolute">
-      <origin xyz="${kuka_kr10r1100sixx_d4} 0 0" rpy="0 0 0"/>
+      <origin xyz="${link3_link4_length} 0 0" rpy="0 0 0"/>
       <parent link="${prefix}link_4"/>
       <child link="${prefix}link_5"/>
@@ -193,5 +193,5 @@
     </joint>
     <joint name="${prefix}joint_a6" type="revolute">
-      <origin xyz="${kuka_kr10r1100sixx_a5} 0 0" rpy="0 0 0"/>
+      <origin xyz="${link5_link6_length} 0 0" rpy="0 0 0"/>
       <parent link="${prefix}link_5"/>
       <child link="${prefix}link_6"/>

Commit message: Modify joint names

File: kuka_kr10_support/urdf/kr10r1100sixx_macro.xacro (robot description, xacro)
@@ -18,4 +18,9 @@
         </geometry>
       </collision>
+      <inertial>
+        <mass value="14" />
+        <origin xyz="-0.0444859 -4.97e-05 0.1100921" rpy="0 0 0" />
+        <inertia ixx="0.08877213773" ixy="-0.000131033070251" ixz="-0.00150261923247" iyy="0.14293778144" iyz="-2.25256850538e-05" izz="0.126259385464" />
+      </inertial>
     </link>
     <link name="${prefix}link_1">
@@ -33,4 +38,9 @@
         </geometry>
       </collision>
+      <inertial>
+        <mass value="11.2" />
+        <origin xyz="0.0146723 5.46e-05 -0.0557645" rpy="0 0 0" />
+        <inertia ixx="0.10800091083" ixy="0.000256908100066" ixz="-0.00448959204754" iyy="0.0892932854513" iyz="-0.000186133409604" izz="0.0838171097348" />
+      </inertial>
     </link>
     <link name="${prefix}link_2">
@@ -48,4 +58,9 @@
         </geometry>
       </collision>
+      <inertial>
+        <mass value="8.4" />
+        <origin xyz="0.2482357 -0.0029221 0.0079418" rpy="0 0 0" />
+        <inertia ixx="0.0365241429014" ixy="0.00223732223794" ixz="-0.00177293915942" iyy="0.378539351981" iyz="2.8964263294e-06" izz="0.392538210121" />
+      </inertial>
     </link>
     <link name="${prefix}link_3">
@@ -63,4 +78,9 @@
         </geometry>
       </collision>
+      <inertial>
+        <mass value="8.4" />
+        <origin xyz="0.0160924 2.38e-05 0.0105013" rpy="0 0 0" />
+        <inertia ixx="0.0238712171376" ixy="1.72719757663e-06" ixz="-0.00409828855491" iyy="0.0325090200419" iyz="-1.11535979101e-05" izz="0.0287380207905" />
+      </inertial>
     </link>
     <link name="${prefix}link_4">
@@ -78,4 +98,9 @@
         </geometry>
       </collision>
+      <inertial>
+        <mass value="5.6" />
+        <origin xyz="0.301148 -0.0004543 0.000235" rpy="0 0 0" />
+        <inertia ixx="0.0101469645454" ixy="0.000122992246096" ixz="-8.45337146292e-05" iyy="0.070495864179" iyz="8.8953596453e-07" izz="0.0717697213772" />
+      </inertial>
     </link>
     <link name="${prefix}link_5">
@@ -93,4 +118,9 @@
         </geometry>
       </collision>
+      <inertial>
+        <mass value="5.6" />
+        <origin xyz="0.0157906 0.0019162 -0.0002449" rpy="0 0 0" />
+        <inertia ixx="0.00402901710341" ixy="0.000210543968708" ixz="4.6068390983e-05" iyy="0.00668778512296" iyz="1.26910167997e-06" izz="0.00711775677213" />
+      </inertial>
     </link>
     <link name="${prefix}link_6">
@@ -108,4 +138,9 @@
         </geometry>
       </collision>
+      <inertial>
+        <mass value="2.8" />
+        <origin xyz="-0.0075312 1e-07 -0.0009341" rpy="0 0 0" />
+        <inertia ixx="0.000603033772181" ixy="-0.0" ixz="-4.00686891815e-06" iyy="-4.00686891815e-06" iyz="-0.0" izz="0.000340583858042" />
+      </inertial>
     </link>
     <!-- This frame corresponds to the $FLANGE coordinate system in KUKA KRC controllers. -->

Commit message: modify parameters for kuka interface

File: kuka_kr10_support/urdf/kr10r1100sixx_macro.xacro (robot description, xacro)
@@ -145,5 +145,5 @@
     </link>
     <!-- This frame corresponds to the $FLANGE coordinate system in KUKA KRC controllers. -->
-    <link name="${prefix}tool0"/>
+    <!--link name="${prefix}tool0"/-->
     <joint name="${prefix}joint_a1" type="revolute">
       <origin xyz="0 0 0.400" rpy="0 0 0"/>
@@ -188,9 +188,9 @@
       <limit effort="0" lower="${-DEG2RAD * 350}" upper="${DEG2RAD * 350}" velocity="${DEG2RAD * 615}"/>
     </joint>
-    <joint name="${prefix}joint_a6-tool0" type="fixed">
+    <!--joint name="${prefix}joint_a6-tool0" type="fixed">
       <parent link="${prefix}link_6"/>
       <child link="${prefix}tool0"/>
       <origin xyz="0 0 0" rpy="0 ${DEG2RAD * 90} 0"/>
-    </joint>
+    </joint-->
     <!-- ROS base_link to KUKA $ROBROOT coordinate system transform -->
     <link name="${prefix}base" />

Commit message: fixed joint limits

File: kuka_kr10_support/urdf/kr10r1100sixx_macro.xacro (robot description, xacro)
@@ -116,5 +116,5 @@
       <child link="${prefix}link_1"/>
       <axis xyz="0 0 -1"/>
-      <limit effort="0" lower="${-DEG2RAD * 170}" upper="${DEG2RAD * 170}" velocity="${DEG2RAD * 360}"/>
+      <limit effort="0" lower="${radians()}" upper="${radians()}" velocity="${radians()}"/>
     </joint>
     <joint name="${prefix}joint_a2" type="revolute">
@@ -123,5 +123,5 @@
       <child link="${prefix}link_2"/>
       <axis xyz="0 1 0"/>
-      <limit effort="0" lower="${-DEG2RAD * 190}" upper="${DEG2RAD * 45}" velocity="${DEG2RAD * 300}"/>
+      <limit effort="0" lower="${radians()}" upper="${radians()}" velocity="${radians()}"/>
     </joint>
     <joint name="${prefix}joint_a3" type="revolute">
@@ -130,5 +130,5 @@
       <child link="${prefix}link_3"/>
       <axis xyz="0 1 0"/>
-      <limit effort="0" lower="${-DEG2RAD * 120}" upper="${DEG2RAD * 156}" velocity="${DEG2RAD * 360}"/>
+      <limit effort="0" lower="${radians()}" upper="${radians()}" velocity="${radians()}"/>
     </joint>
     <joint name="${prefix}joint_a4" type="revolute">
@@ -137,5 +137,5 @@
       <child link="${prefix}link_4"/>
       <axis xyz="-1 0 0"/>
-      <limit effort="0" lower="${-DEG2RAD * 185}" upper="${DEG2RAD * 185}" velocity="${DEG2RAD * 381}"/>
+      <limit effort="0" lower="${radians()}" upper="${radians()}" velocity="${radians()}"/>
     </joint>
     <joint name="${prefix}joint_a5" type="revolute">
@@ -144,5 +144,5 @@
       <child link="${prefix}link_5"/>
       <axis xyz="0 1 0"/>
-      <limit effort="0" lower="${-DEG2RAD * 120}" upper="${DEG2RAD * 120}" velocity="${DEG2RAD * 388}"/>
+      <limit effort="0" lower="${radians()}" upper="${radians()}" velocity="${radians()}"/>
     </joint>
     <joint name="${prefix}joint_a6" type="revolute">
@@ -151,10 +151,10 @@
       <child link="${prefix}link_6"/>
       <axis xyz="-1 0 0"/>
-      <limit effort="0" lower="${-DEG2RAD * 350}" upper="${DEG2RAD * 350}" velocity="${DEG2RAD * 615}"/>
+      <limit effort="0" lower="${radians()}" upper="${radians()}" velocity="${radians()}"/>
     </joint>
     <joint name="${prefix}joint_a6-tool0" type="fixed">
       <parent link="${prefix}link_6"/>
       <child link="${prefix}tool0"/>
-      <origin xyz="0 0 0" rpy="0 ${DEG2RAD * 90} 0"/>
+      <origin xyz="0 0 0" rpy="0 ${radians(90)} 0"/>
     </joint>
     <!-- ROS base_link to KUKA $ROBROOT coordinate system transform -->

Commit message: fixed joint limits

File: kuka_kr10_support/urdf/kr10r1100sixx_macro.xacro (robot description, xacro)
@@ -116,5 +116,5 @@
       <child link="${prefix}link_1"/>
       <axis xyz="0 0 -1"/>
-      <limit effort="0" lower="${radians()}" upper="${radians()}" velocity="${radians()}"/>
+      <limit effort="0" lower="${radians(-170)}" upper="${radians(170)}" velocity="${radians(300)}"/>
     </joint>
     <joint name="${prefix}joint_a2" type="revolute">
@@ -123,5 +123,5 @@
       <child link="${prefix}link_2"/>
       <axis xyz="0 1 0"/>
-      <limit effort="0" lower="${radians()}" upper="${radians()}" velocity="${radians()}"/>
+      <limit effort="0" lower="${radians(-190)}" upper="${radians(45)}" velocity="${radians(225)}"/>
     </joint>
     <joint name="${prefix}joint_a3" type="revolute">
@@ -130,5 +130,5 @@
       <child link="${prefix}link_3"/>
       <axis xyz="0 1 0"/>
-      <limit effort="0" lower="${radians()}" upper="${radians()}" velocity="${radians()}"/>
+      <limit effort="0" lower="${radians(-120)}" upper="${radians(156)}" velocity="${radians(225)}"/>
     </joint>
     <joint name="${prefix}joint_a4" type="revolute">
@@ -137,5 +137,5 @@
       <child link="${prefix}link_4"/>
       <axis xyz="-1 0 0"/>
-      <limit effort="0" lower="${radians()}" upper="${radians()}" velocity="${radians()}"/>
+      <limit effort="0" lower="${radians(-185)}" upper="${radians(185)}" velocity="${radians(381)}"/>
     </joint>
     <joint name="${prefix}joint_a5" type="revolute">
@@ -144,5 +144,5 @@
       <child link="${prefix}link_5"/>
       <axis xyz="0 1 0"/>
-      <limit effort="0" lower="${radians()}" upper="${radians()}" velocity="${radians()}"/>
+      <limit effort="0" lower="${radians(-120)}" upper="${radians(120)}" velocity="${radians(311)}"/>
     </joint>
     <joint name="${prefix}joint_a6" type="revolute">
@@ -151,5 +151,5 @@
       <child link="${prefix}link_6"/>
       <axis xyz="-1 0 0"/>
-      <limit effort="0" lower="${radians()}" upper="${radians()}" velocity="${radians()}"/>
+      <limit effort="0" lower="${radians(-350)}" upper="${radians(350)}" velocity="${radians(492)}"/>
     </joint>
     <joint name="${prefix}joint_a6-tool0" type="fixed">
