Commit message: Replace pi and DEG2RAD xacro properties with radians()

File: kuka_kr10_support/urdf/kr10r1100sixx_macro.xacro (robot description, xacro)
@@ -170,5 +170,5 @@
       <parent link="${prefix}flange"/>
       <child link="${prefix}tool0"/>
-      <origin xyz="0 0 0" rpy="0 ${pi*0.5} 0"/>
+      <origin xyz="0 0 0" rpy="0 ${radians(90)} 0"/>
     </joint>
   </xacro:macro>

File: kuka_kr120_support/urdf/kr120r2500pro_macro.xacro (robot description, xacro)
@@ -1,5 +1,4 @@
 <?xml version="1.0"?>
 <robot xmlns:xacro="http://wiki.ros.org/xacro">
-  <xacro:property name="DEG2RAD" value="0.017453292519943295"/>
   <xacro:macro name="kuka_kr120r2500pro" params="prefix">
     <!-- LINKS -->
@@ -154,5 +153,5 @@
       <child link="${prefix}link_1"/>
       <axis xyz="0 0 -1"/>
-      <limit effort="0" lower="${-DEG2RAD * 185}" upper="${DEG2RAD * 185}" velocity="${DEG2RAD * 156}"/>
+      <limit effort="0" lower="${-radians(185)}" upper="${radians(185)}" velocity="${radians(156)}"/>
     </joint>
     <!-- joint 2 (A2) -->
@@ -162,5 +161,5 @@
       <child link="${prefix}link_2"/>
       <axis xyz="0 1 0"/>
-      <limit effort="0" lower="${-DEG2RAD * 155}" upper="${DEG2RAD * 35}" velocity="${DEG2RAD * 156}"/>
+      <limit effort="0" lower="${-radians(155)}" upper="${radians(35)}" velocity="${radians(156)}"/>
     </joint>
     <!-- joint 3 (A3) -->
@@ -170,5 +169,5 @@
       <child link="${prefix}link_3"/>
       <axis xyz="0 1 0"/>
-      <limit effort="0" lower="${-DEG2RAD * 130}" upper="${DEG2RAD * 154}" velocity="${DEG2RAD * 156}"/>
+      <limit effort="0" lower="${-radians(130)}" upper="${radians(154)}" velocity="${radians(156)}"/>
     </joint>
     <!-- joint 4 (A4) -->
@@ -178,5 +177,5 @@
       <child link="${prefix}link_4"/>
       <axis xyz="-1 0 0"/>
-      <limit effort="0" lower="${-DEG2RAD * 350}" upper="${DEG2RAD * 350}" velocity="${DEG2RAD * 330}"/>
+      <limit effort="0" lower="${-radians(350)}" upper="${radians(350)}" velocity="${radians(330)}"/>
     </joint>
     <!-- joint 5 (A5) -->
@@ -186,5 +185,5 @@
       <child link="${prefix}link_5"/>
       <axis xyz="0 1 0"/>
-      <limit effort="0" lower="${-DEG2RAD * 130}" upper="${DEG2RAD * 130}" velocity="${DEG2RAD * 330}"/>
+      <limit effort="0" lower="${-radians(130)}" upper="${radians(130)}" velocity="${radians(330)}"/>
     </joint>
     <!-- joint 6 (A6) -->
@@ -194,5 +193,5 @@
       <child link="${prefix}link_6"/>
       <axis xyz="-1 0 0"/>
-      <limit effort="0" lower="${-DEG2RAD * 350}" upper="${DEG2RAD * 350}" velocity="${DEG2RAD * 615}"/>
+      <limit effort="0" lower="${-radians(350)}" upper="${radians(350)}" velocity="${radians(615)}"/>
     </joint>
     <!-- tool frame - fixed frame -->
@@ -215,5 +214,5 @@
       <parent link="${prefix}flange"/>
       <child link="${prefix}tool0"/>
-      <origin xyz="0 0 0" rpy="0 ${pi*0.5} 0"/>
+      <origin xyz="0 0 0" rpy="0 ${radians(90)} 0"/>
     </joint>
   </xacro:macro>

File: kuka_kr150_support/urdf/kr150_2_macro.xacro (robot description, xacro)
@@ -180,5 +180,5 @@
       <parent link="${prefix}flange"/>
       <child link="${prefix}tool0"/>
-      <origin xyz="0 0 0" rpy="0 ${pi*0.5} 0"/>
+      <origin xyz="0 0 0" rpy="0 ${radians(90)} 0"/>
     </joint>
   </xacro:macro>

File: kuka_kr16_support/urdf/kr16_2_macro.xacro (robot description, xacro)
@@ -215,5 +215,5 @@
       <parent link="${prefix}flange"/>
       <child link="${prefix}tool0"/>
-      <origin xyz="0 0 0" rpy="0 ${pi*0.5} 0"/>
+      <origin xyz="0 0 0" rpy="0 ${radians(90)} 0"/>
     </joint>
   </xacro:macro>

File: kuka_kr210_support/urdf/kr210l150_macro.xacro (robot description, xacro)
@@ -1,7 +1,4 @@
 <?xml version="1.0"?>
 <robot xmlns:xacro="http://wiki.ros.org/xacro">
-  <property name="pi" value="3.141592654"/>
-  <!--degrees to radians-->
-  <property name="deg" value="0.017453293"/>
   <xacro:macro name="kuka_kr210l150" params="prefix">
     <!-- links -->
@@ -13,5 +10,5 @@
       </inertial>
       <visual>
-        <origin xyz="0 0 0" rpy="${-pi/2} 0 0"/>
+        <origin xyz="0 0 0" rpy="${-radians(90)} 0 0"/>
         <geometry>
           <mesh filename="package://kuka_kr210_support/meshes/kr210l150/visual/base_link.dae"/>
@@ -22,5 +19,5 @@
       </visual>
       <collision>
-        <origin xyz="0 0 0" rpy="${-pi/2} 0 0"/>
+        <origin xyz="0 0 0" rpy="${-radians(90)} 0 0"/>
         <geometry>
           <mesh filename="package://kuka_kr210_support/meshes/kr210l150/collision/base_link.stl"/>
@@ -57,5 +54,5 @@
       </inertial>
       <visual>
-        <origin xyz="0 0 0" rpy="${-pi/2} 0 0"/>
+        <origin xyz="0 0 0" rpy="${-radians(90)} 0 0"/>
         <geometry>
           <mesh filename="package://kuka_kr210_support/meshes/kr210l150/visual/link_2.dae"/>
@@ -79,5 +76,5 @@
       </inertial>
       <visual>
-        <origin xyz="0 0 0" rpy="${-pi/2} 0 0"/>
+        <origin xyz="0 0 0" rpy="${-radians(90)} 0 0"/>
         <geometry>
           <mesh filename="package://kuka_kr210_support/meshes/kr210l150/visual/link_3.dae"/>
@@ -101,5 +98,5 @@
       </inertial>
       <visual>
-        <origin xyz="0 0 0" rpy="${-pi/2} 0 0"/>
+        <origin xyz="0 0 0" rpy="${-radians(90)} 0 0"/>
         <geometry>
           <mesh filename="package://kuka_kr210_support/meshes/kr210l150/visual/link_4.dae"/>
@@ -123,5 +120,5 @@
       </inertial>
       <visual>
-        <origin xyz="0 0 0" rpy="${-pi/2} 0 0"/>
+        <origin xyz="0 0 0" rpy="${-radians(90)} 0 0"/>
         <geometry>
           <mesh filename="package://kuka_kr210_support/meshes/kr210l150/visual/link_5.dae"/>
@@ -168,5 +165,5 @@
       <child link="${prefix}link_1"/>
       <axis xyz="0 0 1"/>
-      <limit lower="${-185*deg}" upper="${185*deg}" effort="0" velocity="${123*deg}"/>
+      <limit lower="${radians(-185)}" upper="${radians(185)}" effort="0" velocity="${radians(123)}"/>
     </joint>
     <joint name="${prefix}joint_a2" type="revolute">
@@ -175,5 +172,5 @@
       <child link="${prefix}link_2"/>
       <axis xyz="0 1 0"/>
-      <limit lower="${-45*deg}" upper="${85*deg}" effort="0" velocity="${115*deg}"/>
+      <limit lower="${radians(-45)}" upper="${radians(85)}" effort="0" velocity="${radians(115)}"/>
     </joint>
     <joint name="${prefix}joint_a3" type="revolute">
@@ -182,5 +179,5 @@
       <child link="${prefix}link_3"/>
       <axis xyz="0 1 0"/>
-      <limit lower="${-210*deg}" upper="${(155-90)*deg}" effort="0" velocity="${112*deg}"/>
+      <limit lower="${radians(-210)}" upper="${radians(65)}" effort="0" velocity="${radians(112)}"/>
     </joint>
     <joint name="${prefix}joint_a4" type="revolute">
@@ -189,5 +186,5 @@
       <child link="${prefix}link_4"/>
       <axis xyz="1 0 0"/>
-      <limit lower="${-350*deg}" upper="${350*deg}" effort="0" velocity="${179*deg}"/>
+      <limit lower="${radians(-350)}" upper="${radians(350)}" effort="0" velocity="${radians(179)}"/>
     </joint>
     <joint name="${prefix}joint_a5" type="revolute">
@@ -196,5 +193,5 @@
       <child link="${prefix}link_5"/>
       <axis xyz="0 1 0"/>
-      <limit lower="${-125*deg}" upper="${125*deg}" effort="0" velocity="${172*deg}"/>
+      <limit lower="${radians(-125)}" upper="${radians(125)}" effort="0" velocity="${radians(172)}"/>
     </joint>
     <joint name="${prefix}joint_a6" type="revolute">
@@ -203,5 +200,5 @@
       <child link="${prefix}link_6"/>
       <axis xyz="1 0 0"/>
-      <limit lower="${-350*deg}" upper="${350*deg}" effort="0" velocity="${219*deg}"/>
+      <limit lower="${radians(-350)}" upper="${radians(350)}" effort="0" velocity="${radians(219)}"/>
     </joint>
     <joint name="${prefix}link_6-flange" type="fixed">
@@ -222,5 +219,5 @@
       <parent link="${prefix}flange"/>
       <child link="${prefix}tool0"/>
-      <origin xyz="0 0 0" rpy="0 ${pi*0.5} 0"/>
+      <origin xyz="0 0 0" rpy="0 ${radians(90)} 0"/>
     </joint>
     <!-- rename 'Link1' to 'link_1', maintain bw-compatibility -->

File: kuka_kr5_support/urdf/kr5_arc_macro.xacro (robot description, xacro)
@@ -211,5 +211,5 @@
     <!-- joint 1 (A1) -->
     <joint name="${prefix}joint_a1" type="revolute">
-      <origin xyz="0 0 0.4" rpy="${pi} 0 0"/>
+      <origin xyz="0 0 0.4" rpy="${radians(180)} 0 0"/>
       <parent link="${prefix}base_link"/>
       <child link="${prefix}link_1"/>
@@ -219,5 +219,5 @@
     <!-- joint 2 (A2) -->
     <joint name="${prefix}joint_a2" type="revolute">
-      <origin xyz="0.18 0 0" rpy="${pi/2} 0 0"/>
+      <origin xyz="0.18 0 0" rpy="${radians(90)} 0 0"/>
       <parent link="${prefix}link_1"/>
       <child link="${prefix}link_2"/>
@@ -235,5 +235,5 @@
     <!-- joint 4 (A4) -->
     <joint name="${prefix}joint_a4" type="revolute">
-      <origin xyz="0 -0.12 0" rpy="0 ${-pi/2} 0"/>
+      <origin xyz="0 -0.12 0" rpy="0 ${-radians(90)} 0"/>
       <parent link="${prefix}link_3"/>
       <child link="${prefix}link_4"/>
@@ -243,5 +243,5 @@
     <!-- joint 5 (A5) -->
     <joint name="${prefix}joint_a5" type="revolute">
-      <origin xyz="0 0 -0.62" rpy="0 ${pi/2} 0"/>
+      <origin xyz="0 0 -0.62" rpy="0 ${radians(90)} 0"/>
       <parent link="${prefix}link_4"/>
       <child link="${prefix}link_5"/>
@@ -251,5 +251,5 @@
     <!-- joint 6 (A6) -->
     <joint name="${prefix}joint_a6" type="revolute">
-      <origin xyz="0 0 0" rpy="0 ${-pi/2} 0"/>
+      <origin xyz="0 0 0" rpy="0 ${-radians(90)} 0"/>
       <parent link="${prefix}link_5"/>
       <child link="${prefix}link_6"/>
@@ -261,5 +261,5 @@
       <parent link="${prefix}link_6"/>
       <child link="${prefix}flange"/>
-      <origin xyz="0 0 -0.115" rpy="0 ${pi*0.5} ${-pi/2}"/>
+      <origin xyz="0 0 -0.115" rpy="0 ${radians(90)} ${-radians(90)}"/>
     </joint>
     <!-- END JOINTS -->
@@ -276,5 +276,5 @@
       <parent link="${prefix}flange"/>
       <child link="${prefix}tool0"/>
-      <origin xyz="0 0 0" rpy="0 ${pi*0.5} 0"/>
+      <origin xyz="0 0 0" rpy="0 ${radians(90)} 0"/>
     </joint>
   </xacro:macro>

File: kuka_kr6_support/urdf/kr6r700sixx_macro.xacro (robot description, xacro)
@@ -116,5 +116,5 @@
       <child link="${prefix}link_1"/>
       <axis xyz="0 0 -1"/>
-      <limit lower="${-170 * DEG2RAD}" upper="${170 * DEG2RAD}" effort="0" velocity="${360 * DEG2RAD}"/>
+      <limit lower="${radians(-170)}" upper="${radians(170)}" effort="0" velocity="${radians(360)}"/>
     </joint>
     <joint name="${prefix}joint_a2" type="revolute">
@@ -123,5 +123,5 @@
       <child link="${prefix}link_2"/>
       <axis xyz="0 1 0"/>
-      <limit lower="${-190 * DEG2RAD}" upper="${45 * DEG2RAD}" effort="0" velocity="${300 * DEG2RAD}"/>
+      <limit lower="${radians(-190)}" upper="${radians(45)}" effort="0" velocity="${radians(300)}"/>
     </joint>
     <joint name="${prefix}joint_a3" type="revolute">
@@ -130,5 +130,5 @@
       <child link="${prefix}link_3"/>
       <axis xyz="0 1 0"/>
-      <limit lower="${-120 * DEG2RAD}" upper="${156 * DEG2RAD}" effort="0" velocity="${360 * DEG2RAD}"/>
+      <limit lower="${radians(-120)}" upper="${radians(156)}" effort="0" velocity="${radians(360)}"/>
     </joint>
     <joint name="${prefix}joint_a4" type="revolute">
@@ -137,5 +137,5 @@
       <child link="${prefix}link_4"/>
       <axis xyz="-1 0 0"/>
-      <limit lower="${-185 * DEG2RAD}" upper="${185 * DEG2RAD}" effort="0" velocity="${381 * DEG2RAD}"/>
+      <limit lower="${radians(-185)}" upper="${radians(185)}" effort="0" velocity="${radians(381)}"/>
     </joint>
     <joint name="${prefix}joint_a5" type="revolute">
@@ -144,5 +144,5 @@
       <child link="${prefix}link_5"/>
       <axis xyz="0 1 0"/>
-      <limit lower="${-120 * DEG2RAD}" upper="${120 * DEG2RAD}" effort="0" velocity="${388 * DEG2RAD}"/>
+      <limit lower="${radians(-120)}" upper="${radians(120)}" effort="0" velocity="${radians(388)}"/>
     </joint>
     <joint name="${prefix}joint_a6" type="revolute">
@@ -151,5 +151,5 @@
       <child link="${prefix}link_6"/>
       <axis xyz="-1 0 0"/>
-      <limit lower="${-350 * DEG2RAD}" upper="${350 * DEG2RAD}" effort="0" velocity="${615 * DEG2RAD}"/>
+      <limit lower="${radians(-350)}" upper="${radians(350)}" effort="0" velocity="${radians(615)}"/>
     </joint>
     <joint name="${prefix}joint_a6-flange" type="fixed">
@@ -170,5 +170,5 @@
       <parent link="${prefix}flange"/>
       <child link="${prefix}tool0"/>
-      <origin xyz="0 0 0" rpy="0 ${pi*0.5} 0"/>
+      <origin xyz="0 0 0" rpy="0 ${radians(90)} 0"/>
     </joint>
   </xacro:macro>

File: kuka_kr6_support/urdf/kr6r900sixx_macro.xacro (robot description, xacro)
@@ -116,5 +116,5 @@
       <child link="${prefix}link_1"/>
       <axis xyz="0 0 -1"/>
-      <limit effort="0" lower="${-DEG2RAD * 170}" upper="${DEG2RAD * 170}" velocity="${DEG2RAD * 360}"/>
+      <limit effort="0" lower="${-radians(170)}" upper="${radians(170)}" velocity="${radians(360)}"/>
     </joint>
     <joint name="${prefix}joint_a2" type="revolute">
@@ -123,5 +123,5 @@
       <child link="${prefix}link_2"/>
       <axis xyz="0 1 0"/>
-      <limit effort="0" lower="${-DEG2RAD * 190}" upper="${DEG2RAD * 45}" velocity="${DEG2RAD * 300}"/>
+      <limit effort="0" lower="${-radians(190)}" upper="${radians(45)}" velocity="${radians(300)}"/>
     </joint>
     <joint name="${prefix}joint_a3" type="revolute">
@@ -130,5 +130,5 @@
       <child link="${prefix}link_3"/>
       <axis xyz="0 1 0"/>
-      <limit effort="0" lower="${-DEG2RAD * 120}" upper="${DEG2RAD * 156}" velocity="${DEG2RAD * 360}"/>
+      <limit effort="0" lower="${-radians(120)}" upper="${radians(156)}" velocity="${radians(360)}"/>
     </joint>
     <joint name="${prefix}joint_a4" type="revolute">
@@ -137,5 +137,5 @@
       <child link="${prefix}link_4"/>
       <axis xyz="-1 0 0"/>
-      <limit effort="0" lower="${-DEG2RAD * 185}" upper="${DEG2RAD * 185}" velocity="${DEG2RAD * 381}"/>
+      <limit effort="0" lower="${-radians(185)}" upper="${radians(185)}" velocity="${radians(381)}"/>
     </joint>
     <joint name="${prefix}joint_a5" type="revolute">
@@ -144,5 +144,5 @@
       <child link="${prefix}link_5"/>
       <axis xyz="0 1 0"/>
-      <limit effort="0" lower="${-DEG2RAD * 120}" upper="${DEG2RAD * 120}" velocity="${DEG2RAD * 388}"/>
+      <limit effort="0" lower="${-radians(120)}" upper="${radians(120)}" velocity="${radians(388)}"/>
     </joint>
     <joint name="${prefix}joint_a6" type="revolute">
@@ -151,5 +151,5 @@
       <child link="${prefix}link_6"/>
       <axis xyz="-1 0 0"/>
-      <limit effort="0" lower="${-DEG2RAD * 350}" upper="${DEG2RAD * 350}" velocity="${DEG2RAD * 615}"/>
+      <limit effort="0" lower="${-radians(350)}" upper="${radians(350)}" velocity="${radians(615)}"/>
     </joint>
     <joint name="${prefix}joint_a6-flange" type="fixed">
@@ -170,5 +170,5 @@
       <parent link="${prefix}flange"/>
       <child link="${prefix}tool0"/>
-      <origin xyz="0 0 0" rpy="0 ${pi*0.5} 0"/>
+      <origin xyz="0 0 0" rpy="0 ${radians(90)} 0"/>
     </joint>
   </xacro:macro>

Commit message: Include a new link called flange to the available robot descriptions (#195)
* Following REP199, include a new link called flange to attach EEFs instead of the previous tool0

* Replace pi and DEG2RAD xacro properties with radians()

File: kuka_kr10_support/urdf/kr10r1100sixx_macro.xacro (robot description, xacro)
@@ -108,6 +108,6 @@
       </collision>
     </link>
-    <!-- This frame corresponds to the $FLANGE coordinate system in KUKA KRC controllers. -->
-    <link name="${prefix}tool0"/>
+    <!-- Following REP199, this frame shall be use to attach EEF or other equipment -->
+    <link name="${prefix}flange" />
     <joint name="${prefix}joint_a1" type="revolute">
       <origin xyz="0 0 0.400" rpy="0 0 0"/>
@@ -152,8 +152,8 @@
       <limit effort="0" lower="${radians(-350)}" upper="${radians(350)}" velocity="${radians(492)}"/>
     </joint>
-    <joint name="${prefix}joint_a6-tool0" type="fixed">
+    <joint name="${prefix}joint_a6-flange" type="fixed">
       <parent link="${prefix}link_6"/>
-      <child link="${prefix}tool0"/>
-      <origin xyz="0 0 0" rpy="0 ${radians(90)} 0"/>
+      <child link="${prefix}flange"/>
+      <origin xyz="0 0 0" rpy="0 0 0"/>
     </joint>
     <!-- ROS base_link to KUKA $ROBROOT coordinate system transform -->
@@ -164,4 +164,11 @@
       <child link="${prefix}base"/>
     </joint>
+    <!-- This frame corresponds to the $TOOL coordinate system in KUKA KRC controllers -->
+    <link name="${prefix}tool0" />
+    <joint name="${prefix}flange-tool0" type="fixed">
+      <parent link="${prefix}flange"/>
+      <child link="${prefix}tool0"/>
+      <origin xyz="0 0 0" rpy="0 ${radians(90)} 0"/>
+    </joint>
   </xacro:macro>
 </robot>

File: kuka_kr210_support/urdf/kr210l150_macro.xacro (robot description, xacro)
@@ -1,5 +1,4 @@
 <?xml version="1.0"?>
 <robot xmlns:xacro="http://wiki.ros.org/xacro">
-  <property name="pi" value="3.141592654"/>
   <xacro:macro name="kuka_kr210l150" params="prefix">
     <!-- links -->
@@ -11,5 +10,5 @@
       </inertial>
       <visual>
-        <origin xyz="0 0 0" rpy="${-pi/2} 0 0"/>
+        <origin xyz="0 0 0" rpy="${-radians(90)} 0 0"/>
         <geometry>
           <mesh filename="package://kuka_kr210_support/meshes/kr210l150/visual/base_link.dae"/>
@@ -20,5 +19,5 @@
       </visual>
       <collision>
-        <origin xyz="0 0 0" rpy="${-pi/2} 0 0"/>
+        <origin xyz="0 0 0" rpy="${-radians(90)} 0 0"/>
         <geometry>
           <mesh filename="package://kuka_kr210_support/meshes/kr210l150/collision/base_link.stl"/>
@@ -55,5 +54,5 @@
       </inertial>
       <visual>
-        <origin xyz="0 0 0" rpy="${-pi/2} 0 0"/>
+        <origin xyz="0 0 0" rpy="${-radians(90)} 0 0"/>
         <geometry>
           <mesh filename="package://kuka_kr210_support/meshes/kr210l150/visual/link_2.dae"/>
@@ -77,5 +76,5 @@
       </inertial>
       <visual>
-        <origin xyz="0 0 0" rpy="${-pi/2} 0 0"/>
+        <origin xyz="0 0 0" rpy="${-radians(90)} 0 0"/>
         <geometry>
           <mesh filename="package://kuka_kr210_support/meshes/kr210l150/visual/link_3.dae"/>
@@ -99,5 +98,5 @@
       </inertial>
       <visual>
-        <origin xyz="0 0 0" rpy="${-pi/2} 0 0"/>
+        <origin xyz="0 0 0" rpy="${-radians(90)} 0 0"/>
         <geometry>
           <mesh filename="package://kuka_kr210_support/meshes/kr210l150/visual/link_4.dae"/>
@@ -121,5 +120,5 @@
       </inertial>
       <visual>
-        <origin xyz="0 0 0" rpy="${-pi/2} 0 0"/>
+        <origin xyz="0 0 0" rpy="${-radians(90)} 0 0"/>
         <geometry>
           <mesh filename="package://kuka_kr210_support/meshes/kr210l150/visual/link_5.dae"/>
@@ -158,6 +157,6 @@
       </collision>
     </link>
-    <!-- This frame corresponds to the $FLANGE coordinate system in KUKA KRC controllers. -->
-    <link name="${prefix}tool0"/>
+    <!-- This frame corresponds to the $TOOL coordinate system in KUKA KRC controllers. -->
+    <link name="${prefix}flange"/>
     <!-- joints -->
     <joint name="${prefix}joint_a1" type="revolute">
@@ -180,5 +179,5 @@
       <child link="${prefix}link_3"/>
       <axis xyz="0 1 0"/>
-      <limit lower="${radians(-210)}" upper="${radians(155-90)}" effort="0" velocity="${radians(112)}"/>
+      <limit lower="${radians(-210)}" upper="${radians(65)}" effort="0" velocity="${radians(112)}"/>
     </joint>
     <joint name="${prefix}joint_a4" type="revolute">
@@ -203,8 +202,22 @@
       <limit lower="${radians(-350)}" upper="${radians(350)}" effort="0" velocity="${radians(219)}"/>
     </joint>
-    <joint name="${prefix}link_6-tool0" type="fixed">
+    <joint name="${prefix}link_6-flange" type="fixed">
       <parent link="${prefix}link_6"/>
+      <child link="${prefix}flange"/>
+      <origin xyz="0.0375 0 -0.00023924" rpy="0 0 0"/>
+    </joint>
+    <!-- ROS base_link to KUKA $ROBROOT coordinate system transform -->
+    <link name="${prefix}base" />
+    <joint name="${prefix}base_link-base" type="fixed">
+      <origin xyz="0 0 0" rpy="0 0 0"/>
+      <parent link="${prefix}base_link"/>
+      <child link="${prefix}base"/>
+    </joint>
+    <!-- This frame corresponds to the $TOOL coordinate system in KUKA KRC controllers -->
+    <link name="${prefix}tool0" />
+    <joint name="${prefix}flange-tool0" type="fixed">
+      <parent link="${prefix}flange"/>
       <child link="${prefix}tool0"/>
-      <origin xyz="0.0375 0 -0.00023924" rpy="0 0 0"/>
+      <origin xyz="0 0 0" rpy="0 ${radians(90)} 0"/>
     </joint>
     <!-- rename 'Link1' to 'link_1', maintain bw-compatibility -->
