Commit message: Add KR10 R1420 support (#216)

File: kuka_kr10_support/urdf/kr10r1420_macro.xacro (robot description, xacro)
@@ -1,5 +1,5 @@
 <?xml version="1.0"?>
 <robot xmlns:xacro="http://wiki.ros.org/xacro">
-  <xacro:macro name="kuka_kr10r1100sixx" params="prefix">
+  <xacro:macro name="kuka_kr10r1420" params="prefix">
     <xacro:include filename="$(find kuka_resources)/urdf/common_materials.xacro"/>
     <link name="${prefix}base_link">
@@ -7,5 +7,5 @@
         <origin xyz="0 0 0" rpy="0 0 0"/>
         <geometry>
-          <mesh filename="package://kuka_kr10_support/meshes/kr10r1100sixx/visual/base_link.stl" />
+          <mesh filename="package://kuka_kr10_support/meshes/kr10r1420/visual/base_link.stl" />
         </geometry>
         <xacro:material_kuka_black />
@@ -14,5 +14,5 @@
         <origin xyz="0 0 0" rpy="0 0 0"/>
         <geometry>
-          <mesh filename="package://kuka_kr10_support/meshes/kr10r1100sixx/collision/base_link.stl" />
+          <mesh filename="package://kuka_kr10_support/meshes/kr10r1420/collision/base_link.stl" />
         </geometry>
       </collision>
@@ -22,5 +22,5 @@
         <origin xyz="0 0 0" rpy="0 0 0"/>
         <geometry>
-          <mesh filename="package://kuka_kr10_support/meshes/kr10r1100sixx/visual/link_1.stl" />
+          <mesh filename="package://kuka_kr10_support/meshes/kr10r1420/visual/link_1.stl" />
         </geometry>
         <xacro:material_kuka_orange />
@@ -29,5 +29,5 @@
         <origin xyz="0 0 0" rpy="0 0 0"/>
         <geometry>
-          <mesh filename="package://kuka_kr10_support/meshes/kr10r1100sixx/collision/link_1.stl" />
+          <mesh filename="package://kuka_kr10_support/meshes/kr10r1420/collision/link_1.stl" />
         </geometry>
       </collision>
@@ -37,5 +37,5 @@
         <origin xyz="0 0 0" rpy="0 0 0"/>
         <geometry>
-          <mesh filename="package://kuka_kr10_support/meshes/kr10r1100sixx/visual/link_2.stl"/>
+          <mesh filename="package://kuka_kr10_support/meshes/kr10r1420/visual/link_2.stl"/>
         </geometry>
         <xacro:material_kuka_orange />
@@ -44,5 +44,5 @@
         <origin xyz="0 0 0" rpy="0 0 0"/>
         <geometry>
-          <mesh filename="package://kuka_kr10_support/meshes/kr10r1100sixx/collision/link_2.stl" />
+          <mesh filename="package://kuka_kr10_support/meshes/kr10r1420/collision/link_2.stl" />
         </geometry>
       </collision>
@@ -52,5 +52,5 @@
         <origin xyz="0 0 0" rpy="0 0 0"/>
         <geometry>
-          <mesh filename="package://kuka_kr10_support/meshes/kr10r1100sixx/visual/link_3.stl" />
+          <mesh filename="package://kuka_kr10_support/meshes/kr10r1420/visual/link_3.stl" />
         </geometry>
         <xacro:material_kuka_orange />
@@ -59,5 +59,5 @@
         <origin xyz="0 0 0" rpy="0 0 0"/>
         <geometry>
-          <mesh filename="package://kuka_kr10_support/meshes/kr10r1100sixx/collision/link_3.stl" />
+          <mesh filename="package://kuka_kr10_support/meshes/kr10r1420/collision/link_3.stl" />
         </geometry>
       </collision>
@@ -67,5 +67,5 @@
         <origin xyz="0 0 0" rpy="0 0 0"/>
         <geometry>
-          <mesh filename="package://kuka_kr10_support/meshes/kr10r1100sixx/visual/link_4.stl" />
+          <mesh filename="package://kuka_kr10_support/meshes/kr10r1420/visual/link_4.stl" />
         </geometry>
         <xacro:material_kuka_orange />
@@ -74,5 +74,5 @@
         <origin xyz="0 0 0" rpy="0 0 0"/>
         <geometry>
-          <mesh filename="package://kuka_kr10_support/meshes/kr10r1100sixx/collision/link_4.stl" />
+          <mesh filename="package://kuka_kr10_support/meshes/kr10r1420/collision/link_4.stl" />
         </geometry>
       </collision>
@@ -82,5 +82,5 @@
         <origin xyz="0 0 0" rpy="0 0 0"/>
         <geometry>
-          <mesh filename="package://kuka_kr10_support/meshes/kr10r1100sixx/visual/link_5.stl" />
+          <mesh filename="package://kuka_kr10_support/meshes/kr10r1420/visual/link_5.stl" />
         </geometry>
         <xacro:material_kuka_orange />
@@ -89,5 +89,5 @@
         <origin xyz="0 0 0" rpy="0 0 0"/>
         <geometry>
-          <mesh filename="package://kuka_kr10_support/meshes/kr10r1100sixx/collision/link_5.stl" />
+          <mesh filename="package://kuka_kr10_support/meshes/kr10r1420/collision/link_5.stl" />
         </geometry>
       </collision>
@@ -97,5 +97,5 @@
         <origin xyz="0 0 0" rpy="0 0 0"/>
         <geometry>
-          <mesh filename="package://kuka_kr10_support/meshes/kr10r1100sixx/visual/link_6.stl" />
+          <mesh filename="package://kuka_kr10_support/meshes/kr10r1420/visual/link_6.stl" />
         </geometry>
         <xacro:material_kuka_pedestal />
@@ -104,44 +104,44 @@
         <origin xyz="0 0 0" rpy="0 0 0"/>
         <geometry>
-          <mesh filename="package://kuka_kr10_support/meshes/kr10r1100sixx/collision/link_6.stl" />
+          <mesh filename="package://kuka_kr10_support/meshes/kr10r1420/collision/link_6.stl" />
         </geometry>
       </collision>
     </link>
-    <!-- This frame corresponds to the $FLANGE coordinate system in KUKA KRC controllers. -->
-    <link name="${prefix}tool0"/>
+    <!-- Following REP199, this frame shall be use to attach EEF or other equipment -->
+    <link name="${prefix}flange" />
     <joint name="${prefix}joint_a1" type="revolute">
-      <origin xyz="0 0 0.400" rpy="0 0 0"/>
+      <origin xyz="0 0 0.450" rpy="0 0 0"/>
       <parent link="${prefix}base_link"/>
       <child link="${prefix}link_1"/>
       <axis xyz="0 0 -1"/>
-      <limit effort="0" lower="${-DEG2RAD * 170}" upper="${DEG2RAD * 170}" velocity="${DEG2RAD * 360}"/>
+      <limit effort="0" lower="${radians(-170)}" upper="${radians(170)}" velocity="${radians(220)}"/>
     </joint>
     <joint name="${prefix}joint_a2" type="revolute">
-      <origin xyz="0.025 0 0" rpy="0 0 0"/>
+      <origin xyz="0.150 0 0" rpy="0 0 0"/>
       <parent link="${prefix}link_1"/>
       <child link="${prefix}link_2"/>
       <axis xyz="0 1 0"/>
-      <limit effort="0" lower="${-DEG2RAD * 190}" upper="${DEG2RAD * 45}" velocity="${DEG2RAD * 300}"/>
+      <limit effort="0" lower="${radians(-185)}" upper="${radians(65)}" velocity="${radians(210)}"/>
     </joint>
     <joint name="${prefix}joint_a3" type="revolute">
-      <origin xyz="0.560 0 0" rpy="0 0 0"/>
+      <origin xyz="0.610 0 0" rpy="0 0 0"/>
       <parent link="${prefix}link_2"/>
       <child link="${prefix}link_3"/>
       <axis xyz="0 1 0"/>
-      <limit effort="0" lower="${-DEG2RAD * 120}" upper="${DEG2RAD * 156}" velocity="${DEG2RAD * 360}"/>
+      <limit effort="0" lower="${radians(-137)}" upper="${radians(163)}" velocity="${radians(270)}"/>
     </joint>
     <joint name="${prefix}joint_a4" type="revolute">
-      <origin xyz="0 0 0.035" rpy="0 0 0"/>
+      <origin xyz="0 0 0.02" rpy="0 0 0"/>
       <parent link="${prefix}link_3"/>
       <child link="${prefix}link_4"/>
       <axis xyz="-1 0 0"/>
-      <limit effort="0" lower="${-DEG2RAD * 185}" upper="${DEG2RAD * 185}" velocity="${DEG2RAD * 381}"/>
+      <limit effort="0" lower="${radians(-185)}" upper="${radians(185)}" velocity="${radians(381)}"/>
     </joint>
     <joint name="${prefix}joint_a5" type="revolute">
-      <origin xyz="0.515 0 0" rpy="0 0 0"/>
+      <origin xyz="0.660 0 0" rpy="0 0 0"/>
       <parent link="${prefix}link_4"/>
       <child link="${prefix}link_5"/>
       <axis xyz="0 1 0"/>
-      <limit effort="0" lower="${-DEG2RAD * 120}" upper="${DEG2RAD * 120}" velocity="${DEG2RAD * 388}"/>
+      <limit effort="0" lower="${radians(-120)}" upper="${radians(120)}" velocity="${radians(311)}"/>
     </joint>
     <joint name="${prefix}joint_a6" type="revolute">
@@ -150,10 +150,10 @@
       <child link="${prefix}link_6"/>
       <axis xyz="-1 0 0"/>
-      <limit effort="0" lower="${-DEG2RAD * 350}" upper="${DEG2RAD * 350}" velocity="${DEG2RAD * 615}"/>
+      <limit effort="0" lower="${radians(-350)}" upper="${radians(350)}" velocity="${radians(492)}"/>
     </joint>
-    <joint name="${prefix}joint_a6-tool0" type="fixed">
+    <joint name="${prefix}joint_a6-flange" type="fixed">
       <parent link="${prefix}link_6"/>
-      <child link="${prefix}tool0"/>
-      <origin xyz="0 0 0" rpy="0 ${DEG2RAD * 90} 0"/>
+      <child link="${prefix}flange"/>
+      <origin xyz="0 0 0" rpy="0 0 0"/>
     </joint>
     <!-- ROS base_link to KUKA $ROBROOT coordinate system transform -->
@@ -164,4 +164,11 @@
       <child link="${prefix}base"/>
     </joint>
+    <!-- This frame corresponds to the $TOOL coordinate system in KUKA KRC controllers -->
+    <link name="${prefix}tool0" />
+    <joint name="${prefix}flange-tool0" type="fixed">
+      <parent link="${prefix}flange"/>
+      <child link="${prefix}tool0"/>
+      <origin xyz="0 0 0" rpy="0 ${radians(90)} 0"/>
+    </joint>
   </xacro:macro>
 </robot>

Commit message: Add KR10 R1420 support (#216)

File: kuka_kr10_support/urdf/kr10r1420_macro.xacro (robot description, xacro)
@@ -1,5 +1,5 @@
 <?xml version="1.0"?>
 <robot xmlns:xacro="http://wiki.ros.org/xacro">
-  <xacro:macro name="kuka_kr10r1100sixx" params="prefix">
+  <xacro:macro name="kuka_kr10r1420" params="prefix">
     <xacro:include filename="$(find kuka_resources)/urdf/common_materials.xacro"/>
     <link name="${prefix}base_link">
@@ -7,5 +7,5 @@
         <origin xyz="0 0 0" rpy="0 0 0"/>
         <geometry>
-          <mesh filename="package://kuka_kr10_support/meshes/kr10r1100sixx/visual/base_link.stl" />
+          <mesh filename="package://kuka_kr10_support/meshes/kr10r1420/visual/base_link.stl" />
         </geometry>
         <xacro:material_kuka_black />
@@ -14,5 +14,5 @@
         <origin xyz="0 0 0" rpy="0 0 0"/>
         <geometry>
-          <mesh filename="package://kuka_kr10_support/meshes/kr10r1100sixx/collision/base_link.stl" />
+          <mesh filename="package://kuka_kr10_support/meshes/kr10r1420/collision/base_link.stl" />
         </geometry>
       </collision>
@@ -22,5 +22,5 @@
         <origin xyz="0 0 0" rpy="0 0 0"/>
         <geometry>
-          <mesh filename="package://kuka_kr10_support/meshes/kr10r1100sixx/visual/link_1.stl" />
+          <mesh filename="package://kuka_kr10_support/meshes/kr10r1420/visual/link_1.stl" />
         </geometry>
         <xacro:material_kuka_orange />
@@ -29,5 +29,5 @@
         <origin xyz="0 0 0" rpy="0 0 0"/>
         <geometry>
-          <mesh filename="package://kuka_kr10_support/meshes/kr10r1100sixx/collision/link_1.stl" />
+          <mesh filename="package://kuka_kr10_support/meshes/kr10r1420/collision/link_1.stl" />
         </geometry>
       </collision>
@@ -37,5 +37,5 @@
         <origin xyz="0 0 0" rpy="0 0 0"/>
         <geometry>
-          <mesh filename="package://kuka_kr10_support/meshes/kr10r1100sixx/visual/link_2.stl"/>
+          <mesh filename="package://kuka_kr10_support/meshes/kr10r1420/visual/link_2.stl"/>
         </geometry>
         <xacro:material_kuka_orange />
@@ -44,5 +44,5 @@
         <origin xyz="0 0 0" rpy="0 0 0"/>
         <geometry>
-          <mesh filename="package://kuka_kr10_support/meshes/kr10r1100sixx/collision/link_2.stl" />
+          <mesh filename="package://kuka_kr10_support/meshes/kr10r1420/collision/link_2.stl" />
         </geometry>
       </collision>
@@ -52,5 +52,5 @@
         <origin xyz="0 0 0" rpy="0 0 0"/>
         <geometry>
-          <mesh filename="package://kuka_kr10_support/meshes/kr10r1100sixx/visual/link_3.stl" />
+          <mesh filename="package://kuka_kr10_support/meshes/kr10r1420/visual/link_3.stl" />
         </geometry>
         <xacro:material_kuka_orange />
@@ -59,5 +59,5 @@
         <origin xyz="0 0 0" rpy="0 0 0"/>
         <geometry>
-          <mesh filename="package://kuka_kr10_support/meshes/kr10r1100sixx/collision/link_3.stl" />
+          <mesh filename="package://kuka_kr10_support/meshes/kr10r1420/collision/link_3.stl" />
         </geometry>
       </collision>
@@ -67,5 +67,5 @@
         <origin xyz="0 0 0" rpy="0 0 0"/>
         <geometry>
-          <mesh filename="package://kuka_kr10_support/meshes/kr10r1100sixx/visual/link_4.stl" />
+          <mesh filename="package://kuka_kr10_support/meshes/kr10r1420/visual/link_4.stl" />
         </geometry>
         <xacro:material_kuka_orange />
@@ -74,5 +74,5 @@
         <origin xyz="0 0 0" rpy="0 0 0"/>
         <geometry>
-          <mesh filename="package://kuka_kr10_support/meshes/kr10r1100sixx/collision/link_4.stl" />
+          <mesh filename="package://kuka_kr10_support/meshes/kr10r1420/collision/link_4.stl" />
         </geometry>
       </collision>
@@ -82,5 +82,5 @@
         <origin xyz="0 0 0" rpy="0 0 0"/>
         <geometry>
-          <mesh filename="package://kuka_kr10_support/meshes/kr10r1100sixx/visual/link_5.stl" />
+          <mesh filename="package://kuka_kr10_support/meshes/kr10r1420/visual/link_5.stl" />
         </geometry>
         <xacro:material_kuka_orange />
@@ -89,5 +89,5 @@
         <origin xyz="0 0 0" rpy="0 0 0"/>
         <geometry>
-          <mesh filename="package://kuka_kr10_support/meshes/kr10r1100sixx/collision/link_5.stl" />
+          <mesh filename="package://kuka_kr10_support/meshes/kr10r1420/collision/link_5.stl" />
         </geometry>
       </collision>
@@ -97,5 +97,5 @@
         <origin xyz="0 0 0" rpy="0 0 0"/>
         <geometry>
-          <mesh filename="package://kuka_kr10_support/meshes/kr10r1100sixx/visual/link_6.stl" />
+          <mesh filename="package://kuka_kr10_support/meshes/kr10r1420/visual/link_6.stl" />
         </geometry>
         <xacro:material_kuka_pedestal />
@@ -104,5 +104,5 @@
         <origin xyz="0 0 0" rpy="0 0 0"/>
         <geometry>
-          <mesh filename="package://kuka_kr10_support/meshes/kr10r1100sixx/collision/link_6.stl" />
+          <mesh filename="package://kuka_kr10_support/meshes/kr10r1420/collision/link_6.stl" />
         </geometry>
       </collision>
@@ -111,26 +111,26 @@
     <link name="${prefix}flange" />
     <joint name="${prefix}joint_a1" type="revolute">
-      <origin xyz="0 0 0.400" rpy="0 0 0"/>
+      <origin xyz="0 0 0.450" rpy="0 0 0"/>
       <parent link="${prefix}base_link"/>
       <child link="${prefix}link_1"/>
       <axis xyz="0 0 -1"/>
-      <limit effort="0" lower="${radians(-170)}" upper="${radians(170)}" velocity="${radians(300)}"/>
+      <limit effort="0" lower="${radians(-170)}" upper="${radians(170)}" velocity="${radians(220)}"/>
     </joint>
     <joint name="${prefix}joint_a2" type="revolute">
-      <origin xyz="0.025 0 0" rpy="0 0 0"/>
+      <origin xyz="0.150 0 0" rpy="0 0 0"/>
       <parent link="${prefix}link_1"/>
       <child link="${prefix}link_2"/>
       <axis xyz="0 1 0"/>
-      <limit effort="0" lower="${radians(-190)}" upper="${radians(45)}" velocity="${radians(225)}"/>
+      <limit effort="0" lower="${radians(-185)}" upper="${radians(65)}" velocity="${radians(210)}"/>
     </joint>
     <joint name="${prefix}joint_a3" type="revolute">
-      <origin xyz="0.560 0 0" rpy="0 0 0"/>
+      <origin xyz="0.610 0 0" rpy="0 0 0"/>
       <parent link="${prefix}link_2"/>
       <child link="${prefix}link_3"/>
       <axis xyz="0 1 0"/>
-      <limit effort="0" lower="${radians(-120)}" upper="${radians(156)}" velocity="${radians(225)}"/>
+      <limit effort="0" lower="${radians(-137)}" upper="${radians(163)}" velocity="${radians(270)}"/>
     </joint>
     <joint name="${prefix}joint_a4" type="revolute">
-      <origin xyz="0 0 0.035" rpy="0 0 0"/>
+      <origin xyz="0 0 0.02" rpy="0 0 0"/>
       <parent link="${prefix}link_3"/>
       <child link="${prefix}link_4"/>
@@ -139,5 +139,5 @@
     </joint>
     <joint name="${prefix}joint_a5" type="revolute">
-      <origin xyz="0.515 0 0" rpy="0 0 0"/>
+      <origin xyz="0.660 0 0" rpy="0 0 0"/>
       <parent link="${prefix}link_4"/>
       <child link="${prefix}link_5"/>
