Commit message: KUKA_DEG2RAD replaced with radians function see #79

File: kuka_kr16_support/urdf/kr16_2_macro.xacro (robot description, xacro)
@@ -1,5 +1,4 @@
 <?xml version="1.0"?>
 <robot xmlns:xacro="http://www.ros.org/wiki/xacro">
-  <xacro:property name="KUKA_DEG2RAD" value="0.017453292519943295"/>
   <xacro:macro name="kuka_kr16_2" params="prefix">
     <!-- LINKS -->
@@ -155,5 +154,5 @@
       <child link="${prefix}link_1"/>
       <axis xyz="0 0 -1"/>
-      <limit effort="0" lower="${-KUKA_DEG2RAD * 185}" upper="${KUKA_DEG2RAD * 185}" velocity="${KUKA_DEG2RAD * 156}"/>
+      <limit effort="0" lower="${radians(-185)}" upper="${radians(185)}" velocity="${radians(156)}"/>
     </joint>
     <!-- joint 2 (A2) -->
@@ -163,5 +162,5 @@
       <child link="${prefix}link_2"/>
       <axis xyz="0 1 0"/>
-      <limit effort="0" lower="${-KUKA_DEG2RAD * 155}" upper="${KUKA_DEG2RAD * 35}" velocity="${KUKA_DEG2RAD * 156}"/>
+      <limit effort="0" lower="${radians(-155)}" upper="${radians(35)}" velocity="${radians(156)}"/>
     </joint>
     <!-- joint 3 (A3) -->
@@ -171,5 +170,5 @@
       <child link="${prefix}link_3"/>
       <axis xyz="0 1 0"/>
-      <limit effort="0" lower="${-KUKA_DEG2RAD * 130}" upper="${KUKA_DEG2RAD * 154}" velocity="${KUKA_DEG2RAD * 156}"/>
+      <limit effort="0" lower="${radians(-130)}" upper="${radians(154)}" velocity="${radians(156)}"/>
     </joint>
     <!-- joint 4 (A4) -->
@@ -179,5 +178,5 @@
       <child link="${prefix}link_4"/>
       <axis xyz="-1 0 0"/>
-      <limit effort="0" lower="${-KUKA_DEG2RAD * 350}" upper="${KUKA_DEG2RAD * 350}" velocity="${KUKA_DEG2RAD * 330}"/>
+      <limit effort="0" lower="${radians(-350)}" upper="${radians(350)}" velocity="${radians(330)}"/>
     </joint>
     <!-- joint 5 (A5) -->
@@ -187,5 +186,5 @@
       <child link="${prefix}link_5"/>
       <axis xyz="0 1 0"/>
-      <limit effort="0" lower="${-KUKA_DEG2RAD * 130}" upper="${KUKA_DEG2RAD * 130}" velocity="${KUKA_DEG2RAD * 330}"/>
+      <limit effort="0" lower="${radians(-130)}" upper="${radians(130)}" velocity="${radians(330)}"/>
     </joint>
     <!-- joint 6 (A6) -->
@@ -195,5 +194,5 @@
       <child link="${prefix}link_6"/>
       <axis xyz="-1 0 0"/>
-      <limit effort="0" lower="${-KUKA_DEG2RAD * 350}" upper="${KUKA_DEG2RAD * 350}" velocity="${KUKA_DEG2RAD * 615}"/>
+      <limit effort="0" lower="${radians(-350)}" upper="${radians(350)}" velocity="${radians(615)}"/>
     </joint>
     <!-- tool frame - fixed frame -->
@@ -201,5 +200,5 @@
       <parent link="${prefix}link_6"/>
       <child link="${prefix}tool0"/>
-      <origin xyz="0.158 0 0" rpy="0 ${KUKA_DEG2RAD * 90} 0"/>
+      <origin xyz="0.158 0 0" rpy="0 ${radians(90)} 0"/>
     </joint>
     <!-- END JOINTS -->
