Commit message: Changed the colour and collision model of the KR16 Original

File: kuka_kr16_support/urdf/kr16.urdf (robot description, URDF)
Before this commit: robot kuka_kr16, 9 links, 8 joints
Links:
- link link_2: geometry collision mesh filename=package://kuka_kr16_support/meshes/kr16/collision/link_2.stl; visual mesh filename=package://kuka_kr16_support/meshes/kr16/visual/link_2.stl
- link link_4: geometry collision mesh filename=package://kuka_kr16_support/meshes/kr16/collision/link_4.stl; visual mesh filename=package://kuka_kr16_support/meshes/kr16/visual/link_4.stl

File: kuka_kr16_support/urdf/kr16.xacro (robot description, xacro)
@@ -1,4 +1,4 @@
 <?xml version="1.0"?>
-<!--Generates a urdf from the macro in kr16_2_macro.xacro -->
+<!--Generates a urdf from the macro in kr16_macro.xacro -->
 <robot name="kuka_kr16" xmlns:xacro="http://wiki.ros.org/xacro">
   <xacro:include filename="$(find kuka_kr16_support)/urdf/kr16_macro.xacro" />

File: kuka_kr16_support/urdf/kr16_macro.xacro (robot description, xacro)
@@ -1,4 +1,6 @@
 <?xml version="1.0"?>
 <robot xmlns:xacro="http://wiki.ros.org/xacro">
+  <xacro:include filename="$(find kuka_resources)/urdf/common_constants.xacro"/>
+  <xacro:include filename="$(find kuka_resources)/urdf/common_materials.xacro"/>
   <xacro:macro name="kuka_kr16" params="prefix">
     <!-- LINKS -->
@@ -15,4 +17,5 @@
           <mesh filename="package://kuka_kr16_support/meshes/kr16/visual/base_link.stl" />
         </geometry>
+        <xacro:material_kuka_pedestal />
       </visual>
       <collision>
@@ -35,4 +38,5 @@
           <mesh filename="package://kuka_kr16_support/meshes/kr16/visual/link_1.stl" />
         </geometry>
+        <xacro:material_kuka_orange />
       </visual>
       <collision>
@@ -55,4 +59,5 @@
           <mesh filename="package://kuka_kr16_support/meshes/kr16/visual/link_2.stl"/>
         </geometry>
+        <xacro:material_kuka_orange />
       </visual>
       <collision>
@@ -75,4 +80,5 @@
           <mesh filename="package://kuka_kr16_support/meshes/kr16/visual/link_3.stl" />
         </geometry>
+        <xacro:material_kuka_orange />
       </visual>
       <collision>
@@ -95,4 +101,5 @@
           <mesh filename="package://kuka_kr16_support/meshes/kr16/visual/link_4.stl" />
         </geometry>
+        <xacro:material_kuka_orange />
       </visual>
       <collision>
@@ -115,4 +122,5 @@
           <mesh filename="package://kuka_kr16_support/meshes/kr16/visual/link_5.stl" />
         </geometry>
+        <xacro:material_kuka_orange />
       </visual>
       <collision>
@@ -135,4 +143,5 @@
           <mesh filename="package://kuka_kr16_support/meshes/kr16/visual/link_6.stl" />
         </geometry>
+        <xacro:material_kuka_pedestal />
       </visual>
       <collision>
