Commit message: move KR 16 R1610 cybertech to kuka_kr16_support

File: kuka_kr16_support/urdf/kr16r1610cybertech_macro.xacro (robot description, xacro)
@@ -1,5 +1,5 @@
 <?xml version="1.0"?>
 <robot xmlns:xacro="http://wiki.ros.org/xacro">
-  <xacro:macro name="kuka_kr16_r1610" params="prefix">
+  <xacro:macro name="kuka_kr16r1610cybertech" params="prefix">
     <!-- LINKS -->
     <!-- base link -->
@@ -13,11 +13,11 @@
         <origin xyz="0 0 0" rpy="0 0 0"/>
         <geometry>
-          <mesh filename="package://kuka_cybertech_kr16_r1610_support/meshes/kr16_r1610/visual/base_link.dae" />
-        </geometry>
-      </visual>
-      <collision>
-        <origin xyz="0 0 0" rpy="0 0 0"/>
-        <geometry>
-          <mesh filename="package://kuka_cybertech_kr16_r1610_support/meshes/kr16_r1610/collision/base_link.stl" />
+          <mesh filename="package://kuka_kr16_support/meshes/kr16r1610cybertech/visual/base_link.dae" />
+        </geometry>
+      </visual>
+      <collision>
+        <origin xyz="0 0 0" rpy="0 0 0"/>
+        <geometry>
+          <mesh filename="package://kuka_kr16_support/meshes/kr16r1610cybertech/collision/base_link.stl" />
         </geometry>
       </collision>
@@ -33,11 +33,11 @@
         <origin xyz="0 0 0" rpy="0 0 0"/>
         <geometry>
-          <mesh filename="package://kuka_cybertech_kr16_r1610_support/meshes/kr16_r1610/visual/link_1.dae" />
-        </geometry>
-      </visual>
-      <collision>
-        <origin xyz="0 0 0" rpy="0 0 0"/>
-        <geometry>
-          <mesh filename="package://kuka_cybertech_kr16_r1610_support/meshes/kr16_r1610/collision/link_1.stl" />
+          <mesh filename="package://kuka_kr16_support/meshes/kr16r1610cybertech/visual/link_1.dae" />
+        </geometry>
+      </visual>
+      <collision>
+        <origin xyz="0 0 0" rpy="0 0 0"/>
+        <geometry>
+          <mesh filename="package://kuka_kr16_support/meshes/kr16r1610cybertech/collision/link_1.stl" />
         </geometry>
       </collision>
@@ -53,11 +53,11 @@
         <origin xyz="0 0 0" rpy="0 0 0"/>
         <geometry>
-          <mesh filename="package://kuka_cybertech_kr16_r1610_support/meshes/kr16_r1610/visual/link_2.dae"/>
-        </geometry>
-      </visual>
-      <collision>
-        <origin xyz="0 0 0" rpy="0 0 0"/>
-        <geometry>
-          <mesh filename="package://kuka_cybertech_kr16_r1610_support/meshes/kr16_r1610/collision/link_2.stl" />
+          <mesh filename="package://kuka_kr16_support/meshes/kr16r1610cybertech/visual/link_2.dae"/>
+        </geometry>
+      </visual>
+      <collision>
+        <origin xyz="0 0 0" rpy="0 0 0"/>
+        <geometry>
+          <mesh filename="package://kuka_kr16_support/meshes/kr16r1610cybertech/collision/link_2.stl" />
         </geometry>
       </collision>
@@ -73,11 +73,11 @@
         <origin xyz="0 0 0" rpy="0 0 0"/>
         <geometry>
-          <mesh filename="package://kuka_cybertech_kr16_r1610_support/meshes/kr16_r1610/visual/link_3.dae" />
-        </geometry>
-      </visual>
-      <collision>
-        <origin xyz="0 0 0" rpy="0 0 0"/>
-        <geometry>
-          <mesh filename="package://kuka_cybertech_kr16_r1610_support/meshes/kr16_r1610/collision/link_3.stl" />
+          <mesh filename="package://kuka_kr16_support/meshes/kr16r1610cybertech/visual/link_3.dae" />
+        </geometry>
+      </visual>
+      <collision>
+        <origin xyz="0 0 0" rpy="0 0 0"/>
+        <geometry>
+          <mesh filename="package://kuka_kr16_support/meshes/kr16r1610cybertech/collision/link_3.stl" />
         </geometry>
       </collision>
@@ -93,11 +93,11 @@
         <origin xyz="0 0 0" rpy="0 0 0"/>
         <geometry>
-          <mesh filename="package://kuka_cybertech_kr16_r1610_support/meshes/kr16_r1610/visual/link_4.dae" />
-        </geometry>
-      </visual>
-      <collision>
-        <origin xyz="0 0 0" rpy="0 0 0"/>
-        <geometry>
-          <mesh filename="package://kuka_cybertech_kr16_r1610_support/meshes/kr16_r1610/collision/link_4.stl" />
+          <mesh filename="package://kuka_kr16_support/meshes/kr16r1610cybertech/visual/link_4.dae" />
+        </geometry>
+      </visual>
+      <collision>
+        <origin xyz="0 0 0" rpy="0 0 0"/>
+        <geometry>
+          <mesh filename="package://kuka_kr16_support/meshes/kr16r1610cybertech/collision/link_4.stl" />
         </geometry>
       </collision>
@@ -113,11 +113,11 @@
         <origin xyz="0 0 0" rpy="0 0 0"/>
         <geometry>
-          <mesh filename="package://kuka_cybertech_kr16_r1610_support/meshes/kr16_r1610/visual/link_5.dae" />
-        </geometry>
-      </visual>
-      <collision>
-        <origin xyz="0 0 0" rpy="0 0 0"/>
-        <geometry>
-          <mesh filename="package://kuka_cybertech_kr16_r1610_support/meshes/kr16_r1610/collision/link_5.stl" />
+          <mesh filename="package://kuka_kr16_support/meshes/kr16r1610cybertech/visual/link_5.dae" />
+        </geometry>
+      </visual>
+      <collision>
+        <origin xyz="0 0 0" rpy="0 0 0"/>
+        <geometry>
+          <mesh filename="package://kuka_kr16_support/meshes/kr16r1610cybertech/collision/link_5.stl" />
         </geometry>
       </collision>
@@ -133,11 +133,11 @@
         <origin xyz="0 0 0" rpy="0 0 0"/>
         <geometry>
-          <mesh filename="package://kuka_cybertech_kr16_r1610_support/meshes/kr16_r1610/visual/link_6.dae" />
-        </geometry>
-      </visual>
-      <collision>
-        <origin xyz="0 0 0" rpy="0 0 0"/>
-        <geometry>
-          <mesh filename="package://kuka_cybertech_kr16_r1610_support/meshes/kr16_r1610/collision/link_6.stl" />
+          <mesh filename="package://kuka_kr16_support/meshes/kr16r1610cybertech/visual/link_6.dae" />
+        </geometry>
+      </visual>
+      <collision>
+        <origin xyz="0 0 0" rpy="0 0 0"/>
+        <geometry>
+          <mesh filename="package://kuka_kr16_support/meshes/kr16r1610cybertech/collision/link_6.stl" />
         </geometry>
       </collision>

Commit message: Update XACRO to include flange

File: kuka_kr16_support/urdf/kr16r1610cybertech_macro.xacro (robot description, xacro)
@@ -143,7 +143,4 @@
       </collision>
     </link>
-    <!-- tool 0 -->
-    <!-- This frame corresponds to the $FLANGE coordinate system in KUKA KRC controllers. -->
-    <link name="${prefix}tool0"/>
     <!-- END LINKS -->
     <!-- JOINTS -->
@@ -196,12 +193,6 @@
       <limit effort="0" lower="${radians(-350)}" upper="${radians(350)}" velocity="${radians(630)}"/>
     </joint>
-    <!-- tool frame - fixed frame -->
-    <joint name="${prefix}joint_a6-tool0" type="fixed">
-      <parent link="${prefix}link_6"/>
-      <child link="${prefix}tool0"/>
-      <origin xyz="0.153 0 0" rpy="0 ${radians(90)} 0"/>
-    </joint>
     <!-- END JOINTS -->
-    <!-- ROS base_link to KUKA $ROBROOT coordinate system transform -->
+    <!-- ROS-Industrial 'base' frame: base_link to KUKA $ROBROOT coordinate system transform -->
     <link name="${prefix}base" />
     <joint name="${prefix}base_link-base" type="fixed">
@@ -210,4 +201,19 @@
       <child link="${prefix}base"/>
     </joint>
+    <!-- ROS-Industrial 'flange' frame: attachment point for EEF models -->
+    <link name="${prefix}flange" />
+    <joint name="${prefix}joint_6-flange" type="fixed">
+      <origin xyz="0.153 0 0" rpy="0 0 0" />
+      <parent link="${prefix}link_6" />
+      <child link="${prefix}flange" />
+    </joint>
+    <!-- ROS-Industrial 'tool0' frame: all-zeros tool frame -->
+    <!-- This frame corresponds to the $FLANGE coordinate system in KUKA KRC controllers. -->
+    <link name="${prefix}tool0"/>
+    <joint name="${prefix}flange-tool0" type="fixed">
+      <parent link="${prefix}flange"/>
+      <child link="${prefix}tool0"/>
+      <origin xyz="0 0 0" rpy="0 ${radians(90)} 0"/>
+    </joint>
   </xacro:macro>
 </robot>

Commit message: Remove dummy inertial and comments

File: kuka_kr16_support/urdf/kr16r1610cybertech_macro.xacro (robot description, xacro)
@@ -2,12 +2,5 @@
 <robot xmlns:xacro="http://wiki.ros.org/xacro">
   <xacro:macro name="kuka_kr16r1610cybertech" params="prefix">
-    <!-- LINKS -->
-    <!-- base link -->
     <link name="${prefix}base_link">
-      <inertial>
-        <origin xyz="0 0 0" rpy="0 0 0"/>
-        <mass value="2"/>
-        <inertia ixx="0.01" ixy="0" ixz="0" iyy="0.01" iyz="0" izz="0.01" />
-      </inertial>
       <visual>
         <origin xyz="0 0 0" rpy="0 0 0"/>
@@ -23,11 +16,5 @@
       </collision>
     </link>
-    <!-- link 1 (A1) -->
     <link name="${prefix}link_1">
-      <inertial>
-        <origin xyz="0 0 0" rpy="0 0 0"/>
-        <mass value="2"/>
-        <inertia ixx="0.01" ixy="0" ixz="0" iyy="0.01" iyz="0" izz="0.01" />
-      </inertial>
       <visual>
         <origin xyz="0 0 0" rpy="0 0 0"/>
@@ -43,11 +30,5 @@
       </collision>
     </link>
-    <!-- link 2 -->
     <link name="${prefix}link_2">
-      <inertial>
-        <origin xyz="0 0 0" rpy="0 0 0"/>
-        <mass value="2"/>
-        <inertia ixx="0.01" ixy="0" ixz="0" iyy="0.01" iyz="0" izz="0.01" />
-      </inertial>
       <visual>
         <origin xyz="0 0 0" rpy="0 0 0"/>
@@ -63,11 +44,5 @@
       </collision>
     </link>
-    <!-- link 3 -->
     <link name="${prefix}link_3">
-      <inertial>
-        <origin xyz="0 0 0" rpy="0 0 0"/>
-        <mass value="2"/>
-        <inertia ixx="0.01" ixy="0" ixz="0" iyy="0.01" iyz="0" izz="0.01" />
-      </inertial>
       <visual>
         <origin xyz="0 0 0" rpy="0 0 0"/>
@@ -83,11 +58,5 @@
       </collision>
     </link>
-    <!-- link 4 -->
     <link name="${prefix}link_4">
-      <inertial>
-        <origin xyz="0 0 0" rpy="0 0 0"/>
-        <mass value="2"/>
-        <inertia ixx="0.01" ixy="0" ixz="0" iyy="0.01" iyz="0" izz="0.01" />
-      </inertial>
       <visual>
         <origin xyz="0 0 0" rpy="0 0 0"/>
@@ -103,11 +72,5 @@
       </collision>
     </link>
-    <!-- link 5 -->
     <link name="${prefix}link_5">
-      <inertial>
-        <origin xyz="0 0 0" rpy="0 0 0"/>
-        <mass value="2"/>
-        <inertia ixx="0.01" ixy="0" ixz="0" iyy="0.01" iyz="0" izz="0.01" />
-      </inertial>
       <visual>
         <origin xyz="0 0 0" rpy="0 0 0"/>
@@ -123,11 +86,5 @@
       </collision>
     </link>
-    <!-- link 6 -->
     <link name="${prefix}link_6">
-      <inertial>
-        <origin xyz="0 0 0" rpy="0 0 0"/>
-        <mass value="2"/>
-        <inertia ixx="0.01" ixy="0" ixz="0" iyy="0.01" iyz="0" izz="0.01" />
-      </inertial>
       <visual>
         <origin xyz="0 0 0" rpy="0 0 0"/>
@@ -143,7 +100,4 @@
       </collision>
     </link>
-    <!-- END LINKS -->
-    <!-- JOINTS -->
-    <!-- joint 1 (A1) -->
     <joint name="${prefix}joint_a1" type="revolute">
       <origin xyz="0 0 0.520" rpy="0 0 0"/>
@@ -153,5 +107,4 @@
       <limit effort="0" lower="${radians(-185)}" upper="${radians(185)}" velocity="${radians(200)}"/>
     </joint>
-    <!-- joint 2 (A2) -->
     <joint name="${prefix}joint_a2" type="revolute">
       <origin xyz="0.160 0 0" rpy="0 0 0"/>
@@ -161,5 +114,4 @@
       <limit effort="0" lower="${radians(-185)}" upper="${radians(65)}" velocity="${radians(175)}"/>
     </joint>
-    <!-- joint 3 (A3) -->
     <joint name="${prefix}joint_a3" type="revolute">
       <origin xyz="0.78 0 0" rpy="0 0 0"/>
@@ -169,5 +121,4 @@
       <limit effort="0" lower="${radians(-138)}" upper="${radians(175)}" velocity="${radians(190)}"/>
     </joint>
-    <!-- joint 4 (A4) -->
     <joint name="${prefix}joint_a4" type="revolute">
       <origin xyz="0.655 0 0.15" rpy="0 0 0"/>
@@ -177,5 +128,4 @@
       <limit effort="0" lower="${radians(-350)}" upper="${radians(350)}" velocity="${radians(430)}"/>
     </joint>
-    <!-- joint 5 (A5) -->
     <joint name="${prefix}joint_a5" type="revolute">
       <origin xyz="0 0 0" rpy="0 0 0"/>
@@ -185,5 +135,4 @@
       <limit effort="0" lower="${radians(-130)}" upper="${radians(130)}" velocity="${radians(430)}"/>
     </joint>
-    <!-- joint 6 (A6) -->
     <joint name="${prefix}joint_a6" type="revolute">
       <origin xyz="0 0 0" rpy="0 0 0"/>
@@ -193,5 +142,4 @@
       <limit effort="0" lower="${radians(-350)}" upper="${radians(350)}" velocity="${radians(630)}"/>
     </joint>
-    <!-- END JOINTS -->
     <!-- ROS-Industrial 'base' frame: base_link to KUKA $ROBROOT coordinate system transform -->
     <link name="${prefix}base" />

Commit message: Move offset from flange to joint_a6

File: kuka_kr16_support/urdf/kr16r1610cybertech_macro.xacro (robot description, xacro)
@@ -136,5 +136,5 @@
     </joint>
     <joint name="${prefix}joint_a6" type="revolute">
-      <origin xyz="0 0 0" rpy="0 0 0"/>
+      <origin xyz="0.153 0 0" rpy="0 0 0"/>
       <parent link="${prefix}link_5"/>
       <child link="${prefix}link_6"/>
@@ -152,5 +152,5 @@
     <link name="${prefix}flange" />
     <joint name="${prefix}joint_6-flange" type="fixed">
-      <origin xyz="0.153 0 0" rpy="0 0 0" />
+      <origin xyz="0 0 0" rpy="0 0 0" />
       <parent link="${prefix}link_6" />
       <child link="${prefix}flange" />
