Commit message: Removed dependecy to schunk_description

File: kuka_kr5_support/urdf/kr5_arc.xacro (robot description, xacro)
@@ -2,5 +2,4 @@
 <!--Generates a urdf from the macro in kr16_2_macro.xacro -->
 <robot name="kuka_kr5_arc" xmlns:xacro="http://www.ros.org/wiki/xacro">
-    <xacro:include filename="$(find schunk_description)/urdf/common.xacro" />
   <link name="world"/>
   <xacro:include filename="$(find kuka_kr5_support)/urdf/kr5_arc_macro.xacro" />

File: kuka_kr5_support/urdf/kr5_arc_macro.xacro (robot description, xacro)
@@ -1,4 +1,5 @@
 <?xml version="1.0"?>
 <robot xmlns:xacro="http://www.ros.org/wiki/xacro">
+  <xacro:property name="M_PI" value="3.1415926535897931" />
   <xacro:property name="KUKA_DEG2RAD" value="0.017453292519943295"/>
   <xacro:macro name="kuka_kr5_arc" params="prefix parent *origin has_podest">
@@ -11,5 +12,9 @@
       </joint>
       <link name="${prefix}podest_link">
-        <xacro:default_inertial/>
+        <inertial>
+          <mass value="0.01" />
+          <origin xyz="0 0 0" />
+          <inertia ixx="0.001" ixy="0.0" ixz="0.0" iyy="0.001" iyz="0.0" izz="0.001" />
+        </inertial>
         <visual>
             <origin rpy="0 0 0" xyz="0 0 0"/>

Commit message: Podest remove and file restructured. Removed test folder since whole launch folder can be tested.

File: kuka_kr5_support/urdf/kr5_arc.xacro (robot description, xacro)
@@ -2,8 +2,5 @@
 <!--Generates a urdf from the macro in kr16_2_macro.xacro -->
 <robot name="kuka_kr5_arc" xmlns:xacro="http://www.ros.org/wiki/xacro">
-  <link name="world"/>
   <xacro:include filename="$(find kuka_kr5_support)/urdf/kr5_arc_macro.xacro" />
-  <xacro:kuka_kr5_arc prefix="" parent="world" has_podest="true">
-      <origin xyz="0 0 0" rpy="0 0 0" />
-  </xacro:kuka_kr5_arc>
+  <xacro:kuka_kr5_arc prefix=""/>
 </robot>

File: kuka_kr5_support/urdf/kr5_arc_macro.xacro (robot description, xacro)
@@ -1,53 +1,5 @@
 <?xml version="1.0"?>
 <robot xmlns:xacro="http://www.ros.org/wiki/xacro">
-  <xacro:property name="pi" value="3.1415926535897931" />
-  <xacro:property name="KUKA_DEG2RAD" value="0.017453292519943295"/>
-  <xacro:macro name="kuka_kr5_arc" params="prefix parent *origin has_podest">
-<xacro:if value="${has_podest}">
-      <!-- joint between base_link and lwa4p_extended_connector_link -->
-      <joint name="${prefix}joint_podest" type="fixed">
-        <xacro:insert_block name="origin" />
-        <parent link="${parent}"/>
-        <child link="${prefix}podest_link"/>
-      </joint>
-      <link name="${prefix}podest_link">
-        <inertial>
-          <mass value="0.01" />
-          <origin xyz="0 0 0" />
-          <inertia ixx="0.001" ixy="0.0" ixz="0.0" iyy="0.001" iyz="0.0" izz="0.001" />
-        </inertial>
-        <visual>
-            <origin rpy="0 0 0" xyz="0 0 0"/>
-            <geometry>
-            <mesh filename="package://kuka_kr5_support/meshes/kr5_arc/visual/podest_link.dae" />
-            </geometry>
-        </visual>
-        <collision>
-            <origin rpy="0 0 0" xyz="0 0 0"/>
-            <geometry>
-            <mesh filename="package://kuka_kr5_support/meshes/kr5_arc/collision/podest_link.stl" scale="0.001 0.001 0.001" />
-            </geometry>
-        </collision>
-      </link>
-      <joint name="${prefix}base_joint" type="fixed">
-        <origin xyz="0 0 0.441" rpy="0 0 0" />
-        <parent link="${prefix}podest_link"/>
-        <child link="${prefix}base_link"/>
-      </joint>
-    </xacro:if>
-    <xacro:unless value="${has_podest}">
-      <joint name="${prefix}base_joint" type="fixed">
-        <xacro:insert_block name="origin" />
-        <parent link="${parent}"/>
-        <child link="${prefix}base_link"/>
-      </joint>
-    </xacro:unless>
-    <link name="${prefix}base" />
-    <!-- TODO: Check this with robots controller (c.f. http://wiki.ros.org/Industrial/Tutorials/Create%20a%20URDF%20for%20an%20Industrial%20Robot#Additional.2BAC8-Standard_Frames) -->
-    <joint name="${prefix}base_link-base" type="fixed">
-      <parent link="${prefix}base_link" />
-      <child link="${prefix}base" />
-      <origin xyz="0 0 0" rpy="0 0 0" />
-    </joint>
+  <xacro:macro name="kuka_kr5_arc" params="prefix">
     <!-- LINKS -->
     <!-- base link -->
@@ -254,5 +206,5 @@
     <!-- tool link -->
     <!-- This frame corresponds to the $FLANGE coordinate system in KUKA KRC controllers. -->
-    <link name="${prefix}tool_link"/>
+    <link name="${prefix}tool0"/>
     <!-- END LINKS -->
     <!-- JOINTS -->
@@ -287,5 +239,5 @@
       <child link="${prefix}link_4"/>
       <axis xyz="0 0 1"/>
-      <limit effort="0" lower="${radians(350)}" upper="${radians(350)}" velocity="${radians(343)}"/>
+      <limit effort="0" lower="${radians(-350)}" upper="${radians(350)}" velocity="${radians(343)}"/>
     </joint>
     <!-- joint 5 (A5) -->
@@ -312,4 +264,11 @@
     </joint>
     <!-- END JOINTS -->
+    <!-- ROS base_link to KUKA $ROBROOT coordinate system transform -->
+    <link name="${prefix}base" />
+    <joint name="${prefix}base_link-base" type="fixed">
+      <origin xyz="0 0 0" rpy="0 0 0" />
+      <parent link="${prefix}base_link" />
+      <child link="${prefix}base" />
+    </joint>
   </xacro:macro>
 </robot>

Commit message: Fixed accoring to comments

File: kuka_kr5_support/urdf/kr5_arc.xacro (robot description, xacro)
@@ -1,4 +1,3 @@
 <?xml version="1.0"?>
-<!--Generates a urdf from the macro in kr16_2_macro.xacro -->
 <robot name="kuka_kr5_arc" xmlns:xacro="http://www.ros.org/wiki/xacro">
   <xacro:include filename="$(find kuka_kr5_support)/urdf/kr5_arc_macro.xacro" />

File: kuka_kr5_support/urdf/kr5_arc_macro.xacro (robot description, xacro)
@@ -33,19 +33,19 @@
     <link name="${prefix}link_1">
       <inertial>
-      <origin
-        xyz="0.0359968408135882 0.00783796591813503 -0.0864969937502713"
-        rpy="0 0 0" />
-      <mass
-        value="5.77242340173648" />
-      <inertia
-        ixx="0.0327019582662897"
-        ixy="-0.00189987845379704"
-        ixz="0.00937014136132958"
-        iyy="0.0373787564144547"
-        iyz="-0.00197023031658988"
-        izz="0.0348614383349291" />
-    </inertial>
-      <visual>
-        <origin xyz="0 0 0" rpy="0  0 0"/>
+        <origin
+          xyz="0.0359968408135882 0.00783796591813503 -0.0864969937502713"
+          rpy="0 0 0" />
+        <mass
+          value="5.77242340173648" />
+        <inertia
+          ixx="0.0327019582662897"
+          ixy="-0.00189987845379704"
+          ixz="0.00937014136132958"
+          iyy="0.0373787564144547"
+          iyz="-0.00197023031658988"
+          izz="0.0348614383349291" />
+      </inertial>
+      <visual>
+        <origin xyz="0 0 0" rpy="0 0 0"/>
         <geometry>
           <mesh filename="package://kuka_kr5_support/meshes/kr5_arc/visual/link_1.dae" />
@@ -62,17 +62,17 @@
     <link name="${prefix}link_2">
       <inertial>
-      <origin
-        xyz="0.00610231661046294 0.0401115026555897 -0.11531122862673"
-        rpy="0 0 0" />
-      <mass
-        value="4.64974639735464" />
-      <inertia
-        ixx="0.0663459530931455"
-        ixy="0.000173652478770081"
-        ixz="0.000586191290902105"
-        iyy="0.070407913174161"
-        iyz="-0.00203071071007864"
-        izz="0.0102816377550493" />
-    </inertial>
+        <origin
+          xyz="0.00610231661046294 0.0401115026555897 -0.11531122862673"
+          rpy="0 0 0" />
+        <mass
+          value="4.64974639735464" />
+        <inertia
+          ixx="0.0663459530931455"
+          ixy="0.000173652478770081"
+          ixz="0.000586191290902105"
+          iyy="0.070407913174161"
+          iyz="-0.00203071071007864"
+          izz="0.0102816377550493" />
+      </inertial>
       <visual>
         <origin xyz="0 0 0" rpy="0 0 0"/>
@@ -91,17 +91,17 @@
     <link name="${prefix}link_3">
       <inertial>
-      <origin
-        xyz="0.0755031858462784 -0.046481517407519 -0.00506472105904233"
-        rpy="0 0 0" />
-      <mass
-        value="4.3593398708568" />
-      <inertia
-        ixx="0.0202008069207718"
-        ixy="5.72394748332304E-05"
-        ixz="0.000556621203065716"
-        iyy="0.0246796752429931"
-        iyz="0.000697020296811431"
-        izz="0.0178067561136726" />
-    </inertial>
+        <origin
+          xyz="0.0755031858462784 -0.046481517407519 -0.00506472105904233"
+          rpy="0 0 0" />
+        <mass
+          value="4.3593398708568" />
+        <inertia
+          ixx="0.0202008069207718"
+          ixy="5.72394748332304E-05"
+          ixz="0.000556621203065716"
+          iyy="0.0246796752429931"
+          iyz="0.000697020296811431"
+          izz="0.0178067561136726" />
+      </inertial>
       <visual>
         <origin xyz="0 0 0" rpy="0 0 0"/>
@@ -120,17 +120,17 @@
     <link name="${prefix}link_4">
       <inertial>
-      <origin
-        xyz="0.0857493724873204 -0.00149370513017266 -0.00271609825446984"
-        rpy="0 0 0" />
-      <mass
-        value="2.06809715541017" />
-      <inertia
-        ixx="0.00444943757623485"
-        ixy="-0.000424915429214687"
-        ixz="-0.000117340671961173"
-        iyy="0.00882693069799353"
-        iyz="0.000136971152627904"
-        izz="0.0101131228921778" />
-    </inertial>
+        <origin
+          xyz="0.0857493724873204 -0.00149370513017266 -0.00271609825446984"
+          rpy="0 0 0" />
+        <mass
+          value="2.06809715541017" />
+        <inertia
+          ixx="0.00444943757623485"
+          ixy="-0.000424915429214687"
+          ixz="-0.000117340671961173"
+          iyy="0.00882693069799353"
+          iyz="0.000136971152627904"
+          izz="0.0101131228921778" />
+      </inertial>
       <visual>
         <origin xyz="0 0 0" rpy="0 0 0"/>
@@ -149,17 +149,17 @@
     <link name="${prefix}link_5">
       <inertial>
-      <origin
-        xyz="0 0 0"
-        rpy="0 0 0" />
-      <mass
-        value="0.328309098974388" />
-      <inertia
-        ixx="0.000221789219477276"
-        ixy="-9.59628913869705E-07"
-        ixz="1.40395663663479E-20"
-        iyy="0.000321152451627032"
-        iyz="-4.44973606670705E-20"
-        izz="0.000275966419870925" />
-    </inertial>
+        <origin
+          xyz="0 0 0"
+          rpy="0 0 0" />
+        <mass
+          value="0.328309098974388" />
+        <inertia
+          ixx="0.000221789219477276"
+          ixy="-9.59628913869705E-07"
+          ixz="1.40395663663479E-20"
+          iyy="0.000321152451627032"
+          iyz="-4.44973606670705E-20"
+          izz="0.000275966419870925" />
+      </inertial>
       <visual>
         <origin xyz="0 0 0" rpy="0 0 0"/>
@@ -178,17 +178,17 @@
     <link name="${prefix}link_6">
       <inertial>
-      <origin
-        xyz="0.00983949894991115 -2.78372724487979E-05 -1.11022302462516E-15"
-        rpy="0 0 0" />
-      <mass
-        value="0.0789494717998531" />
-      <inertia
-        ixx="3.53285039019399E-05"
-        ixy="-3.23299732456798E-08"
-        ixz="-6.9643163510009E-19"
-        iyy="2.30177957763861E-05"
-        iyz="-9.26550270485857E-19"
-        izz="2.28539400944714E-05" />
-    </inertial>
+        <origin
+          xyz="0.00983949894991115 -2.78372724487979E-05 -1.11022302462516E-15"
+          rpy="0 0 0" />
+        <mass
+          value="0.0789494717998531" />
+        <inertia
+          ixx="3.53285039019399E-05"
+          ixy="-3.23299732456798E-08"
+          ixz="-6.9643163510009E-19"
+          iyy="2.30177957763861E-05"
+          iyz="-9.26550270485857E-19"
+          izz="2.28539400944714E-05" />
+      </inertial>
       <visual>
         <origin xyz="0 0 0" rpy="0 0 0"/>
