Commit message: Added KR5 Podest

File: kuka_kr5_support/urdf/kr5_arc_macro.xacro (robot description, xacro)
@@ -12,20 +12,19 @@
       <link name="${prefix}podest_link">
         <xacro:default_inertial/>
-       <!-- <visual>
-          <origin xyz="0 0 0" rpy="0 0 ${-M_PI/2}" />
-          <geometry>
-            <mesh filename="package://schunk_description/meshes/lwa4p/A0_1.stl" scale="0.001 0.001 0.001" />
-          </geometry>
-          <material name="Schunk/DarkGrey" />
+        <visual>
+            <origin rpy="0 0 0" xyz="0 0 0"/>
+            <geometry>
+            <mesh filename="package://kuka_kr5_support/meshes/kr5_arc/visual/podest_link.dae" />
+            </geometry>
         </visual>
         <collision>
-          <origin xyz="0 0 0" rpy="0 0 ${-M_PI/2}" />
-          <geometry>
-            <mesh filename="package://schunk_description/meshes/lwa4p/A0_1.stl" scale="0.001 0.001 0.001" />
-          </geometry>
-        </collision>-->
+            <origin rpy="0 0 0" xyz="0 0 0"/>
+            <geometry>
+            <mesh filename="package://kuka_kr5_support/meshes/kr5_arc/collision/podest_link.stl" scale="0.001 0.001 0.001" />
+            </geometry>
+        </collision>
       </link>
       <joint name="${prefix}base_joint" type="fixed">
-        <origin xyz="0 0 0.30" rpy="0 0 0" />
+        <origin xyz="0 0 0.441" rpy="0 0 0" />
         <parent link="${prefix}podest_link"/>
         <child link="${prefix}base_link"/>

Commit message: Partitial changes as disscussed... the rest follows

File: kuka_kr5_support/urdf/kr5_arc_macro.xacro (robot description, xacro)
@@ -1,5 +1,5 @@
 <?xml version="1.0"?>
 <robot xmlns:xacro="http://www.ros.org/wiki/xacro">
-  <xacro:property name="M_PI" value="3.1415926535897931" />
+  <xacro:property name="pi" value="3.1415926535897931" />
   <xacro:property name="KUKA_DEG2RAD" value="0.017453292519943295"/>
   <xacro:macro name="kuka_kr5_arc" params="prefix parent *origin has_podest">
@@ -43,4 +43,11 @@
       </joint>
     </xacro:unless>
+    <link name="${prefix}base" />
+    <!-- TODO: Check this with robots controller (c.f. http://wiki.ros.org/Industrial/Tutorials/Create%20a%20URDF%20for%20an%20Industrial%20Robot#Additional.2BAC8-Standard_Frames) -->
+    <joint name="${prefix}base_link-base" type="fixed">
+      <parent link="${prefix}base_link" />
+      <child link="${prefix}base" />
+      <origin xyz="0 0 0" rpy="0 0 0" />
+    </joint>
     <!-- LINKS -->
     <!-- base link -->
@@ -252,17 +259,17 @@
     <!-- joint 1 (A1) -->
     <joint name="${prefix}joint_a1" type="revolute">
-      <origin xyz="0 0 0.4" rpy="${M_PI} 0 0"/>
+      <origin xyz="0 0 0.4" rpy="${pi} 0 0"/>
       <parent link="${prefix}base_link"/>
       <child link="${prefix}link_1"/>
       <axis xyz="0 0 1"/>
-      <limit effort="0" lower="${-KUKA_DEG2RAD * 155}" upper="${KUKA_DEG2RAD * 155}" velocity="${KUKA_DEG2RAD * 154}"/>
+      <limit effort="0" lower="${radians(-155)}" upper="${radians(155)}" velocity="${radians(154)}"/>
     </joint>
     <!-- joint 2 (A2) -->
     <joint name="${prefix}joint_a2" type="revolute">
-      <origin xyz="0.18 0 0" rpy="${M_PI/2} 0 0"/>
+      <origin xyz="0.18 0 0" rpy="${pi/2} 0 0"/>
       <parent link="${prefix}link_1"/>
       <child link="${prefix}link_2"/>
       <axis xyz="0 0 1"/>
-      <limit effort="0" lower="${-KUKA_DEG2RAD * 180}" upper="${KUKA_DEG2RAD * 65}" velocity="${KUKA_DEG2RAD * 154}"/>
+      <limit effort="0" lower="${radians(-180)}" upper="${radians(65)}" velocity="${radians(154)}"/>
     </joint>
     <!-- joint 3 (A3) -->
@@ -272,35 +279,35 @@
       <child link="${prefix}link_3"/>
       <axis xyz="0 0 1"/>
-      <limit effort="0" lower="${-KUKA_DEG2RAD * 15}" upper="${KUKA_DEG2RAD * 158}" velocity="${KUKA_DEG2RAD * 228}"/>
+      <limit effort="0" lower="${radians(-15)}" upper="${radians(158)}" velocity="${radians(228)}"/>
     </joint>
     <!-- joint 4 (A4) -->
     <joint name="${prefix}joint_a4" type="revolute">
-      <origin xyz="0.62 -0.12 0" rpy="0 ${-M_PI/2} 0"/>
+      <origin xyz="0.62 -0.12 0" rpy="0 ${-pi/2} 0"/>
       <parent link="${prefix}link_3"/>
       <child link="${prefix}link_4"/>
       <axis xyz="0 0 1"/>
-      <limit effort="0" lower="${-KUKA_DEG2RAD * 350}" upper="${KUKA_DEG2RAD * 350}" velocity="${KUKA_DEG2RAD * 343}"/>
+      <limit effort="0" lower="${radians(350)}" upper="${radians(350)}" velocity="${radians(343)}"/>
     </joint>
     <!-- joint 5 (A5) -->
     <joint name="${prefix}joint_a5" type="revolute">
-      <origin xyz="0 0 0" rpy="0 ${M_PI/2} 0"/>
+      <origin xyz="0 0 0" rpy="0 ${pi/2} 0"/>
       <parent link="${prefix}link_4"/>
       <child link="${prefix}link_5"/>
       <axis xyz="0 0 1"/>
-      <limit effort="0" lower="${-KUKA_DEG2RAD * 130}" upper="${KUKA_DEG2RAD * 130}" velocity="${KUKA_DEG2RAD * 384}"/>
+      <limit effort="0" lower="${radians(-130)}" upper="${radians(130)}" velocity="${radians(384)}"/>
     </joint>
     <!-- joint 6 (A6) -->
     <joint name="${prefix}joint_a6" type="revolute">
-      <origin xyz="0 0 0" rpy="0 ${-M_PI/2} 0"/>
+      <origin xyz="0 0 0" rpy="0 ${-pi/2} 0"/>
       <parent link="${prefix}link_5"/>
       <child link="${prefix}link_6"/>
       <axis xyz="0 0 1"/>
-      <limit effort="0" lower="${-KUKA_DEG2RAD * 350}" upper="${KUKA_DEG2RAD * 350}" velocity="${KUKA_DEG2RAD * 721}"/>
+      <limit effort="0" lower="${radians(-350)}" upper="${radians(350)}" velocity="${radians(721)}"/>
     </joint>
     <!-- tool frame - fixed frame -->
     <joint name="${prefix}joint_a6-tool0" type="fixed">
       <parent link="${prefix}link_6"/>
-      <child link="${prefix}tool_link"/>
-      <origin xyz="0 0 -0.115" rpy="0 ${-M_PI} 0"/>
+      <child link="${prefix}tool0"/>
+      <origin xyz="0 0 -0.115" rpy="0 ${-pi} 0"/>
     </joint>
     <!-- END JOINTS -->

Commit message: Removed shift in two axes on joint A4 and tool0 according to kuka manual

File: kuka_kr5_support/urdf/kr5_arc_macro.xacro (robot description, xacro)
@@ -235,5 +235,5 @@
     <!-- joint 4 (A4) -->
     <joint name="${prefix}joint_a4" type="revolute">
-      <origin xyz="0.62 -0.12 0" rpy="0 ${-pi/2} 0"/>
+      <origin xyz="0 -0.12 0" rpy="0 ${-pi/2} 0"/>
       <parent link="${prefix}link_3"/>
       <child link="${prefix}link_4"/>
@@ -243,5 +243,5 @@
     <!-- joint 5 (A5) -->
     <joint name="${prefix}joint_a5" type="revolute">
-      <origin xyz="0 0 0" rpy="0 ${pi/2} 0"/>
+      <origin xyz="0 0 -0.62" rpy="0 ${pi/2} 0"/>
       <parent link="${prefix}link_4"/>
       <child link="${prefix}link_5"/>
@@ -261,5 +261,5 @@
       <parent link="${prefix}link_6"/>
       <child link="${prefix}tool0"/>
-      <origin xyz="0 0 -0.115" rpy="0 ${-pi} 0"/>
+      <origin xyz="0 0 -0.115" rpy="0 ${-pi} ${-pi/2}"/>
     </joint>
     <!-- END JOINTS -->

Commit message: kr5arc: change collision mesh units to meters.

File: kuka_kr5_support/urdf/kr5_arc_macro.xacro (robot description, xacro)
@@ -26,5 +26,5 @@
         <origin rpy="0 0 0" xyz="0 0 0"/>
         <geometry>
-          <mesh filename="package://kuka_kr5_support/meshes/kr5_arc/collision/base_link.stl" scale="0.001 0.001 0.001" />
+          <mesh filename="package://kuka_kr5_support/meshes/kr5_arc/collision/base_link.stl" />
         </geometry>
       </collision>
@@ -55,5 +55,5 @@
         <origin xyz="0 0 0" rpy="0 0 0"/>
         <geometry>
-          <mesh filename="package://kuka_kr5_support/meshes/kr5_arc/collision/link_1.stl" scale="0.001 0.001 0.001" />
+          <mesh filename="package://kuka_kr5_support/meshes/kr5_arc/collision/link_1.stl" />
         </geometry>
       </collision>
@@ -84,5 +84,5 @@
         <origin xyz="0 0 0" rpy="0 0 0"/>
         <geometry>
-          <mesh filename="package://kuka_kr5_support/meshes/kr5_arc/collision/link_2.stl" scale="0.001 0.001 0.001"  />
+          <mesh filename="package://kuka_kr5_support/meshes/kr5_arc/collision/link_2.stl"  />
         </geometry>
       </collision>
@@ -113,5 +113,5 @@
         <origin xyz="0 0 0" rpy="0 0 0"/>
         <geometry>
-          <mesh filename="package://kuka_kr5_support/meshes/kr5_arc/collision/link_3.stl" scale="0.001 0.001 0.001"  />
+          <mesh filename="package://kuka_kr5_support/meshes/kr5_arc/collision/link_3.stl"  />
         </geometry>
       </collision>
@@ -142,5 +142,5 @@
         <origin xyz="0 0 0" rpy="0 0 0"/>
         <geometry>
-          <mesh filename="package://kuka_kr5_support/meshes/kr5_arc/collision/link_4.stl" scale="0.001 0.001 0.001"  />
+          <mesh filename="package://kuka_kr5_support/meshes/kr5_arc/collision/link_4.stl"  />
         </geometry>
       </collision>
@@ -171,5 +171,5 @@
         <origin xyz="0 0 0" rpy="0 0 0"/>
         <geometry>
-          <mesh filename="package://kuka_kr5_support/meshes/kr5_arc/collision/link_5.stl" scale="0.001 0.001 0.001" />
+          <mesh filename="package://kuka_kr5_support/meshes/kr5_arc/collision/link_5.stl" />
         </geometry>
       </collision>
@@ -200,5 +200,5 @@
         <origin xyz="0 0 0" rpy="0 0 0"/>
         <geometry>
-          <mesh filename="package://kuka_kr5_support/meshes/kr5_arc/collision/link_6.stl" scale="0.001 0.001 0.001" />
+          <mesh filename="package://kuka_kr5_support/meshes/kr5_arc/collision/link_6.stl" />
         </geometry>
       </collision>
