Commit message: moved joint_a6-tool0 translation to joint_a5-joint_a6

File: kuka_kr150_support/urdf/kr150_2_macro.xacro (robot description, xacro)
@@ -155,5 +155,5 @@
     <!-- joint 6 (A6) -->
     <joint name="${prefix}joint_a6" type="revolute">
-      <origin xyz="0 0 0" rpy="0 0 0"/>
+      <origin xyz="0.23 0 0" rpy="0 0 0"/>
       <parent link="${prefix}link_5"/>
       <child link="${prefix}link_6"/>
@@ -165,5 +165,5 @@
       <parent link="${prefix}link_6"/>
       <child link="${prefix}tool0"/>
-      <origin xyz="0.23 0 0" rpy="0 ${pi/2} 0"/>
+      <origin xyz="0 0 0" rpy="0 ${pi/2} 0"/>
     </joint>
     <!-- END JOINTS -->
