Commit message: Review changes KR 150 R3100-2
- renamed kr150_r3100-2 to kr150r3100_2
- added doc title of spec document
- adapted xacro to ROS-I standards
- opw params: removed kinematics_solver

File: kuka_kr150_support/urdf/kr150r3100_2_macro.xacro (robot description, xacro)
@@ -1,7 +1,6 @@
 <?xml version="1.0"?>
 <robot xmlns:xacro="http://wiki.ros.org/xacro">
-  <xacro:include filename="$(find kuka_resources)/urdf/common_constants.xacro"/>
-  <xacro:include filename="$(find kuka_resources)/urdf/common_materials.xacro"/>
-  <xacro:macro name="kuka_kr150_r3100-2" params="prefix">
+  <xacro:macro name="kuka_kr150r3100_2" params="prefix">
+    <xacro:include filename="$(find kuka_resources)/urdf/common_materials.xacro"/>
     <!-- LINKS -->
     <!-- base link -->
@@ -10,5 +9,5 @@
         <origin rpy="0 0 0" xyz="0 0 0"/>
         <geometry>
-          <mesh filename="package://kuka_kr150_support/meshes/kr150_r3100-2/visual/base_link.stl" />
+          <mesh filename="package://kuka_kr150_support/meshes/kr150r3100_2/visual/base_link.stl" />
         </geometry>
         <xacro:material_kuka_pedestal />
@@ -17,5 +16,5 @@
         <origin rpy="0 0 0" xyz="0 0 0"/>
         <geometry>
-          <mesh filename="package://kuka_kr150_support/meshes/kr150_r3100-2/collision/base_link.stl" />
+          <mesh filename="package://kuka_kr150_support/meshes/kr150r3100_2/collision/base_link.stl" />
         </geometry>
       </collision>
@@ -26,5 +25,5 @@
         <origin xyz="0 0 0" rpy="0 0 0"/>
         <geometry>
-          <mesh filename="package://kuka_kr150_support/meshes/kr150_r3100-2/visual/link_1.stl" />
+          <mesh filename="package://kuka_kr150_support/meshes/kr150r3100_2/visual/link_1.stl" />
         </geometry>
         <xacro:material_kuka_orange />
@@ -33,5 +32,5 @@
         <origin xyz="0 0 0" rpy="0 0 0"/>
         <geometry>
-          <mesh filename="package://kuka_kr150_support/meshes/kr150_r3100-2/collision/link_1.stl" />
+          <mesh filename="package://kuka_kr150_support/meshes/kr150r3100_2/collision/link_1.stl" />
         </geometry>
       </collision>
@@ -42,5 +41,5 @@
         <origin xyz="0 0 0" rpy="0 0 0"/>
         <geometry>
-          <mesh filename="package://kuka_kr150_support/meshes/kr150_r3100-2/visual/link_2.stl"/>
+          <mesh filename="package://kuka_kr150_support/meshes/kr150r3100_2/visual/link_2.stl"/>
         </geometry>
         <xacro:material_kuka_orange />
@@ -49,5 +48,5 @@
         <origin xyz="0 0 0" rpy="0 0 0"/>
         <geometry>
-          <mesh filename="package://kuka_kr150_support/meshes/kr150_r3100-2/collision/link_2.stl"  />
+          <mesh filename="package://kuka_kr150_support/meshes/kr150r3100_2/collision/link_2.stl"  />
         </geometry>
       </collision>
@@ -58,5 +57,5 @@
         <origin xyz="0 0 0" rpy="0 0 0"/>
         <geometry>
-          <mesh filename="package://kuka_kr150_support/meshes/kr150_r3100-2/visual/link_3.stl" />
+          <mesh filename="package://kuka_kr150_support/meshes/kr150r3100_2/visual/link_3.stl" />
         </geometry>
         <xacro:material_kuka_orange />
@@ -65,5 +64,5 @@
         <origin xyz="0 0 0" rpy="0 0 0"/>
         <geometry>
-          <mesh filename="package://kuka_kr150_support/meshes/kr150_r3100-2/collision/link_3.stl"  />
+          <mesh filename="package://kuka_kr150_support/meshes/kr150r3100_2/collision/link_3.stl"  />
         </geometry>
       </collision>
@@ -74,5 +73,5 @@
         <origin xyz="0 0 0" rpy="0 0 0"/>
         <geometry>
-          <mesh filename="package://kuka_kr150_support/meshes/kr150_r3100-2/visual/link_4.stl" />
+          <mesh filename="package://kuka_kr150_support/meshes/kr150r3100_2/visual/link_4.stl" />
         </geometry>
         <xacro:material_kuka_orange />
@@ -81,5 +80,5 @@
         <origin xyz="0 0 0" rpy="0 0 0"/>
         <geometry>
-          <mesh filename="package://kuka_kr150_support/meshes/kr150_r3100-2/collision/link_4.stl"  />
+          <mesh filename="package://kuka_kr150_support/meshes/kr150r3100_2/collision/link_4.stl"  />
         </geometry>
       </collision>
@@ -90,5 +89,5 @@
         <origin xyz="0 0 0" rpy="0 0 0"/>
         <geometry>
-          <mesh filename="package://kuka_kr150_support/meshes/kr150_r3100-2/visual/link_5.stl" />
+          <mesh filename="package://kuka_kr150_support/meshes/kr150r3100_2/visual/link_5.stl" />
         </geometry>
         <xacro:material_kuka_orange />
@@ -97,5 +96,5 @@
         <origin xyz="0 0 0" rpy="0 0 0"/>
         <geometry>
-          <mesh filename="package://kuka_kr150_support/meshes/kr150_r3100-2/collision/link_5.stl" />
+          <mesh filename="package://kuka_kr150_support/meshes/kr150r3100_2/collision/link_5.stl" />
         </geometry>
       </collision>
@@ -106,5 +105,5 @@
         <origin xyz="0 0 0" rpy="0 0 0"/>
         <geometry>
-          <mesh filename="package://kuka_kr150_support/meshes/kr150_r3100-2/visual/link_6.stl" />
+          <mesh filename="package://kuka_kr150_support/meshes/kr150r3100_2/visual/link_6.stl" />
         </geometry>
         <xacro:material_kuka_orange />
@@ -113,5 +112,5 @@
         <origin xyz="0 0 0" rpy="0 0 0"/>
         <geometry>
-          <mesh filename="package://kuka_kr150_support/meshes/kr150_r3100-2/collision/link_6.stl" />
+          <mesh filename="package://kuka_kr150_support/meshes/kr150r3100_2/collision/link_6.stl" />
         </geometry>
       </collision>
@@ -170,17 +169,25 @@
       <limit effort="0" lower="${radians(-350)}" upper="${radians(350)}" velocity="${radians(260)}"/>
     </joint>
-    <!-- tool frame - fixed frame -->
-    <joint name="${prefix}joint_a6-tool0" type="fixed">
-      <parent link="${prefix}link_6"/>
-      <child link="${prefix}tool0"/>
-      <origin xyz="0 0 0" rpy="0 ${pi/2} 0"/>
-    </joint>
-    <!-- END JOINTS -->
-    <!-- ROS base_link to KUKA $ROBROOT coordinate system transform -->
+    <!-- ROS-Industrial 'base' frame: base_link to KUKA $ROBROOT coordinate system transform -->
     <link name="${prefix}base" />
     <joint name="${prefix}base_link-base" type="fixed">
+      <origin xyz="0 0 0" rpy="0 0 0"/>
+      <parent link="${prefix}base_link"/>
+      <child link="${prefix}base"/>
+    </joint>
+    <!-- ROS-Industrial 'flange' frame: attachment point for EEF models -->
+    <link name="${prefix}flange" />
+    <joint name="${prefix}joint_6-flange" type="fixed">
       <origin xyz="0 0 0" rpy="0 0 0" />
-      <parent link="${prefix}base_link" />
-      <child link="${prefix}base" />
+      <parent link="${prefix}link_6" />
+      <child link="${prefix}flange" />
+    </joint>
+    <!-- ROS-Industrial 'tool0' frame: all-zeros tool frame -->
+    <!-- This frame corresponds to the $FLANGE coordinate system in KUKA KRC controllers. -->
+    <link name="${prefix}tool0"/>
+    <joint name="${prefix}flange-tool0" type="fixed">
+      <parent link="${prefix}flange"/>
+      <child link="${prefix}tool0"/>
+      <origin xyz="0 0 0" rpy="0 ${radians(90)} 0"/>
     </joint>
   </xacro:macro>

Commit message: Removed duplicated tool0 link

File: kuka_kr150_support/urdf/kr150r3100_2_macro.xacro (robot description, xacro)
@@ -116,7 +116,4 @@
       </collision>
     </link>
-    <!-- tool link -->
-    <!-- This frame corresponds to the $FLANGE coordinate system in KUKA KRC controllers. -->
-    <link name="${prefix}tool0"/>
     <!-- END LINKS -->
     <!-- JOINTS -->
