Commit message: Use Jade+ radians() in place of constant

File: kuka_kr3_support/urdf/kr3r540_macro.xacro (robot description, xacro)
@@ -1,5 +1,4 @@
 <?xml version="1.0"?>
 <robot xmlns:xacro="http://wiki.ros.org/xacro">
-  <xacro:include filename="$(find kuka_resources)/urdf/common_constants.xacro"/>
   <xacro:include filename="$(find kuka_resources)/urdf/common_materials.xacro"/>
   <xacro:macro name="kuka_kr3r540" params="prefix">
@@ -116,5 +115,5 @@
       <child link="${prefix}link_1"/>
       <axis xyz="0 0 -1"/>
-      <limit lower="${-170 * DEG2RAD}" upper="${170 * DEG2RAD}" effort="0" velocity="${530 * DEG2RAD}"/>
+      <limit lower="${radians(-170)}" upper="${radians(170)}" effort="0" velocity="${radians(530)}"/>
     </joint>
     <joint name="${prefix}joint_a2" type="revolute">
@@ -123,5 +122,5 @@
       <child link="${prefix}link_2"/>
       <axis xyz="0 1 0"/>
-      <limit lower="${-170 * DEG2RAD}" upper="${50 * DEG2RAD}" effort="0" velocity="${529 * DEG2RAD}"/>
+      <limit lower="${radians(-170)}" upper="${radians(50)}" effort="0" velocity="${radians(529)}"/>
     </joint>
     <joint name="${prefix}joint_a3" type="revolute">
@@ -130,5 +129,5 @@
       <child link="${prefix}link_3"/>
       <axis xyz="0 1 0"/>
-      <limit lower="${-110 * DEG2RAD}" upper="${155 * DEG2RAD}" effort="0" velocity="${538 * DEG2RAD}"/>
+      <limit lower="${radians(-110)}" upper="${radians(155)}" effort="0" velocity="${radians(538)}"/>
     </joint>
     <joint name="${prefix}joint_a4" type="revolute">
@@ -137,5 +136,5 @@
       <child link="${prefix}link_4"/>
       <axis xyz="-1 0 0"/>
-      <limit lower="${-175 * DEG2RAD}" upper="${175 * DEG2RAD}" effort="0" velocity="${600 * DEG2RAD}"/>
+      <limit lower="${radians(-175)}" upper="${radians(175)}" effort="0" velocity="${radians(600)}"/>
     </joint>
     <joint name="${prefix}joint_a5" type="revolute">
@@ -144,5 +143,5 @@
       <child link="${prefix}link_5"/>
       <axis xyz="0 1 0"/>
-      <limit lower="${-120 * DEG2RAD}" upper="${120 * DEG2RAD}" effort="0" velocity="${600 * DEG2RAD}"/>
+      <limit lower="${radians(-120)}" upper="${radians(120)}" effort="0" velocity="${radians(600)}"/>
     </joint>
     <joint name="${prefix}joint_a6" type="revolute">
@@ -151,10 +150,10 @@
       <child link="${prefix}link_6"/>
       <axis xyz="-1 0 0"/>
-      <limit lower="${-350 * DEG2RAD}" upper="${350 * DEG2RAD}" effort="0" velocity="${800 * DEG2RAD}"/>
+      <limit lower="${radians(-350)}" upper="${radians(350)}" effort="0" velocity="${radians(800)}"/>
     </joint>
     <joint name="${prefix}joint_a6-tool0" type="fixed">
       <parent link="${prefix}link_6"/>
       <child link="${prefix}tool0"/>
-      <origin xyz="0 0 0" rpy="0 ${90 * DEG2RAD} 0"/>
+      <origin xyz="0 0 0" rpy="0 ${radians(90)} 0"/>
     </joint>
     <!-- ROS base_link to KUKA $ROBROOT coordinate system transform -->

Commit message: Switching to stl from dae for size considerations

File: kuka_kr3_support/urdf/kr3r540_macro.xacro (robot description, xacro)
@@ -7,5 +7,5 @@
         <origin xyz="0 0 0" rpy="0 0 0" />
         <geometry>
-          <mesh filename="package://kuka_kr3_support/meshes/kr3r540/visual/base_link.dae" />
+          <mesh filename="package://kuka_kr3_support/meshes/kr3r540/visual/base_link.stl" />
         </geometry>
         <xacro:material_kuka_pedestal />
@@ -22,5 +22,5 @@
         <origin xyz="0 0 0" rpy="0 0 0" />
         <geometry>
-          <mesh filename="package://kuka_kr3_support/meshes/kr3r540/visual/link_1.dae" />
+          <mesh filename="package://kuka_kr3_support/meshes/kr3r540/visual/link_1.stl" />
         </geometry>
         <xacro:material_kuka_ral_pure_white />
@@ -37,5 +37,5 @@
         <origin xyz="0 0 0" rpy="0 0 0" />
         <geometry>
-          <mesh filename="package://kuka_kr3_support/meshes/kr3r540/visual/link_2.dae" />
+          <mesh filename="package://kuka_kr3_support/meshes/kr3r540/visual/link_2.stl" />
         </geometry>
         <xacro:material_kuka_ral_pure_white />
@@ -52,5 +52,5 @@
         <origin xyz="0 0 0" rpy="0 0 0" />
         <geometry>
-          <mesh filename="package://kuka_kr3_support/meshes/kr3r540/visual/link_3.dae" />
+          <mesh filename="package://kuka_kr3_support/meshes/kr3r540/visual/link_3.stl" />
         </geometry>
         <xacro:material_kuka_ral_pure_white />
@@ -67,5 +67,5 @@
         <origin xyz="0 0 0" rpy="0 0 0" />
         <geometry>
-          <mesh filename="package://kuka_kr3_support/meshes/kr3r540/visual/link_4.dae" />
+          <mesh filename="package://kuka_kr3_support/meshes/kr3r540/visual/link_4.stl" />
         </geometry>
         <xacro:material_kuka_ral_pure_white />
@@ -82,5 +82,5 @@
         <origin xyz="0 0 0" rpy="0 0 0" />
         <geometry>
-          <mesh filename="package://kuka_kr3_support/meshes/kr3r540/visual/link_5.dae" />
+          <mesh filename="package://kuka_kr3_support/meshes/kr3r540/visual/link_5.stl" />
         </geometry>
         <xacro:material_kuka_ral_pure_white />
@@ -97,5 +97,5 @@
         <origin xyz="0 0 0" rpy="0 0 0" />
         <geometry>
-          <mesh filename="package://kuka_kr3_support/meshes/kr3r540/visual/link_6.dae" />
+          <mesh filename="package://kuka_kr3_support/meshes/kr3r540/visual/link_6.stl" />
         </geometry>
         <xacro:material_kuka_pedestal />
