Commit message: new stl files and matching frames to allow for only one offset per joint in xacro

File: kuka_lbr_iiwa_support/urdf/lbr_iiwa_14_r820_macro.xacro (robot description, xacro)
@@ -7,5 +7,5 @@
         <origin xyz="0 0 0" rpy="0 0 0" />
         <geometry>
-          <mesh filename="package://kuka_lbr_iiwa_support/meshes/lbr_iiwa_14_r820/visual/base_link.dae" />
+          <mesh filename="package://kuka_lbr_iiwa_support/meshes/lbr_iiwa_14_r820/visual/base_link.stl" />
         </geometry>
       </visual>
@@ -21,5 +21,5 @@
         <origin xyz="0 0 0" rpy="0 0 0" />
         <geometry>
-          <mesh filename="package://kuka_lbr_iiwa_support/meshes/lbr_iiwa_14_r820/visual/link_1.dae" />
+          <mesh filename="package://kuka_lbr_iiwa_support/meshes/lbr_iiwa_14_r820/visual/link_1.stl" />
         </geometry>
       </visual>
@@ -35,5 +35,5 @@
         <origin xyz="0 0 0" rpy="0 0 0" />
         <geometry>
-          <mesh filename="package://kuka_lbr_iiwa_support/meshes/lbr_iiwa_14_r820/visual/link_2.dae" />
+          <mesh filename="package://kuka_lbr_iiwa_support/meshes/lbr_iiwa_14_r820/visual/link_2.stl" />
         </geometry>
       </visual>
@@ -49,5 +49,5 @@
         <origin xyz="0 0 0" rpy="0 0 0" />
         <geometry>
-          <mesh filename="package://kuka_lbr_iiwa_support/meshes/lbr_iiwa_14_r820/visual/link_3.dae" />
+          <mesh filename="package://kuka_lbr_iiwa_support/meshes/lbr_iiwa_14_r820/visual/link_3.stl" />
         </geometry>
       </visual>
@@ -63,5 +63,5 @@
         <origin xyz="0 0 0" rpy="0 0 0" />
         <geometry>
-          <mesh filename="package://kuka_lbr_iiwa_support/meshes/lbr_iiwa_14_r820/visual/link_4.dae" />
+          <mesh filename="package://kuka_lbr_iiwa_support/meshes/lbr_iiwa_14_r820/visual/link_4.stl" />
         </geometry>
       </visual>
@@ -77,5 +77,5 @@
         <origin xyz="0 0 0" rpy="0 0 0" />
         <geometry>
-          <mesh filename="package://kuka_lbr_iiwa_support/meshes/lbr_iiwa_14_r820/visual/link_5.dae" />
+          <mesh filename="package://kuka_lbr_iiwa_support/meshes/lbr_iiwa_14_r820/visual/link_5.stl" />
         </geometry>
       </visual>
@@ -91,5 +91,5 @@
         <origin xyz="0 0 0" rpy="0 0 0" />
         <geometry>
-          <mesh filename="package://kuka_lbr_iiwa_support/meshes/lbr_iiwa_14_r820/visual/link_6.dae" />
+          <mesh filename="package://kuka_lbr_iiwa_support/meshes/lbr_iiwa_14_r820/visual/link_6.stl" />
         </geometry>
       </visual>
@@ -105,5 +105,5 @@
         <origin xyz="0 0 0" rpy="0 0 0" />
         <geometry>
-          <mesh filename="package://kuka_lbr_iiwa_support/meshes/lbr_iiwa_14_r820/visual/link_7.dae" />
+          <mesh filename="package://kuka_lbr_iiwa_support/meshes/lbr_iiwa_14_r820/visual/link_7.stl" />
         </geometry>
       </visual>
@@ -119,54 +119,54 @@
     <!-- joint list -->
     <joint name="${prefix}joint_a1" type="revolute">
-      <origin xyz="0 0 0" rpy="0 0 0" />
+      <origin xyz="0 0 0.36" rpy="0 0 0" />
       <parent link="${prefix}base_link" />
       <child link="${prefix}link_1" />
       <axis xyz="0 0 1" />
-      <limit lower="-2.9668" upper="2.9668" effort="0" velocity="1.4834" />
+      <limit lower="-2.967" upper="2.967" effort="0" velocity="1.4835" />
     </joint>
     <joint name="${prefix}joint_a2" type="revolute">
-      <origin xyz="-0.00043624 0 0.36" rpy="0 0 0" />
+      <origin xyz="0 0 0" rpy="0 0 0" />
       <parent link="${prefix}link_1" />
       <child link="${prefix}link_2" />
       <axis xyz="0 1 0" />
-      <limit lower="-2.0942" upper="2.0942" effort="0" velocity="1.4834" />
+      <limit lower="-2.094" upper="2.094" effort="0" velocity="1.4835" />
     </joint>
     <joint name="${prefix}joint_a3" type="revolute">
-      <origin xyz="0 0 0" rpy="0 0 0" />
+      <origin xyz="0 0 0.42" rpy="0 0 0" />
       <parent link="${prefix}link_2" />
       <child link="${prefix}link_3" />
       <axis xyz="0 0 1" />
-      <limit lower="-2.9668" upper="2.9668" effort="0" velocity="1.7452" />
+      <limit lower="-2.967" upper="2.967" effort="0" velocity="1.7453" />
     </joint>
     <joint name="${prefix}joint_a4" type="revolute">
-      <origin xyz="0.00043624 0 0.42" rpy="0 0 0" />
+      <origin xyz="0 0 0" rpy="0 0 0" />
       <parent link="${prefix}link_3" />
       <child link="${prefix}link_4" />
       <axis xyz="0 -1 0" />
-      <limit lower="-2.0942" upper="2.0942" effort="0" velocity="1.3089" />
+      <limit lower="-2.094" upper="2.094" effort="0" velocity="1.3089" />
     </joint>
     <joint name="${prefix}joint_a5" type="revolute">
-      <origin xyz="0 0 0" rpy="0 0 0" />
+      <origin xyz="0 0 0.40" rpy="0 0 0" />
       <parent link="${prefix}link_4" />
       <child link="${prefix}link_5" />
       <axis xyz="0 0 1" />
-      <limit lower="-2.9668" upper="2.9668" effort="0" velocity="2.2688" />
+      <limit lower="-2.967" upper="2.967" effort="0" velocity="2.2689" />
     </joint>
     <joint name="${prefix}joint_a6" type="revolute">
-      <origin xyz="0 0 0.4" rpy="0 0 0" />
+      <origin xyz="0 0 0" rpy="0 0 0" />
       <parent link="${prefix}link_5" />
       <child link="${prefix}link_6" />
       <axis xyz="0 1 0" />
-      <limit lower="-2.0942" upper="2.0942" effort="0" velocity="2.356" />
+      <limit lower="-2.094" upper="2.094" effort="0" velocity="2.356" />
     </joint>
     <joint name="${prefix}joint_a7" type="revolute">
-      <origin xyz="0 0 0" rpy="0 0 0" />
+      <origin xyz="0 0 0.126" rpy="0 0 0" />
       <parent link="${prefix}link_6" />
       <child link="${prefix}link_7" />
       <axis xyz="0 0 1" />
-      <limit lower="-3.0541" upper="3.0541" effort="0" velocity="2.356" />
+      <limit lower="-3.054" upper="3.054" effort="0" velocity="2.356" />
     </joint>
     <joint name="${prefix}joint_a7-tool0" type="fixed">
-      <origin xyz="0 0 0.126" rpy="0 0 0" />
+      <origin xyz="0 0 0" rpy="0 0 0" />
       <parent link="${prefix}link_7" />
       <child link="${prefix}tool0" />

Commit message: updated joint limits and velocities to radians macros

File: kuka_lbr_iiwa_support/urdf/lbr_iiwa_14_r820_macro.xacro (robot description, xacro)
@@ -123,5 +123,5 @@
       <child link="${prefix}link_1" />
       <axis xyz="0 0 1" />
-      <limit lower="-2.967" upper="2.967" effort="0" velocity="1.4835" />
+      <limit lower="${radians(-170)}" upper="${radians(170)}" effort="0" velocity="${radians(85)}" />
     </joint>
     <joint name="${prefix}joint_a2" type="revolute">
@@ -130,5 +130,5 @@
       <child link="${prefix}link_2" />
       <axis xyz="0 1 0" />
-      <limit lower="-2.094" upper="2.094" effort="0" velocity="1.4835" />
+      <limit lower="${radians(-120)}" upper="${radians(120)}" effort="0" velocity="${radians(85)}" />
     </joint>
     <joint name="${prefix}joint_a3" type="revolute">
@@ -137,5 +137,5 @@
       <child link="${prefix}link_3" />
       <axis xyz="0 0 1" />
-      <limit lower="-2.967" upper="2.967" effort="0" velocity="1.7453" />
+      <limit lower="${radians(-170)}" upper="${radians(170)}" effort="0" velocity="${radians(100)}" />
     </joint>
     <joint name="${prefix}joint_a4" type="revolute">
@@ -144,5 +144,5 @@
       <child link="${prefix}link_4" />
       <axis xyz="0 -1 0" />
-      <limit lower="-2.094" upper="2.094" effort="0" velocity="1.3089" />
+      <limit lower="${radians(-120)}" upper="${radians(120)}" effort="0" velocity="${radians(75)}" />
     </joint>
     <joint name="${prefix}joint_a5" type="revolute">
@@ -151,5 +151,5 @@
       <child link="${prefix}link_5" />
       <axis xyz="0 0 1" />
-      <limit lower="-2.967" upper="2.967" effort="0" velocity="2.2689" />
+      <limit lower="${radians(-170)}" upper="${radians(170)}" effort="0" velocity="${radians(130)}" />
     </joint>
     <joint name="${prefix}joint_a6" type="revolute">
@@ -158,5 +158,5 @@
       <child link="${prefix}link_6" />
       <axis xyz="0 1 0" />
-      <limit lower="-2.094" upper="2.094" effort="0" velocity="2.356" />
+      <limit lower="${radians(-120)}" upper="${radians(120)}" effort="0" velocity="${radians(-135)}" />
     </joint>
     <joint name="${prefix}joint_a7" type="revolute">
@@ -165,5 +165,5 @@
       <child link="${prefix}link_7" />
       <axis xyz="0 0 1" />
-      <limit lower="-3.054" upper="3.054" effort="0" velocity="2.356" />
+      <limit lower="${radians(-175)}" upper="${radians(175)}" effort="0" velocity="${radians(135)}" />
     </joint>
     <joint name="${prefix}joint_a7-tool0" type="fixed">

Commit message: updated colors, decimated, added xacro for specifying flange type

File: kuka_lbr_iiwa_support/urdf/lbr_iiwa_14_r820_macro.xacro (robot description, xacro)
@@ -1,4 +1,8 @@
 <?xml version="1.0"?>
 <robot xmlns:xacro="http://wiki.ros.org/xacro">
+  <xacro:include filename="$(find kuka_resources)/urdf/common_materials.xacro"/>
+  <xacro:include filename="$(find kuka_lbr_iiwa_support)/urdf/lbr_iiwa_flanges_macro.xacro"/>
+  <!-- current support for the following values: basic, pneumatic_touch -->
+  <xacro:arg name="flange_type" default="basic" />
   <xacro:macro name="kuka_lbr_iiwa_14_r820" params="prefix">
     <!-- link list -->
@@ -9,4 +13,5 @@
           <mesh filename="package://kuka_lbr_iiwa_support/meshes/lbr_iiwa_14_r820/visual/base_link.stl" />
         </geometry>
+	<xacro:material_kuka_ral_pearly_white />
       </visual>
       <collision>
@@ -23,4 +28,5 @@
           <mesh filename="package://kuka_lbr_iiwa_support/meshes/lbr_iiwa_14_r820/visual/link_1.stl" />
         </geometry>
+	<xacro:material_kuka_ral_pearly_white />
       </visual>
       <collision>
@@ -37,4 +43,5 @@
           <mesh filename="package://kuka_lbr_iiwa_support/meshes/lbr_iiwa_14_r820/visual/link_2.stl" />
         </geometry>
+	<xacro:material_kuka_ral_pearly_white />
       </visual>
       <collision>
@@ -51,4 +58,5 @@
           <mesh filename="package://kuka_lbr_iiwa_support/meshes/lbr_iiwa_14_r820/visual/link_3.stl" />
         </geometry>
+	<xacro:material_kuka_ral_pearly_white />
       </visual>
       <collision>
@@ -65,4 +73,5 @@
           <mesh filename="package://kuka_lbr_iiwa_support/meshes/lbr_iiwa_14_r820/visual/link_4.stl" />
         </geometry>
+	<xacro:material_kuka_ral_pearly_white />
       </visual>
       <collision>
@@ -79,4 +88,5 @@
           <mesh filename="package://kuka_lbr_iiwa_support/meshes/lbr_iiwa_14_r820/visual/link_5.stl" />
         </geometry>
+	<xacro:material_kuka_ral_pearly_white />
       </visual>
       <collision>
@@ -93,4 +103,5 @@
           <mesh filename="package://kuka_lbr_iiwa_support/meshes/lbr_iiwa_14_r820/visual/link_6.stl" />
         </geometry>
+	<xacro:material_kuka_ral_pearly_white />
       </visual>
       <collision>
@@ -101,18 +112,5 @@
       </collision>
     </link>
-    <link name="${prefix}link_7">
-      <visual>
-        <origin xyz="0 0 0" rpy="0 0 0" />
-        <geometry>
-          <mesh filename="package://kuka_lbr_iiwa_support/meshes/lbr_iiwa_14_r820/visual/link_7.stl" />
-        </geometry>
-      </visual>
-      <collision>
-        <origin xyz="0 0 0" rpy="0 0 0" />
-        <geometry>
-          <mesh filename="package://kuka_lbr_iiwa_support/meshes/lbr_iiwa_14_r820/collision/link_7.stl" />
-        </geometry>
-      </collision>
-    </link>
+    <xacro:kuka_lbr_iiwa_flange_link prefix="${prefix}" flange_type="$(arg flange_type)"/>
     <link name="${prefix}tool0" />
     <!-- end of link list -->
@@ -160,11 +158,5 @@
       <limit lower="${radians(-120)}" upper="${radians(120)}" effort="0" velocity="${radians(-135)}" />
     </joint>
-    <joint name="${prefix}joint_a7" type="revolute">
-      <origin xyz="0 0 0.126" rpy="0 0 0" />
-      <parent link="${prefix}link_6" />
-      <child link="${prefix}link_7" />
-      <axis xyz="0 0 1" />
-      <limit lower="${radians(-175)}" upper="${radians(175)}" effort="0" velocity="${radians(135)}" />
-    </joint>
+    <xacro:kuka_lbr_iiwa_flange_joint prefix="${prefix}" flange_type="$(arg flange_type)"/>
     <joint name="${prefix}joint_a7-tool0" type="fixed">
       <origin xyz="0 0 0" rpy="0 0 0" />

Commit message: missed a merge diff in the macro.xacro

File: kuka_lbr_iiwa_support/urdf/lbr_iiwa_14_r820_macro.xacro (robot description, xacro)
@@ -112,22 +112,5 @@
       </collision>
     </link>
-<<<<<<< HEAD
     <xacro:kuka_lbr_iiwa_flange_link prefix="${prefix}" flange_type="$(arg flange_type)"/>
-=======
-    <link name="${prefix}link_7">
-      <visual>
-        <origin xyz="0 0 0" rpy="0 0 0" />
-        <geometry>
-          <mesh filename="package://kuka_lbr_iiwa_support/meshes/lbr_iiwa_14_r820/visual/link_7.stl" />
-        </geometry>
-      </visual>
-      <collision>
-        <origin xyz="0 0 0" rpy="0 0 0" />
-        <geometry>
-          <mesh filename="package://kuka_lbr_iiwa_support/meshes/lbr_iiwa_14_r820/collision/link_7.stl" />
-        </geometry>
-      </collision>
-    </link>
->>>>>>> 90d28ba4e9541f3ba9392e667ebb19260d333760
     <link name="${prefix}tool0" />
     <!-- end of link list -->
@@ -174,14 +157,4 @@
       <axis xyz="0 1 0" />
       <limit lower="${radians(-120)}" upper="${radians(120)}" effort="0" velocity="${radians(-135)}" />
-<<<<<<< HEAD
-=======
-    </joint>
-    <joint name="${prefix}joint_a7" type="revolute">
-      <origin xyz="0 0 0.126" rpy="0 0 0" />
-      <parent link="${prefix}link_6" />
-      <child link="${prefix}link_7" />
-      <axis xyz="0 0 1" />
-      <limit lower="${radians(-175)}" upper="${radians(175)}" effort="0" velocity="${radians(135)}" />
->>>>>>> 90d28ba4e9541f3ba9392e667ebb19260d333760
     </joint>
     <xacro:kuka_lbr_iiwa_flange_joint prefix="${prefix}" flange_type="$(arg flange_type)"/>
