Commit message: addition of meshes to be modified

File: kuka_lbr_iiwa_support/urdf/lbr_iiwa_7_r800_macro.xacro (robot description, xacro)
@@ -1,5 +1,5 @@
 <?xml version="1.0"?>
 <robot xmlns:xacro="http://ros.org/wiki/xacro">
-  <xacro:macro name="kuka_lbr_iiwa_14_r820" params="prefix">
+  <xacro:macro name="kuka_lbr_iiwa_7_r800" params="prefix">
     <!-- link list -->
     <link name="${prefix}base_link">

Commit message: added new mesh files converted from .stp file on KUKA website

File: kuka_lbr_iiwa_support/urdf/lbr_iiwa_7_r800_macro.xacro (robot description, xacro)
@@ -7,5 +7,5 @@
         <origin xyz="0 0 0" rpy="0 0 0" />
         <geometry>
-          <mesh filename="package://kuka_lbr_iiwa_support/meshes/lbr_iiwa_14_r820/visual/base_link.dae" />
+          <mesh filename="package://kuka_lbr_iiwa_support/meshes/lbr_iiwa_7_r800/visual/base_link.dae" />
         </geometry>
       </visual>
@@ -13,5 +13,5 @@
         <origin xyz="0 0 0" rpy="0 0 0" />
         <geometry>
-          <mesh filename="package://kuka_lbr_iiwa_support/meshes/lbr_iiwa_14_r820/collision/base_link.stl" />
+          <mesh filename="package://kuka_lbr_iiwa_support/meshes/lbr_iiwa_7_r800/collision/base_link.stl" />
         </geometry>
       </collision>
@@ -21,5 +21,5 @@
         <origin xyz="0 0 0" rpy="0 0 0" />
         <geometry>
-          <mesh filename="package://kuka_lbr_iiwa_support/meshes/lbr_iiwa_14_r820/visual/link_1.dae" />
+          <mesh filename="package://kuka_lbr_iiwa_support/meshes/lbr_iiwa_7_r800/visual/link_1.dae" />
         </geometry>
       </visual>
@@ -27,5 +27,5 @@
         <origin xyz="0 0 0" rpy="0 0 0" />
         <geometry>
-          <mesh filename="package://kuka_lbr_iiwa_support/meshes/lbr_iiwa_14_r820/collision/link_1.stl" />
+          <mesh filename="package://kuka_lbr_iiwa_support/meshes/lbr_iiwa_7_r800/collision/link_1.stl" />
         </geometry>
       </collision>
@@ -35,5 +35,5 @@
         <origin xyz="0 0 0" rpy="0 0 0" />
         <geometry>
-          <mesh filename="package://kuka_lbr_iiwa_support/meshes/lbr_iiwa_14_r820/visual/link_2.dae" />
+          <mesh filename="package://kuka_lbr_iiwa_support/meshes/lbr_iiwa_7_r800/visual/link_2.dae" />
         </geometry>
       </visual>
@@ -41,5 +41,5 @@
         <origin xyz="0 0 0" rpy="0 0 0" />
         <geometry>
-          <mesh filename="package://kuka_lbr_iiwa_support/meshes/lbr_iiwa_14_r820/collision/link_2.stl" />
+          <mesh filename="package://kuka_lbr_iiwa_support/meshes/lbr_iiwa_7_r800/collision/link_2.stl" />
         </geometry>
       </collision>
@@ -49,5 +49,5 @@
         <origin xyz="0 0 0" rpy="0 0 0" />
         <geometry>
-          <mesh filename="package://kuka_lbr_iiwa_support/meshes/lbr_iiwa_14_r820/visual/link_3.dae" />
+          <mesh filename="package://kuka_lbr_iiwa_support/meshes/lbr_iiwa_7_r800/visual/link_3.dae" />
         </geometry>
       </visual>
@@ -55,5 +55,5 @@
         <origin xyz="0 0 0" rpy="0 0 0" />
         <geometry>
-          <mesh filename="package://kuka_lbr_iiwa_support/meshes/lbr_iiwa_14_r820/collision/link_3.stl" />
+          <mesh filename="package://kuka_lbr_iiwa_support/meshes/lbr_iiwa_7_r800/collision/link_3.stl" />
         </geometry>
       </collision>
@@ -63,5 +63,5 @@
         <origin xyz="0 0 0" rpy="0 0 0" />
         <geometry>
-          <mesh filename="package://kuka_lbr_iiwa_support/meshes/lbr_iiwa_14_r820/visual/link_4.dae" />
+          <mesh filename="package://kuka_lbr_iiwa_support/meshes/lbr_iiwa_7_r800/visual/link_4.dae" />
         </geometry>
       </visual>
@@ -69,5 +69,5 @@
         <origin xyz="0 0 0" rpy="0 0 0" />
         <geometry>
-          <mesh filename="package://kuka_lbr_iiwa_support/meshes/lbr_iiwa_14_r820/collision/link_4.stl" />
+          <mesh filename="package://kuka_lbr_iiwa_support/meshes/lbr_iiwa_7_r800/collision/link_4.stl" />
         </geometry>
       </collision>
@@ -77,5 +77,5 @@
         <origin xyz="0 0 0" rpy="0 0 0" />
         <geometry>
-          <mesh filename="package://kuka_lbr_iiwa_support/meshes/lbr_iiwa_14_r820/visual/link_5.dae" />
+          <mesh filename="package://kuka_lbr_iiwa_support/meshes/lbr_iiwa_7_r800/visual/link_5.dae" />
         </geometry>
       </visual>
@@ -83,5 +83,5 @@
         <origin xyz="0 0 0" rpy="0 0 0" />
         <geometry>
-          <mesh filename="package://kuka_lbr_iiwa_support/meshes/lbr_iiwa_14_r820/collision/link_5.stl" />
+          <mesh filename="package://kuka_lbr_iiwa_support/meshes/lbr_iiwa_7_r800/collision/link_5.stl" />
         </geometry>
       </collision>
@@ -91,5 +91,5 @@
         <origin xyz="0 0 0" rpy="0 0 0" />
         <geometry>
-          <mesh filename="package://kuka_lbr_iiwa_support/meshes/lbr_iiwa_14_r820/visual/link_6.dae" />
+          <mesh filename="package://kuka_lbr_iiwa_support/meshes/lbr_iiwa_7_r800/visual/link_6.dae" />
         </geometry>
       </visual>
@@ -97,5 +97,5 @@
         <origin xyz="0 0 0" rpy="0 0 0" />
         <geometry>
-          <mesh filename="package://kuka_lbr_iiwa_support/meshes/lbr_iiwa_14_r820/collision/link_6.stl" />
+          <mesh filename="package://kuka_lbr_iiwa_support/meshes/lbr_iiwa_7_r800/collision/link_6.stl" />
         </geometry>
       </collision>
@@ -105,5 +105,5 @@
         <origin xyz="0 0 0" rpy="0 0 0" />
         <geometry>
-          <mesh filename="package://kuka_lbr_iiwa_support/meshes/lbr_iiwa_14_r820/visual/link_7.dae" />
+          <mesh filename="package://kuka_lbr_iiwa_support/meshes/lbr_iiwa_7_r800/visual/link_7.dae" />
         </geometry>
       </visual>
@@ -111,5 +111,5 @@
         <origin xyz="0 0 0" rpy="0 0 0" />
         <geometry>
-          <mesh filename="package://kuka_lbr_iiwa_support/meshes/lbr_iiwa_14_r820/collision/link_7.stl" />
+          <mesh filename="package://kuka_lbr_iiwa_support/meshes/lbr_iiwa_7_r800/collision/link_7.stl" />
         </geometry>
       </collision>

Commit message: adjusted joint angles and velocities to radian macros

File: kuka_lbr_iiwa_support/urdf/lbr_iiwa_7_r800_macro.xacro (robot description, xacro)
@@ -123,5 +123,5 @@
       <child link="${prefix}link_1" />
       <axis xyz="0 0 1" />
-      <limit lower="-2.967" upper="2.967" effort="0" velocity="1.710" />
+      <limit lower="${radians(-170)}" upper="${radians(170)}" effort="0" velocity="${radians(98)}" />
     </joint>
     <joint name="${prefix}joint_a2" type="revolute">
@@ -130,5 +130,5 @@
       <child link="${prefix}link_2" />
       <axis xyz="0 1 0" />
-      <limit lower="-2.094" upper="2.094" effort="0" velocity="1.710" />
+      <limit lower="${radians(-120)}" upper="${radians(120)}" effort="0" velocity="${radians(98)}" />
     </joint>
     <joint name="${prefix}joint_a3" type="revolute">
@@ -137,5 +137,5 @@
       <child link="${prefix}link_3" />
       <axis xyz="0 0 1" />
-      <limit lower="-2.967" upper="2.967" effort="0" velocity="1.745" />
+      <limit lower="${radians(-170)}" upper="${radians(170)}" effort="0" velocity="${radians(100)}" />
     </joint>
     <joint name="${prefix}joint_a4" type="revolute">
@@ -144,5 +144,5 @@
       <child link="${prefix}link_4" />
       <axis xyz="0 -1 0" />
-      <limit lower="-2.094" upper="2.094" effort="0" velocity="2.269" />
+      <limit lower="${radians(-120)}" upper="${radians(120)}" effort="0" velocity="${radians(130)}" />
     </joint>
     <joint name="${prefix}joint_a5" type="revolute">
@@ -151,5 +151,5 @@
       <child link="${prefix}link_5" />
       <axis xyz="0 0 1" />
-      <limit lower="-2.967" upper="2.967" effort="0" velocity="2.443" />
+      <limit lower="${radians(-170)}" upper="${radians(170)}" effort="0" velocity="${radians(140)}" />
     </joint>
     <joint name="${prefix}joint_a6" type="revolute">
@@ -158,5 +158,5 @@
       <child link="${prefix}link_6" />
       <axis xyz="0 1 0" />
-      <limit lower="-2.094" upper="2.094" effort="0" velocity="3.142" />
+      <limit lower="${radians(-120)}" upper="${radians(120)}" effort="0" velocity="${radians(180)}" />
     </joint>
     <joint name="${prefix}joint_a7" type="revolute">
@@ -165,5 +165,5 @@
       <child link="${prefix}link_7" />
       <axis xyz="0 0 1" />
-      <limit lower="-3.054" upper="3.054" effort="0" velocity="3.142" />
+      <limit lower="${radians(-175)}" upper="${radians(175)}" effort="0" velocity="${radians(180)}" />
     </joint>
     <joint name="${prefix}joint_a7-tool0" type="fixed">

Commit message: replicated r820 modifications for flange xacro

File: kuka_lbr_iiwa_support/urdf/lbr_iiwa_7_r800_macro.xacro (robot description, xacro)
@@ -1,4 +1,8 @@
 <?xml version="1.0"?>
 <robot xmlns:xacro="http://wiki.ros.org/xacro">
+  <xacro:include filename="$(find kuka_resources)/urdf/common_materials.xacro"/>
+  <xacro:include filename="$(find kuka_lbr_iiwa_support)/urdf/lbr_iiwa_flanges_macro.xacro"/>
+  <!-- current support for the following values: basic, pneumatic_touch -->
+  <xacro:arg name="flange_type" default="basic" />
   <xacro:macro name="kuka_lbr_iiwa_7_r800" params="prefix">
     <!-- link list -->
@@ -9,4 +13,5 @@
           <mesh filename="package://kuka_lbr_iiwa_support/meshes/lbr_iiwa_7_r800/visual/base_link.stl" />
         </geometry>
+	<xacro:material_kuka_ral_pearly_white />
       </visual>
       <collision>
@@ -23,4 +28,5 @@
           <mesh filename="package://kuka_lbr_iiwa_support/meshes/lbr_iiwa_7_r800/visual/link_1.stl" />
         </geometry>
+	<xacro:material_kuka_ral_pearly_white />
       </visual>
       <collision>
@@ -37,4 +43,5 @@
           <mesh filename="package://kuka_lbr_iiwa_support/meshes/lbr_iiwa_7_r800/visual/link_2.stl" />
         </geometry>
+	<xacro:material_kuka_ral_pearly_white />
       </visual>
       <collision>
@@ -51,4 +58,5 @@
           <mesh filename="package://kuka_lbr_iiwa_support/meshes/lbr_iiwa_7_r800/visual/link_3.stl" />
         </geometry>
+	<xacro:material_kuka_ral_pearly_white />
       </visual>
       <collision>
@@ -65,4 +73,5 @@
           <mesh filename="package://kuka_lbr_iiwa_support/meshes/lbr_iiwa_7_r800/visual/link_4.stl" />
         </geometry>
+	<xacro:material_kuka_ral_pearly_white />
       </visual>
       <collision>
@@ -79,4 +88,5 @@
           <mesh filename="package://kuka_lbr_iiwa_support/meshes/lbr_iiwa_7_r800/visual/link_5.stl" />
         </geometry>
+	<xacro:material_kuka_ral_pearly_white />
       </visual>
       <collision>
@@ -93,4 +103,5 @@
           <mesh filename="package://kuka_lbr_iiwa_support/meshes/lbr_iiwa_7_r800/visual/link_6.stl" />
         </geometry>
+	<xacro:material_kuka_ral_pearly_white />
       </visual>
       <collision>
@@ -101,27 +112,14 @@
       </collision>
     </link>
-    <link name="${prefix}link_7">
-      <visual>
-        <origin xyz="0 0 0" rpy="0 0 0" />
-        <geometry>
-          <mesh filename="package://kuka_lbr_iiwa_support/meshes/lbr_iiwa_7_r800/visual/link_7.stl" />
-        </geometry>
-      </visual>
-      <collision>
-        <origin xyz="0 0 0" rpy="0 0 0" />
-        <geometry>
-          <mesh filename="package://kuka_lbr_iiwa_support/meshes/lbr_iiwa_7_r800/collision/link_7.stl" />
-        </geometry>
-      </collision>
-    </link>
+    <xacro:kuka_lbr_iiwa_flange_link prefix="${prefix}" flange_type="$(arg flange_type)"/>
     <link name="${prefix}tool0" />
     <!-- end of link list -->
     <!-- joint list -->
     <joint name="${prefix}joint_a1" type="revolute">
-      <origin xyz="0 0 0.34" rpy="0 0 0" />
+      <origin xyz="0 0 0.36" rpy="0 0 0" />
       <parent link="${prefix}base_link" />
       <child link="${prefix}link_1" />
       <axis xyz="0 0 1" />
-      <limit lower="${radians(-170)}" upper="${radians(170)}" effort="0" velocity="${radians(98)}" />
+      <limit lower="${radians(-170)}" upper="${radians(170)}" effort="0" velocity="${radians(85)}" />
     </joint>
     <joint name="${prefix}joint_a2" type="revolute">
@@ -130,8 +128,8 @@
       <child link="${prefix}link_2" />
       <axis xyz="0 1 0" />
-      <limit lower="${radians(-120)}" upper="${radians(120)}" effort="0" velocity="${radians(98)}" />
+      <limit lower="${radians(-120)}" upper="${radians(120)}" effort="0" velocity="${radians(85)}" />
     </joint>
     <joint name="${prefix}joint_a3" type="revolute">
-      <origin xyz="0 0 0.40" rpy="0 0 0" />
+      <origin xyz="0 0 0.42" rpy="0 0 0" />
       <parent link="${prefix}link_2" />
       <child link="${prefix}link_3" />
@@ -144,5 +142,5 @@
       <child link="${prefix}link_4" />
       <axis xyz="0 -1 0" />
-      <limit lower="${radians(-120)}" upper="${radians(120)}" effort="0" velocity="${radians(130)}" />
+      <limit lower="${radians(-120)}" upper="${radians(120)}" effort="0" velocity="${radians(75)}" />
     </joint>
     <joint name="${prefix}joint_a5" type="revolute">
@@ -151,5 +149,5 @@
       <child link="${prefix}link_5" />
       <axis xyz="0 0 1" />
-      <limit lower="${radians(-170)}" upper="${radians(170)}" effort="0" velocity="${radians(140)}" />
+      <limit lower="${radians(-170)}" upper="${radians(170)}" effort="0" velocity="${radians(130)}" />
     </joint>
     <joint name="${prefix}joint_a6" type="revolute">
@@ -158,13 +156,7 @@
       <child link="${prefix}link_6" />
       <axis xyz="0 1 0" />
-      <limit lower="${radians(-120)}" upper="${radians(120)}" effort="0" velocity="${radians(180)}" />
+      <limit lower="${radians(-120)}" upper="${radians(120)}" effort="0" velocity="${radians(-135)}" />
     </joint>
-    <joint name="${prefix}joint_a7" type="revolute">
-      <origin xyz="0 0 0.126" rpy="0 0 0" />
-      <parent link="${prefix}link_6" />
-      <child link="${prefix}link_7" />
-      <axis xyz="0 0 1" />
-      <limit lower="${radians(-175)}" upper="${radians(175)}" effort="0" velocity="${radians(180)}" />
-    </joint>
+    <xacro:kuka_lbr_iiwa_flange_joint prefix="${prefix}" flange_type="$(arg flange_type)"/>
     <joint name="${prefix}joint_a7-tool0" type="fixed">
       <origin xyz="0 0 0" rpy="0 0 0" />

Commit message: decimated and fixed joint offset issues from cloning 14_r820 xacro

File: kuka_lbr_iiwa_support/urdf/lbr_iiwa_7_r800_macro.xacro (robot description, xacro)
@@ -117,9 +117,9 @@
     <!-- joint list -->
     <joint name="${prefix}joint_a1" type="revolute">
-      <origin xyz="0 0 0.36" rpy="0 0 0" />
+      <origin xyz="0 0 0.34" rpy="0 0 0" />
       <parent link="${prefix}base_link" />
       <child link="${prefix}link_1" />
       <axis xyz="0 0 1" />
-      <limit lower="${radians(-170)}" upper="${radians(170)}" effort="0" velocity="${radians(85)}" />
+      <limit lower="${radians(-170)}" upper="${radians(170)}" effort="0" velocity="${radians(98)}" />
     </joint>
     <joint name="${prefix}joint_a2" type="revolute">
@@ -128,8 +128,8 @@
       <child link="${prefix}link_2" />
       <axis xyz="0 1 0" />
-      <limit lower="${radians(-120)}" upper="${radians(120)}" effort="0" velocity="${radians(85)}" />
+      <limit lower="${radians(-120)}" upper="${radians(120)}" effort="0" velocity="${radians(98)}" />
     </joint>
     <joint name="${prefix}joint_a3" type="revolute">
-      <origin xyz="0 0 0.42" rpy="0 0 0" />
+      <origin xyz="0 0 0.40" rpy="0 0 0" />
       <parent link="${prefix}link_2" />
       <child link="${prefix}link_3" />
@@ -142,5 +142,5 @@
       <child link="${prefix}link_4" />
       <axis xyz="0 -1 0" />
-      <limit lower="${radians(-120)}" upper="${radians(120)}" effort="0" velocity="${radians(75)}" />
+      <limit lower="${radians(-120)}" upper="${radians(120)}" effort="0" velocity="${radians(130)}" />
     </joint>
     <joint name="${prefix}joint_a5" type="revolute">
@@ -149,5 +149,5 @@
       <child link="${prefix}link_5" />
       <axis xyz="0 0 1" />
-      <limit lower="${radians(-170)}" upper="${radians(170)}" effort="0" velocity="${radians(130)}" />
+      <limit lower="${radians(-170)}" upper="${radians(170)}" effort="0" velocity="${radians(140)}" />
     </joint>
     <joint name="${prefix}joint_a6" type="revolute">
@@ -156,5 +156,5 @@
       <child link="${prefix}link_6" />
       <axis xyz="0 1 0" />
-      <limit lower="${radians(-120)}" upper="${radians(120)}" effort="0" velocity="${radians(-135)}" />
+      <limit lower="${radians(-120)}" upper="${radians(120)}" effort="0" velocity="${radians(180)}" />
     </joint>
     <xacro:kuka_lbr_iiwa_flange_joint prefix="${prefix}" flange_type="$(arg flange_type)"/>
