Commit message: Modify kr10 gazebo. Add service for DIO in rsi_hw_interface

File: kuka_kr10_gazebo/urdf/ft_macro.xacro (robot description, xacro)
@@ -6,16 +6,15 @@
   <xacro:kuka_ft_sensor prefix="${prefix}" />
   <gazebo reference="${prefix}ft_sensor_link">
-    <gravity>true</gravity>
-    <self_collide>false</self_collide>
-    <material value="Gazebo/Green" />
+    <material>Gazebo/Green</material>
+    <turnGravityOff>true</turnGravityOff>
+    <provideFeedback>true</provideFeedback>
   </gazebo>
   <gazebo reference="${prefix}tool_link">
-    <gravity>true</gravity>
-    <self_collide>false</self_collide>
-    <material value="Gazebo/Black" />
+    <material>Gazebo/Grey</material>
+    <turnGravityOff>true</turnGravityOff>
     <provideFeedback>true</provideFeedback>
   </gazebo>
   <!-- Enable the Joint Feedback -->
-  <gazebo reference="${prefix}ft_sensor_joint">
+  <gazebo reference="${prefix}joint_ft_sensor">
     <provideFeedback>true</provideFeedback>
   </gazebo>
@@ -23,5 +22,5 @@
     <robotNamespace>/${prefix}</robotNamespace>
     <type>transmission_interface/SimpleTransmission</type>
-    <joint name="${prefix}ft_sensor_joint">
+    <joint name="${prefix}joint_ft_sensor">
       <hardwareInterface>hardware_interface/PositionJointInterface</hardwareInterface>
     </joint>
@@ -33,8 +32,8 @@
   <gazebo>
     <plugin name="ft_sensor" filename="libgazebo_ros_ft_sensor.so">
-      <updateRate>100.0</updateRate>
+      <updateRate>1000.0</updateRate>
       <robotNamespace>${prefix}</robotNamespace>
       <topicName>/optoforce_node/OptoForceWrench</topicName>
-      <jointName>${prefix}ft_sensor_joint</jointName>
+      <jointName>${prefix}joint_ft_sensor</jointName>
       <noise>
         <type>gaussian</type>
@@ -44,4 +43,7 @@
     </plugin>
   </gazebo>
+  <gazebo reference="world">
+    <dampingFactor>0.0002</dampingFactor>
+  </gazebo>
 </xacro:macro>
 </robot>

File: kuka_kr10_gazebo/urdf/kr10.xacro (robot description, xacro)
@@ -8,6 +8,6 @@
   </xacro:kuka_kr10_robot>
   <!-- FT Senzor -->
-  <xacro:include filename="$(find kuka_kr10_gazebo)/urdf/ft_macro.xacro"/>
+  <!--xacro:include filename="$(find kuka_kr10_gazebo)/urdf/ft_macro.xacro"/-->
   <!-- arm -->
-  <xacro:FT_sensor_gazebo prefix=""/>
+  <!--xacro:FT_sensor_gazebo prefix=""/-->
 </robot>

File: kuka_kr10_support/urdf/ft_sensor_macro.xacro (robot description, xacro)
@@ -45,5 +45,5 @@
     </link>
     <!-- joint between arm_6_link and ft_sensor_link -->
-    <joint name="${prefix}ft_sensor_joint" type="revolute">
+    <joint name="${prefix}joint_ft_sensor" type="revolute">
       <origin xyz="0.0185 0 0" rpy="0 ${DEG2RAD * 90} 0" />
       <parent link="${prefix}link_6"/>
@@ -51,8 +51,7 @@
       <axis xyz="1 0 0" />
       <limit effort="0" velocity="0" lower="0" upper="0" />
-      <!--safety_controller k_position="20" k_velocity="25" soft_lower_limit="${-2.09 + 0.01}" soft_upper_limit="${2.09 - 0.01}" /-->
     </joint>
     <!-- joint between ft_sensor_link and tool_link -->
-    <joint name="${prefix}tool_joint" type="fixed">
+    <joint name="${prefix}joint_tool" type="fixed">
       <origin xyz="-0.035 -0.035 0.01875" rpy="${DEG2RAD * 90} 0 ${DEG2RAD * 90}" />
       <parent link="${prefix}ft_sensor_link"/>

File: kuka_kr10_support/urdf/kr10r1100sixx.xacro (robot description, xacro)
@@ -3,5 +3,5 @@
   <xacro:include filename="$(find kuka_kr10_support)/urdf/kr10r1100sixx_macro.xacro" />
   <xacro:kuka_kr10r1100sixx prefix=""/>
-  <xacro:include filename="$(find kuka_kr10_support)/urdf/ft_sensor_macro.xacro" />
-  <xacro:kuka_ft_sensor prefix=""/>
+  <!--xacro:include filename="$(find kuka_kr10_support)/urdf/ft_sensor_macro.xacro" /-->
+  <!--xacro:kuka_ft_sensor prefix=""/-->
 </robot>

File: kuka_kr10_support/urdf/kr10r1100sixx_macro.xacro (robot description, xacro)
@@ -200,12 +200,12 @@
       <inertial>
         <origin xyz="0 0 0" rpy="0 0 0" />
-        <mass value="1000000.0"/>
-        <inertia ixx="0.0"  ixy="0"  ixz="0" iyy="0.0" iyz="0" izz="0.0" />
+        <mass value="10000000000.0"/>
+        <inertia ixx="100000.0"  ixy="100000"  ixz="100000" iyy="100000.0" iyz="100000" izz="100000.0" />
       </inertial>
     </link>
     <joint name="${prefix}base_link-base" type="fixed">
       <origin xyz="0 0 0" rpy="0 0 0"/>
-      <parent link="${prefix}base_link"/>
-      <child link="${prefix}base"/>
+      <parent link="${prefix}base"/>
+      <child link="${prefix}base_link"/>
     </joint>
   </xacro:macro>
