Commit message: Revert changes to indigo

File: kuka_kr10_gazebo/urdf/kr10.xacro (robot description, xacro)
@@ -1,4 +1,4 @@
 <?xml version="1.0" ?>
-<robot name="kuka_kr10_gazebo" xmlns:xacro="http://ros.org/wiki/xacro">
+<robot name="kuka_kr10_gazebo" xmlns:xacro="http://wiki.ros.org/xacro">
   <!-- kr10 -->
   <xacro:include filename="$(find kuka_kr10_gazebo)/urdf/kr10_macro.xacro"/>

File: kuka_kr10_gazebo/urdf/kr10_macro.xacro (robot description, xacro)
@@ -1,4 +1,4 @@
 <?xml version="1.0"?>
-<robot xmlns:xacro="http://ros.org/wiki/xacro">
+<robot xmlns:xacro="http://wiki.ros.org/xacro">
 <xacro:include filename="$(find kuka_kr10_support)/urdf/kr10r1100sixx_macro.xacro"/>
 <xacro:macro name="kuka_kr10_robot" params="prefix">
@@ -73,21 +73,21 @@
   </gazebo>
   <gazebo reference="${prefix}link_1">
-    <material>Gazebo/DarkGrey</material>
+    <material>Gazebo/Orange</material>
     <turnGravityOff>true</turnGravityOff>
   </gazebo>
   <gazebo reference="${prefix}link_2">
-    <material>Gazebo/DarkGrey</material>
+    <material>Gazebo/Orange</material>
     <turnGravityOff>true</turnGravityOff>
   </gazebo>
   <gazebo reference="${prefix}link_3">
-    <material>Gazebo/DarkGrey</material>
+    <material>Gazebo/Orange</material>
     <turnGravityOff>true</turnGravityOff>
   </gazebo>
   <gazebo reference="${prefix}link_4">
-    <material>Gazebo/DarkGrey</material>
+    <material>Gazebo/Orange</material>
     <turnGravityOff>true</turnGravityOff>
   </gazebo>
   <gazebo reference="${prefix}link_5">
-    <material>Gazebo/DarkGrey</material>
+    <material>Gazebo/Orange</material>
     <turnGravityOff>true</turnGravityOff>
   </gazebo>

Commit message: Add pipe experiment tool for kr10. Add FT sensor. Add world for pipe experiment.

File: kuka_kr10_gazebo/urdf/kr10.xacro (robot description, xacro)
@@ -7,3 +7,7 @@
   	<origin xyz="0 0 0" rpy="0 0 0" />
   </xacro:kuka_kr10_robot>
+  <!-- FT Senzor -->
+  <xacro:include filename="$(find kuka_kr10_gazebo)/urdf/ft_macro.xacro"/>
+  <!-- arm -->
+  <xacro:FT_sensor_gazebo prefix=""/>
 </robot>

File: kuka_kr10_support/urdf/kr10r1100sixx.xacro (robot description, xacro)
@@ -3,3 +3,5 @@
   <xacro:include filename="$(find kuka_kr10_support)/urdf/kr10r1100sixx_macro.xacro" />
   <xacro:kuka_kr10r1100sixx prefix=""/>
+  <xacro:include filename="$(find kuka_kr10_support)/urdf/ft_sensor_macro.xacro" />
+  <xacro:kuka_ft_sensor prefix=""/>
 </robot>

File: kuka_kr10_support/urdf/kr10r1100sixx_macro.xacro (robot description, xacro)
@@ -19,7 +19,10 @@
       </collision>
       <inertial>
-        <mass value="14" />
-        <origin xyz="-0.0444859 -4.97e-05 0.1100921" rpy="0 0 0" />
-        <inertia ixx="0.08877213773" ixy="-0.000131033070251" ixz="-0.00150261923247" iyy="0.14293778144" iyz="-2.25256850538e-05" izz="0.126259385464" />
+        <!--mass value="14" /-->
+        <!--origin xyz="-0.0444859 -4.97e-05 0.1100921" rpy="0 0 0" /-->
+        <!--inertia ixx="0.08877213773" ixy="-0.000131033070251" ixz="-0.00150261923247" iyy="0.14293778144" iyz="-2.25256850538e-05" izz="0.126259385464" /-->
+        <origin xyz="0 0 0" rpy="0 0 0" />
+        <mass value="10000.0"/>
+        <inertia ixx="10000.0"  ixy="0"  ixz="0" iyy="10000.0" iyz="0" izz="10000.0" />
       </inertial>
     </link>
@@ -194,5 +197,11 @@
     </joint-->
     <!-- ROS base_link to KUKA $ROBROOT coordinate system transform -->
-    <link name="${prefix}base" />
+    <link name="${prefix}base">
+      <inertial>
+        <origin xyz="0 0 0" rpy="0 0 0" />
+        <mass value="1000000.0"/>
+        <inertia ixx="0.0"  ixy="0"  ixz="0" iyy="0.0" iyz="0" izz="0.0" />
+      </inertial>
+    </link>
     <joint name="${prefix}base_link-base" type="fixed">
       <origin xyz="0 0 0" rpy="0 0 0"/>

Commit message: Add endorse tool

File: kuka_kr10_gazebo/urdf/kr10.xacro (robot description, xacro)
@@ -11,3 +11,7 @@
   <!-- arm -->
   <!--xacro:FT_sensor_gazebo prefix=""/-->
+  <!-- ENDORSE Tool -->
+  <xacro:include filename="$(find kuka_kr10_gazebo)/urdf/endorse_tool_macro.xacro"/>
+  <!-- tool -->
+  <xacro:endorse_tool_gazebo prefix=""/>
 </robot>

File: kuka_kr10_gazebo/urdf/kr10_macro.xacro (robot description, xacro)
@@ -69,25 +69,25 @@
   <!-- Gazebo-specific link properties -->
   <gazebo reference="${prefix}base_link">
-    <material>Gazebo/Black</material>
+    <material>Gazebo/Grey</material>
     <turnGravityOff>true</turnGravityOff>
   </gazebo>
   <gazebo reference="${prefix}link_1">
-    <material>Gazebo/DarkGrey</material>
+    <material>Gazebo/Orange</material>
     <turnGravityOff>true</turnGravityOff>
   </gazebo>
   <gazebo reference="${prefix}link_2">
-    <material>Gazebo/DarkGrey</material>
+    <material>Gazebo/Orange</material>
     <turnGravityOff>true</turnGravityOff>
   </gazebo>
   <gazebo reference="${prefix}link_3">
-    <material>Gazebo/DarkGrey</material>
+    <material>Gazebo/Orange</material>
     <turnGravityOff>true</turnGravityOff>
   </gazebo>
   <gazebo reference="${prefix}link_4">
-    <material>Gazebo/DarkGrey</material>
+    <material>Gazebo/Orange</material>
     <turnGravityOff>true</turnGravityOff>
   </gazebo>
   <gazebo reference="${prefix}link_5">
-    <material>Gazebo/DarkGrey</material>
+    <material>Gazebo/Orange</material>
     <turnGravityOff>true</turnGravityOff>
   </gazebo>

File: kuka_kr10_support/urdf/kr10r1100sixx.xacro (robot description, xacro)
@@ -3,4 +3,6 @@
   <xacro:include filename="$(find kuka_kr10_support)/urdf/kr10r1100sixx_macro.xacro" />
   <xacro:kuka_kr10r1100sixx prefix=""/>
+  <xacro:include filename="$(find kuka_kr10_support)/urdf/endorse_tool_macro.xacro" />
+  <xacro:endorse_tool prefix=""/>
   <!--xacro:include filename="$(find kuka_kr10_support)/urdf/ft_sensor_macro.xacro" /-->
   <!--xacro:kuka_ft_sensor prefix=""/-->

File: kuka_kr10_support/urdf/kr10r1100sixx_macro.xacro (robot description, xacro)
@@ -175,5 +175,6 @@
       <child link="${prefix}link_4"/>
       <axis xyz="-1 0 0"/>
-      <limit effort="0" lower="${-DEG2RAD * 185}" upper="${DEG2RAD * 185}" velocity="${DEG2RAD * 381}"/>
+      <!--limit effort="0" lower="${-DEG2RAD * 185}" upper="${DEG2RAD * 185}" velocity="${DEG2RAD * 381}"/-->
+	<limit effort="0" lower="${-DEG2RAD * 120}" upper="${DEG2RAD * 120}" velocity="${DEG2RAD * 381}"/>
     </joint>
     <joint name="${prefix}joint_a5" type="revolute">

Commit message: Add proxxon driller support

File: kuka_kr10_gazebo/urdf/kr10.xacro (robot description, xacro)
@@ -14,6 +14,6 @@
   <!--xacro:include filename="$(find kuka_kr10_gazebo)/urdf/endorse_tool_macro.xacro"/-->
   <!-- Proxxon Drilling Tool -->
-  <xacro:include filename="$(find kuka_kr10_gazebo)/urdf/proxxon_drill_macro.xacro"/>
+  <!--xacro:include filename="$(find kuka_kr10_gazebo)/urdf/proxxon_drill_macro.xacro"/-->
   <!-- tool -->
-  <xacro:proxxon_drilling_tool_gazebo prefix=""/>
+  <!--xacro:proxxon_drilling_tool_gazebo prefix=""/-->
 </robot>

File: kuka_kr10_support/urdf/proxxon_drill_macro.xacro (robot description, xacro)
@@ -6,5 +6,5 @@
     <link name="${prefix}drilling_tool_link">
       <visual>
-        <origin xyz="-0.1564 0 -0.066" rpy="-${DEG2RAD * 90} -${DEG2RAD * 0} ${DEG2RAD * 90}"/>
+        <origin xyz="-0.1555 0 -0.066" rpy="-${DEG2RAD * 90} -${DEG2RAD * 0} ${DEG2RAD * 90}"/>
         <geometry>
           <mesh filename="package://kuka_kr10_support/meshes/kr10r1100sixx/visual/proxxon_drilling_v2.stl" scale="0.001 0.001 0.001" />
@@ -15,9 +15,9 @@
         <origin xyz="-0.1564 0 -0.066" rpy="-${DEG2RAD * 90} -${DEG2RAD * 0} ${DEG2RAD * 90}"/>
         <geometry>
-          <mesh filename="package://kuka_kr10_support/meshes/kr10r1100sixx/collision/proxxon_drilling_v2.stl" scale="0.001 0.001 0.001" />
+          <mesh filename="package://kuka_kr10_support/meshes/kr10r1100sixx/collision/proxxon_drilling_v2.stl" scale="0.0008 0.0008 0.0008" />
         </geometry>
       </collision>
       <inertial>
-        <mass value="50" />
+        <mass value="5.6" />
         <origin xyz="-0.1564 0 -0.066" rpy="-${DEG2RAD * 90} -${DEG2RAD * 0} ${DEG2RAD * 90}" />
         <inertia ixx="0.00402901710341" ixy="0.000210543968708" ixz="4.6068390983e-05" iyy="0.00668778512296" iyz="1.26910167997e-06" izz="0.00711775677213" />
