Commit message: One Value for the velocity for joint 6 was wrong for KR70 r2100

File: kuka_kr70_support/urdf/kr70_r2100_macro.xacro (robot description, xacro)
@@ -194,5 +194,5 @@
       <child link="${prefix}link_6"/>
       <axis xyz="-1 0 0"/>
-      <limit effort="0" lower="${radians(-350)}" upper="${radians(350)}" velocity="${radians(3)}"/>
+      <limit effort="0" lower="${radians(-350)}" upper="${radians(350)}" velocity="${radians(320)}"/>
     </joint>
     <!-- tool frame - fixed frame -->
