Commit message: Use predefined material

File: kuka_kr270_support/urdf/kr270r2700_macro.xacro (robot description, xacro)
@@ -2,4 +2,5 @@
 <robot xmlns:xacro="http://wiki.ros.org/xacro">
   <xacro:macro name="kuka_kr270r2700" params="prefix">
+    <xacro:include filename="$(find kuka_resources)/urdf/common_materials.xacro"/>
     <!-- links -->
     <link name="${prefix}base_link">
@@ -14,7 +15,5 @@
           <mesh filename="package://kuka_kr270_support/meshes/kr270r2700/visual/base_link.dae"/>
         </geometry>
-        <material name="">
-          <color rgba="0.75294 0.75294 0.75294 1"/>
-        </material>
+        <xacro:material_kuka_pedestal />
       </visual>
       <collision>
@@ -36,7 +35,5 @@
           <mesh filename="package://kuka_kr270_support/meshes/kr270r2700/visual/link_1.dae"/>
         </geometry>
-        <material name="">
-          <color rgba="0.75294 0.75294 0.75294 1"/>
-        </material>
+        <xacro:material_kuka_pedestal />
       </visual>
       <collision>
@@ -58,7 +55,5 @@
           <mesh filename="package://kuka_kr270_support/meshes/kr270r2700/visual/link_2.dae"/>
         </geometry>
-        <material name="">
-          <color rgba="0.75294 0.75294 0.75294 1"/>
-        </material>
+        <xacro:material_kuka_pedestal />
       </visual>
       <collision>
@@ -80,7 +75,5 @@
           <mesh filename="package://kuka_kr270_support/meshes/kr270r2700/visual/link_3.dae"/>
         </geometry>
-        <material name="">
-          <color rgba="0.75294 0.75294 0.75294 1"/>
-        </material>
+        <xacro:material_kuka_pedestal />
       </visual>
       <collision>
@@ -102,7 +95,5 @@
           <mesh filename="package://kuka_kr270_support/meshes/kr270r2700/visual/link_4.dae"/>
         </geometry>
-        <material name="">
-          <color rgba="0.75294 0.75294 0.75294 1"/>
-        </material>
+        <xacro:material_kuka_pedestal />
       </visual>
       <collision>
@@ -124,7 +115,5 @@
           <mesh filename="package://kuka_kr270_support/meshes/kr270r2700/visual/link_5.dae"/>
         </geometry>
-        <material name="">
-          <color rgba="0.75294 0.75294 0.75294 1"/>
-        </material>
+        <xacro:material_kuka_pedestal />
       </visual>
       <collision>
@@ -146,7 +135,5 @@
           <mesh filename="package://kuka_kr270_support/meshes/kr270r2700/visual/link_6.dae"/>
         </geometry>
-        <material name="">
-          <color rgba="0.75294 0.75294 0.75294 1"/>
-        </material>
+        <xacro:material_kuka_pedestal />
       </visual>
       <collision>

Commit message: Remove (wrong) inertia data

File: kuka_kr270_support/urdf/kr270r2700_macro.xacro (robot description, xacro)
@@ -5,9 +5,4 @@
     <!-- links -->
     <link name="${prefix}base_link">
-      <inertial>
-        <origin xyz="-0.027804 0.00039112 0.14035" rpy="0 0 0"/>
-        <mass value="1572.9"/>
-        <inertia ixx="89.282" ixy="-0.47721" ixz="0.85562" iyy="107.51" iyz="0.0067576" izz="172.02"/>
-      </inertial>
       <visual>
         <origin xyz="0 0 0" rpy="0 0 0"/>
@@ -25,9 +20,4 @@
     </link>
     <link name="${prefix}link_1">
-      <inertial>
-        <origin xyz="-0.036811 -0.024697 0.56577" rpy="0 0 0"/>
-        <mass value="1385.5"/>
-        <inertia ixx="90.873" ixy="33.809" ixz="17.159" iyy="147.03" iyz="0.063634" izz="168.19"/>
-      </inertial>
       <visual>
         <origin xyz="0 0 0" rpy="0 0 0"/>
@@ -45,9 +35,4 @@
     </link>
     <link name="${prefix}link_2">
-      <inertial>
-        <origin xyz="0.016923 -0.19196 0.44751" rpy="0 0 0"/>
-        <mass value="958.62"/>
-        <inertia ixx="180.42" ixy="-0.83462" ixz="0.32549" iyy="177.68" iyz="-20.82" izz="20.495"/>
-      </inertial>
       <visual>
         <origin xyz="0 0 0" rpy="0 ${radians(90)} 0"/>
@@ -65,9 +50,4 @@
     </link>
     <link name="${prefix}link_3">
-      <inertial>
-        <origin xyz="0.18842 0.18344 -0.042799" rpy="0 0 0"/>
-        <mass value="710.03"/>
-        <inertia ixx="11.887" ixy="-0.12154" ixz="-1.3604" iyy="98.805" iyz="-0.056505" izz="96.251"/>
-      </inertial>
       <visual>
         <origin xyz="0 0 0" rpy="0 0 0"/>
@@ -85,9 +65,4 @@
     </link>
     <link name="${prefix}link_4">
-      <inertial>
-        <origin xyz="0.27146 -0.007326 5.2775E-05" rpy="0 0 0"/>
-        <mass value="173.73"/>
-        <inertia ixx="1.8001" ixy="-0.18515" ixz="0.00051232" iyy="5.514" iyz="0.00070469" izz="6.3498"/>
-      </inertial>
       <visual>
         <origin xyz="0 0 0" rpy="0 0 0"/>
@@ -105,9 +80,4 @@
     </link>
     <link name="${prefix}link_5">
-      <inertial>
-        <origin xyz="0.04379 0.025984 3.5491E-07" rpy="0 0 0"/>
-        <mass value="72.17"/>
-        <inertia ixx="0.3938" ixy="-0.085332" ixz="1.7223E-06" iyy="0.68945" iyz="-7.0292E-06" izz="0.67292"/>
-      </inertial>
       <visual>
         <origin xyz="0 0 0" rpy="0 0 0"/>
@@ -125,9 +95,4 @@
     </link>
     <link name="${prefix}link_6">
-      <inertial>
-        <origin xyz="-0.017956 -1.5237E-05 0.00015484" rpy="0 0 0"/>
-        <mass value="6.3154"/>
-        <inertia ixx="0.031746" ixy="1.7673E-07" ixz="-6.6558E-06" iyy="0.016686" iyz="1.4304E-07" izz="0.016723"/>
-      </inertial>
       <visual>
         <origin xyz="0.240 0 0 " rpy="0 0 0"/>

Commit message: Turn link_2 meshes and translate link_6 meshes to zero transform

File: kuka_kr270_support/urdf/kr270r2700_macro.xacro (robot description, xacro)
@@ -36,5 +36,5 @@
     <link name="${prefix}link_2">
       <visual>
-        <origin xyz="0 0 0" rpy="0 ${radians(90)} 0"/>
+        <origin xyz="0 0 0" rpy="0 0 0"/>
         <geometry>
           <mesh filename="package://kuka_kr270_support/meshes/kr270r2700/visual/link_2.dae"/>
@@ -43,5 +43,5 @@
       </visual>
       <collision>
-        <origin xyz="0 0 0" rpy="0 ${radians(90)} 0"/>
+        <origin xyz="0 0 0" rpy="0 0 0"/>
         <geometry>
           <mesh filename="package://kuka_kr270_support/meshes/kr270r2700/collision/link_2.stl"/>
@@ -96,5 +96,5 @@
     <link name="${prefix}link_6">
       <visual>
-        <origin xyz="0.240 0 0 " rpy="0 0 0"/>
+        <origin xyz="0 0 0 " rpy="0 0 0"/>
         <geometry>
           <mesh filename="package://kuka_kr270_support/meshes/kr270r2700/visual/link_6.dae"/>
@@ -103,5 +103,5 @@
       </visual>
       <collision>
-        <origin xyz="0.240 0 0" rpy="0 0 0"/>
+        <origin xyz="0 0 0" rpy="0 0 0"/>
         <geometry>
           <mesh filename="package://kuka_kr270_support/meshes/kr270r2700/collision/link_6.stl"/>

Commit message: Move flange link definition to the corresponding joint definition

File: kuka_kr270_support/urdf/kr270r2700_macro.xacro (robot description, xacro)
@@ -109,6 +109,4 @@
       </collision>
     </link>
-    <!-- This frame corresponds to the $TOOL coordinate system in KUKA KRC controllers. -->
-    <link name="${prefix}flange"/>
     <!-- joints -->
     <joint name="${prefix}joint_a1" type="revolute">
@@ -154,4 +152,6 @@
       <limit lower="${radians(-350)}" upper="${radians(350)}" effort="0" velocity="${radians(175)}"/>
     </joint>
+    <!-- This frame corresponds to the $TOOL coordinate system in KUKA KRC controllers. -->
+    <link name="${prefix}flange"/>
     <joint name="${prefix}link_6-flange" type="fixed">
       <parent link="${prefix}link_6"/>

Commit message: Correct upper limit of third joint
Co-authored-by: Simon Schmeisser <s.schmeisser@gmx.net>

File: kuka_kr270_support/urdf/kr270r2700_macro.xacro (robot description, xacro)
@@ -129,5 +129,5 @@
       <child link="${prefix}link_3"/>
       <axis xyz="0 1 0"/>
-      <limit lower="${radians(-120)}" upper="${radians(150)}" effort="0" velocity="${radians(107)}"/>
+      <limit lower="${radians(-120)}" upper="${radians(155)}" effort="0" velocity="${radians(107)}"/>
     </joint>
     <joint name="${prefix}joint_a4" type="revolute">
