Commit message: Place links in macro using cad

File: kuka_kr300_support/urdf/kr300r2700_2_macro.xacro (robot description, xacro)
@@ -10,7 +10,64 @@
       </inertial>
       <visual>
-        <origin xyz="0 0 0" rpy="${-radians(90)} 0 0"/>
+        <origin xyz="0 0 0" rpy="0 0 0"/>
         <geometry>
           <mesh filename="package://kuka_kr300_support/meshes/kr300r2700_2/visual/base_link.dae"/>
+        </geometry>
+      </visual>
+      <collision>
+        <origin xyz="0 0 0" rpy="0 0 0"/>
+        <geometry>
+          <mesh filename="package://kuka_kr300_support/meshes/kr300r2700_2/collision/base_link.stl"/>
+        </geometry>
+      </collision>
+    </link>
+    <link name="${prefix}link_1">
+      <inertial>
+        <origin xyz="-0.036811 -0.024697 0.56577" rpy="0 0 0"/>
+        <mass value="1385.5"/>
+        <inertia ixx="90.873" ixy="33.809" ixz="17.159" iyy="147.03" iyz="0.063634" izz="168.19"/>
+      </inertial>
+      <visual>
+        <origin xyz="0 0 0" rpy="0 0 0"/>
+        <geometry>
+          <mesh filename="package://kuka_kr300_support/meshes/kr300r2700_2/visual/link_1.dae"/>
+        </geometry>
+      </visual>
+      <collision>
+        <origin xyz="0 0 0" rpy="0 0 0"/>
+        <geometry>
+          <mesh filename="package://kuka_kr300_support/meshes/kr300r2700_2/collision/link_1.stl"/>
+        </geometry>
+      </collision>
+    </link>
+    <link name="${prefix}link_2">
+      <inertial>
+        <origin xyz="0.016923 -0.19196 0.44751" rpy="0 0 0"/>
+        <mass value="958.62"/>
+        <inertia ixx="180.42" ixy="-0.83462" ixz="0.32549" iyy="177.68" iyz="-20.82" izz="20.495"/>
+      </inertial>
+      <visual>
+        <origin xyz="0 0 0" rpy="0 0 0"/>
+        <geometry>
+          <mesh filename="package://kuka_kr300_support/meshes/kr300r2700_2/visual/link_2.dae"/>
+        </geometry>
+      </visual>
+      <collision>
+        <origin xyz="0 0 0" rpy="0 0 0"/>
+        <geometry>
+          <mesh filename="package://kuka_kr300_support/meshes/kr300r2700_2/collision/link_2.stl"/>
+        </geometry>
+      </collision>
+    </link>
+    <link name="${prefix}link_3">
+      <inertial>
+        <origin xyz="0.18842 0.18344 -0.042799" rpy="0 0 0"/>
+        <mass value="710.03"/>
+        <inertia ixx="11.887" ixy="-0.12154" ixz="-1.3604" iyy="98.805" iyz="-0.056505" izz="96.251"/>
+      </inertial>
+      <visual>
+        <origin xyz="0 0 0" rpy="0 0 0"/>
+        <geometry>
+          <mesh filename="package://kuka_kr300_support/meshes/kr300r2700_2/visual/link_3.dae"/>
         </geometry>
         <material name="">
@@ -19,70 +76,4 @@
       </visual>
       <collision>
-        <origin xyz="0 0 0" rpy="${-radians(90)} 0 0"/>
-        <geometry>
-          <mesh filename="package://kuka_kr300_support/meshes/kr300r2700_2/collision/base_link.stl"/>
-        </geometry>
-      </collision>
-    </link>
-    <link name="${prefix}link_1">
-      <inertial>
-        <origin xyz="-0.036811 -0.024697 0.56577" rpy="0 0 0"/>
-        <mass value="1385.5"/>
-        <inertia ixx="90.873" ixy="33.809" ixz="17.159" iyy="147.03" iyz="0.063634" izz="168.19"/>
-      </inertial>
-      <visual>
-        <origin xyz="0 0 0" rpy="0 0 0"/>
-        <geometry>
-          <mesh filename="package://kuka_kr300_support/meshes/kr300r2700_2/visual/link_1.dae"/>
-        </geometry>
-        <material name="">
-          <color rgba="0.75294 0.75294 0.75294 1"/>
-        </material>
-      </visual>
-      <collision>
-        <origin xyz="0 0 0" rpy="0 0 0"/>
-        <geometry>
-          <mesh filename="package://kuka_kr300_support/meshes/kr300r2700_2/collision/link_1.stl"/>
-        </geometry>
-      </collision>
-    </link>
-    <link name="${prefix}link_2">
-      <inertial>
-        <origin xyz="0.016923 -0.19196 0.44751" rpy="0 0 0"/>
-        <mass value="958.62"/>
-        <inertia ixx="180.42" ixy="-0.83462" ixz="0.32549" iyy="177.68" iyz="-20.82" izz="20.495"/>
-      </inertial>
-      <visual>
-        <origin xyz="0 0 0" rpy="${-radians(90)} 0 0"/>
-        <geometry>
-          <mesh filename="package://kuka_kr300_support/meshes/kr300r2700_2/visual/link_2.dae"/>
-        </geometry>
-        <material name="">
-          <color rgba="0.75294 0.75294 0.75294 1"/>
-        </material>
-      </visual>
-      <collision>
-        <origin xyz="0 0 0" rpy="0 0 0"/>
-        <geometry>
-          <mesh filename="package://kuka_kr300_support/meshes/kr300r2700_2/collision/link_2.stl"/>
-        </geometry>
-      </collision>
-    </link>
-    <link name="${prefix}link_3">
-      <inertial>
-        <origin xyz="0.18842 0.18344 -0.042799" rpy="0 0 0"/>
-        <mass value="710.03"/>
-        <inertia ixx="11.887" ixy="-0.12154" ixz="-1.3604" iyy="98.805" iyz="-0.056505" izz="96.251"/>
-      </inertial>
-      <visual>
-        <origin xyz="0 0 0" rpy="${-radians(90)} 0 0"/>
-        <geometry>
-          <mesh filename="package://kuka_kr300_support/meshes/kr300r2700_2/visual/link_3.dae"/>
-        </geometry>
-        <material name="">
-          <color rgba="0.75294 0.75294 0.75294 1"/>
-        </material>
-      </visual>
-      <collision>
         <origin xyz="0 0 0" rpy="0 0 0"/>
         <geometry>
@@ -98,11 +89,8 @@
       </inertial>
       <visual>
-        <origin xyz="0 0 0" rpy="${-radians(90)} 0 0"/>
+        <origin xyz="0 0 0" rpy="0 0 0"/>
         <geometry>
           <mesh filename="package://kuka_kr300_support/meshes/kr300r2700_2/visual/link_4.dae"/>
         </geometry>
-        <material name="">
-          <color rgba="0.75294 0.75294 0.75294 1"/>
-        </material>
       </visual>
       <collision>
@@ -120,11 +108,8 @@
       </inertial>
       <visual>
-        <origin xyz="0 0 0" rpy="${-radians(90)} 0 0"/>
+        <origin xyz="0 0 0" rpy="0 0 0"/>
         <geometry>
           <mesh filename="package://kuka_kr300_support/meshes/kr300r2700_2/visual/link_5.dae"/>
         </geometry>
-        <material name="">
-          <color rgba="0.75294 0.75294 0.75294 1"/>
-        </material>
       </visual>
       <collision>
@@ -146,7 +131,4 @@
           <mesh filename="package://kuka_kr300_support/meshes/kr300r2700_2/visual/link_6.dae"/>
         </geometry>
-        <material name="">
-          <color rgba="0.75294 0.75294 0.75294 1"/>
-        </material>
       </visual>
       <collision>
@@ -161,26 +143,26 @@
     <!-- joints -->
     <joint name="${prefix}joint_a1" type="revolute">
-      <origin xyz="-0.00262 0.00097586 0.33099" rpy="0 0 0"/>
+      <origin xyz="0 0 0.2356" rpy="0 0 0"/>
       <parent link="${prefix}base_link"/>
       <child link="${prefix}link_1"/>
       <axis xyz="0 0 1"/>
-      <limit lower="${radians(-185)}" upper="${radians(185)}" effort="0" velocity="${radians(123)}"/>
+      <limit lower="${radians(-185)}" upper="${radians(185)}" effort="0" velocity="${radians(105)}"/>
     </joint>
     <joint name="${prefix}joint_a2" type="revolute">
-      <origin xyz="0.35277 -0.037476 0.4192" rpy="0 0 0"/>
+      <origin xyz="0.33 0.09 0.4094" rpy="0 0 0"/>
       <parent link="${prefix}link_1"/>
       <child link="${prefix}link_2"/>
       <axis xyz="0 1 0"/>
-      <limit lower="${radians(-45)}" upper="${radians(85)}" effort="0" velocity="${radians(115)}"/>
+      <limit lower="${radians(-55)}" upper="${radians(85)}" effort="0" velocity="${radians(115)}"/>
     </joint>
     <joint name="${prefix}joint_a3" type="revolute">
-      <origin xyz="-9.8483E-05 -0.1475 1.2499" rpy="0 0 0"/>
+      <origin xyz="0 -0.195 1.145" rpy="0 0 0"/>
       <parent link="${prefix}link_2"/>
       <child link="${prefix}link_3"/>
       <axis xyz="0 1 0"/>
-      <limit lower="${radians(-210)}" upper="${radians(65)}" effort="0" velocity="${radians(112)}"/>
+      <limit lower="${radians(-210)}" upper="${radians(78)}" effort="0" velocity="${radians(112)}"/>
     </joint>
     <joint name="${prefix}joint_a4" type="revolute">
-      <origin xyz="0.95795 0.184 -0.055059" rpy="0 0 0"/>
+      <origin xyz="0.8685 0.105 0.112" rpy="0 0 0"/>
       <parent link="${prefix}link_3"/>
       <child link="${prefix}link_4"/>
@@ -189,5 +171,5 @@
     </joint>
     <joint name="${prefix}joint_a5" type="revolute">
-      <origin xyz="0.542 0 0" rpy="0 0 0"/>
+      <origin xyz="0.3515 0 0" rpy="0 0 0"/>
       <parent link="${prefix}link_4"/>
       <child link="${prefix}link_5"/>
@@ -196,5 +178,5 @@
     </joint>
     <joint name="${prefix}joint_a6" type="revolute">
-      <origin xyz="0.1925 0 0" rpy="0 0 0"/>
+      <origin xyz="0.2 0 0" rpy="0 0 0"/>
       <parent link="${prefix}link_5"/>
       <child link="${prefix}link_6"/>

Commit message: Update xacro to match the datasheet exactly

File: kuka_kr300_support/urdf/kr300r2700_2_macro.xacro (robot description, xacro)
@@ -143,5 +143,5 @@
     <!-- joints -->
     <joint name="${prefix}joint_a1" type="revolute">
-      <origin xyz="0 0 0.2356" rpy="0 0 0"/>
+      <origin xyz="0 0 0.245" rpy="0 0 0"/>
       <parent link="${prefix}base_link"/>
       <child link="${prefix}link_1"/>
@@ -150,23 +150,23 @@
     </joint>
     <joint name="${prefix}joint_a2" type="revolute">
-      <origin xyz="0.33 0.09 0.4094" rpy="0 0 0"/>
+      <origin xyz="0.33 0.09 0.4" rpy="0 0 0"/>
       <parent link="${prefix}link_1"/>
       <child link="${prefix}link_2"/>
       <axis xyz="0 1 0"/>
-      <limit lower="${radians(-55)}" upper="${radians(85)}" effort="0" velocity="${radians(115)}"/>
+      <limit lower="${radians(-55)}" upper="${radians(85)}" effort="0" velocity="${radians(101)}"/>
     </joint>
     <joint name="${prefix}joint_a3" type="revolute">
-      <origin xyz="0 -0.195 1.145" rpy="0 0 0"/>
+      <origin xyz="0 -0.195 1.15" rpy="0 0 0"/>
       <parent link="${prefix}link_2"/>
       <child link="${prefix}link_3"/>
       <axis xyz="0 1 0"/>
-      <limit lower="${radians(-210)}" upper="${radians(78)}" effort="0" velocity="${radians(112)}"/>
+      <limit lower="${radians(-210)}" upper="${radians(78)}" effort="0" velocity="${radians(107)}"/>
     </joint>
     <joint name="${prefix}joint_a4" type="revolute">
-      <origin xyz="0.8685 0.105 0.112" rpy="0 0 0"/>
+      <origin xyz="0.8685 0.105 0.115" rpy="0 0 0"/>
       <parent link="${prefix}link_3"/>
       <child link="${prefix}link_4"/>
       <axis xyz="1 0 0"/>
-      <limit lower="${radians(-350)}" upper="${radians(350)}" effort="0" velocity="${radians(179)}"/>
+      <limit lower="${radians(-350)}" upper="${radians(350)}" effort="0" velocity="${radians(140)}"/>
     </joint>
     <joint name="${prefix}joint_a5" type="revolute">
@@ -175,5 +175,5 @@
       <child link="${prefix}link_5"/>
       <axis xyz="0 1 0"/>
-      <limit lower="${radians(-125)}" upper="${radians(125)}" effort="0" velocity="${radians(172)}"/>
+      <limit lower="${radians(-122.5)}" upper="${radians(122.5)}" effort="0" velocity="${radians(113)}"/>
     </joint>
     <joint name="${prefix}joint_a6" type="revolute">
@@ -182,10 +182,10 @@
       <child link="${prefix}link_6"/>
       <axis xyz="1 0 0"/>
-      <limit lower="${radians(-350)}" upper="${radians(350)}" effort="0" velocity="${radians(219)}"/>
+      <limit lower="${radians(-350)}" upper="${radians(350)}" effort="0" velocity="${radians(180)}"/>
     </joint>
     <joint name="${prefix}link_6-flange" type="fixed">
       <parent link="${prefix}link_6"/>
       <child link="${prefix}flange"/>
-      <origin xyz="0.0375 0 -0.00023924" rpy="0 0 0"/>
+      <origin xyz="0.04 0 0" rpy="0 0 0"/>
     </joint>
     <!-- ROS base_link to KUKA $ROBROOT coordinate system transform -->
