Commit message: Update xacro to match datasheet

File: kuka_kr180_support/urdf/kr180r3500_ultra_k_macro.xacro (robot description, xacro)
@@ -143,5 +143,5 @@
     <!-- joints -->
     <joint name="${prefix}joint_a1" type="revolute">
-      <origin xyz="0 0 0.245" rpy="0 0 0"/>
+      <origin xyz="0 0 0.22" rpy="0 0 0"/>
       <parent link="${prefix}base_link"/>
       <child link="${prefix}link_1"/>
@@ -150,42 +150,42 @@
     </joint>
     <joint name="${prefix}joint_a2" type="revolute">
-      <origin xyz="0.33 0.09 0.4" rpy="0 0 0"/>
+      <origin xyz="0.75 0 0.37" rpy="0 0 0"/>
       <parent link="${prefix}link_1"/>
       <child link="${prefix}link_2"/>
       <axis xyz="0 1 0"/>
-      <limit lower="${radians(-55)}" upper="${radians(85)}" effort="0" velocity="${radians(101)}"/>
+      <limit lower="${radians(-30)}" upper="${radians(160)}" effort="0" velocity="${radians(101)}"/>
     </joint>
     <joint name="${prefix}joint_a3" type="revolute">
-      <origin xyz="0 -0.195 1.15" rpy="0 0 0"/>
+      <origin xyz="0 -0.168 1.35" rpy="0 0 0"/>
       <parent link="${prefix}link_2"/>
       <child link="${prefix}link_3"/>
       <axis xyz="0 1 0"/>
-      <limit lower="${radians(-210)}" upper="${radians(78)}" effort="0" velocity="${radians(107)}"/>
+      <limit lower="${radians(-210)}" upper="${radians(65)}" effort="0" velocity="${radians(107)}"/>
     </joint>
     <joint name="${prefix}joint_a4" type="revolute">
-      <origin xyz="0.8685 0.105 0.115" rpy="0 0 0"/>
+      <origin xyz="1.16 0.168 -0.041" rpy="0 0 0"/>
       <parent link="${prefix}link_3"/>
       <child link="${prefix}link_4"/>
       <axis xyz="1 0 0"/>
-      <limit lower="${radians(-350)}" upper="${radians(350)}" effort="0" velocity="${radians(140)}"/>
+      <limit lower="${radians(-350)}" upper="${radians(350)}" effort="0" velocity="${radians(179)}"/>
     </joint>
     <joint name="${prefix}joint_a5" type="revolute">
-      <origin xyz="0.3515 0 0" rpy="0 0 0"/>
+      <origin xyz="0.240 0 0" rpy="0 0 0"/>
       <parent link="${prefix}link_4"/>
       <child link="${prefix}link_5"/>
       <axis xyz="0 1 0"/>
-      <limit lower="${radians(-122.5)}" upper="${radians(122.5)}" effort="0" velocity="${radians(113)}"/>
+      <limit lower="${radians(-125)}" upper="${radians(125)}" effort="0" velocity="${radians(172)}"/>
     </joint>
     <joint name="${prefix}joint_a6" type="revolute">
-      <origin xyz="0.2 0 0" rpy="0 0 0"/>
+      <origin xyz="0.188 0 0" rpy="0 0 0"/>
       <parent link="${prefix}link_5"/>
       <child link="${prefix}link_6"/>
       <axis xyz="1 0 0"/>
-      <limit lower="${radians(-350)}" upper="${radians(350)}" effort="0" velocity="${radians(180)}"/>
+      <limit lower="${radians(-350)}" upper="${radians(350)}" effort="0" velocity="${radians(219)}"/>
     </joint>
     <joint name="${prefix}link_6-flange" type="fixed">
       <parent link="${prefix}link_6"/>
       <child link="${prefix}flange"/>
-      <origin xyz="0.04 0 0" rpy="0 0 0"/>
+      <origin xyz="0.027 0 0" rpy="0 0 0"/>
     </joint>
     <!-- ROS base_link to KUKA $ROBROOT coordinate system transform -->
