Commit message: KR420: rename r3330f to r3330 default version, fix typos

File: kuka_kr420_support/urdf/kr420r3330_macro.xacro (robot description, xacro)
@@ -1,5 +1,5 @@
 <?xml version="1.0"?>
 <robot xmlns:xacro="http://wiki.ros.org/xacro">
-  <xacro:macro name="kuka_kr420r3330f" params="prefix">
+  <xacro:macro name="kuka_kr420r3330" params="prefix">
     <xacro:include filename="$(find kuka_resources)/urdf/common_materials.xacro"/>
     <link name="${prefix}base_link">
@@ -7,5 +7,5 @@
         <origin xyz="0 0 0" rpy="0 0 0"/>
         <geometry>
-          <mesh filename="package://kuka_kr420_support/meshes/kr420r3330f/visual/base_link.stl" />
+          <mesh filename="package://kuka_kr420_support/meshes/kr420r3330/visual/base_link.stl" />
         </geometry>
         <xacro:material_kuka_black />
@@ -14,5 +14,5 @@
         <origin xyz="0 0 0" rpy="0 0 0"/>
         <geometry>
-          <mesh filename="package://kuka_kr420_support/meshes/kr420r3330f/collision/base_link.stl" />
+          <mesh filename="package://kuka_kr420_support/meshes/kr420r3330/collision/base_link.stl" />
         </geometry>
       </collision>
@@ -22,5 +22,5 @@
         <origin xyz="0 0 0" rpy="0 0 0"/>
         <geometry>
-          <mesh filename="package://kuka_kr420_support/meshes/kr420r3330f/visual/link_1.stl" />
+          <mesh filename="package://kuka_kr420_support/meshes/kr420r3330/visual/link_1.stl" />
         </geometry>
         <xacro:material_kuka_orange />
@@ -29,5 +29,5 @@
         <origin xyz="0 0 0" rpy="0 0 0"/>
         <geometry>
-          <mesh filename="package://kuka_kr420_support/meshes/kr420r3330f/collision/link_1.stl" />
+          <mesh filename="package://kuka_kr420_support/meshes/kr420r3330/collision/link_1.stl" />
         </geometry>
       </collision>
@@ -37,5 +37,5 @@
         <origin xyz="0 0 0" rpy="0 0 0"/>
         <geometry>
-          <mesh filename="package://kuka_kr420_support/meshes/kr420r3330f/visual/link_2.stl"/>
+          <mesh filename="package://kuka_kr420_support/meshes/kr420r3330/visual/link_2.stl"/>
         </geometry>
         <xacro:material_kuka_orange />
@@ -44,5 +44,5 @@
         <origin xyz="0 0 0" rpy="0 0 0"/>
         <geometry>
-          <mesh filename="package://kuka_kr420_support/meshes/kr420r3330f/collision/link_2.stl" />
+          <mesh filename="package://kuka_kr420_support/meshes/kr420r3330/collision/link_2.stl" />
         </geometry>
       </collision>
@@ -52,5 +52,5 @@
         <origin xyz="0 0 0" rpy="0 0 0"/>
         <geometry>
-          <mesh filename="package://kuka_kr420_support/meshes/kr420r3330f/visual/link_3.stl" />
+          <mesh filename="package://kuka_kr420_support/meshes/kr420r3330/visual/link_3.stl" />
         </geometry>
         <xacro:material_kuka_orange />
@@ -59,5 +59,5 @@
         <origin xyz="0 0 0" rpy="0 0 0"/>
         <geometry>
-          <mesh filename="package://kuka_kr420_support/meshes/kr420r3330f/collision/link_3.stl" />
+          <mesh filename="package://kuka_kr420_support/meshes/kr420r3330/collision/link_3.stl" />
         </geometry>
       </collision>
@@ -67,5 +67,5 @@
         <origin xyz="0 0 0" rpy="0 0 0"/>
         <geometry>
-          <mesh filename="package://kuka_kr420_support/meshes/kr420r3330f/visual/link_4.stl" />
+          <mesh filename="package://kuka_kr420_support/meshes/kr420r3330/visual/link_4.stl" />
         </geometry>
         <xacro:material_kuka_ral_traffic_white />
@@ -74,5 +74,5 @@
         <origin xyz="0 0 0" rpy="0 0 0"/>
         <geometry>
-          <mesh filename="package://kuka_kr420_support/meshes/kr420r3330f/collision/link_4.stl" />
+          <mesh filename="package://kuka_kr420_support/meshes/kr420r3330/collision/link_4.stl" />
         </geometry>
       </collision>
@@ -82,5 +82,5 @@
         <origin xyz="0 0 0" rpy="0 0 0"/>
         <geometry>
-          <mesh filename="package://kuka_kr420_support/meshes/kr420r3330f/visual/link_5.stl" />
+          <mesh filename="package://kuka_kr420_support/meshes/kr420r3330/visual/link_5.stl" />
         </geometry>
         <xacro:material_kuka_ral_traffic_white />
@@ -89,5 +89,5 @@
         <origin xyz="0 0 0" rpy="0 0 0"/>
         <geometry>
-          <mesh filename="package://kuka_kr420_support/meshes/kr420r3330f/collision/link_5.stl" />
+          <mesh filename="package://kuka_kr420_support/meshes/kr420r3330/collision/link_5.stl" />
         </geometry>
       </collision>
@@ -97,5 +97,5 @@
         <origin xyz="0 0 0" rpy="0 0 0"/>
         <geometry>
-          <mesh filename="package://kuka_kr420_support/meshes/kr420r3330f/visual/link_6.stl" />
+          <mesh filename="package://kuka_kr420_support/meshes/kr420r3330/visual/link_6.stl" />
         </geometry>
         <xacro:material_kuka_black />
@@ -104,5 +104,5 @@
         <origin xyz="0 0 0" rpy="0 0 0"/>
         <geometry>
-          <mesh filename="package://kuka_kr420_support/meshes/kr420r3330f/collision/link_6.stl" />
+          <mesh filename="package://kuka_kr420_support/meshes/kr420r3330/collision/link_6.stl" />
         </geometry>
       </collision>

Commit message: KR420: fix package.xml description, add ROS-I flange

File: kuka_kr420_support/urdf/kr420r3330_macro.xacro (robot description, xacro)
@@ -108,6 +108,4 @@
       </collision>
     </link>
-    <!-- This frame corresponds to the $FLANGE coordinate system in KUKA KRC controllers. -->
-    <link name="${prefix}tool0"/>
     <joint name="${prefix}joint_a1" type="revolute">
       <origin xyz="0 0 1.045" rpy="0 0 0"/>
@@ -152,10 +150,5 @@
       <limit effort="0" lower="${radians(-350)}" upper="${radians(350)}" velocity="${radians(110)}"/>
     </joint>
-    <joint name="${prefix}joint_a6-tool0" type="fixed">
-      <parent link="${prefix}link_6"/>
-      <child link="${prefix}tool0"/>
-      <origin xyz="0 0 0" rpy="0 ${radians(90)} 0"/>
-    </joint>
-    <!-- ROS base_link to KUKA $ROBROOT coordinate system transform -->
+    <!-- ROS-Industrial 'base' frame: base_link to KUKA $ROBROOT coordinate system transform -->
     <link name="${prefix}base" />
     <joint name="${prefix}base_link-base" type="fixed">
@@ -164,4 +157,19 @@
       <child link="${prefix}base"/>
     </joint>
+    <!-- ROS-Industrial 'flange' frame: attachment point for EEF models -->
+    <link name="${prefix}flange" />
+    <joint name="${prefix}joint_6-flange" type="fixed">
+      <origin xyz="0 0 0" rpy="0 0 0" />
+      <parent link="${prefix}link_6" />
+      <child link="${prefix}flange" />
+    </joint>
+    <!-- ROS-Industrial 'tool0' frame: all-zeros tool frame -->
+    <!-- This frame corresponds to the $FLANGE coordinate system in KUKA KRC controllers. -->
+    <link name="${prefix}tool0"/>
+    <joint name="${prefix}joint_a6-tool0" type="fixed">
+      <parent link="${prefix}link_6"/>
+      <child link="${prefix}tool0"/>
+      <origin xyz="0 0 0" rpy="0 ${radians(90)} 0"/>
+    </joint>
   </xacro:macro>
 </robot>
