Commit message: update KR20 R1810-2

File: kuka_kr20_support/urdf/kr20_r1810_2.xacro (robot description, xacro)
@@ -1,6 +1,5 @@
 <?xml version="1.0"?>
-<!--Generates a urdf from the macro in kr16_2_macro.xacro -->
 <robot name="kuka_kr20_r1810_2" xmlns:xacro="http://wiki.ros.org/xacro">
-  <xacro:include filename="$(find kuka_kr20_support)/urdf/kuka_kr20_r1810_2.xacro" />
+  <xacro:include filename="$(find kuka_kr20_support)/urdf/kr20_r1810_2_macro.xacro" />
   <xacro:kuka_kr20_r1810_2 prefix=""/>
 </robot>

File: kuka_kr20_support/urdf/kr20_r1810_2_macro.xacro (robot description, xacro)
@@ -1,40 +1,26 @@
 <?xml version="1.0"?>
 <robot xmlns:xacro="http://wiki.ros.org/xacro">
-  <xacro:include filename="$(find kuka_resources)/urdf/common_constants.xacro"/>
-  <xacro:include filename="$(find kuka_resources)/urdf/common_materials.xacro"/>
   <xacro:macro name="kuka_kr20_r1810_2" params="prefix">
-    <!-- LINKS -->
-    <!-- base link -->
+    <xacro:include filename="$(find kuka_resources)/urdf/common_materials.xacro"/>
     <link name="${prefix}base_link">
-      <inertial>
-        <origin xyz="0 0 0" rpy="0 0 0"/>
-        <mass value="2"/>
-        <inertia ixx="0.01" ixy="0" ixz="0" iyy="0.01" iyz="0" izz="0.01" />
-      </inertial>
       <visual>
         <origin xyz="0 0 0" rpy="0 0 0"/>
         <geometry>
-          <mesh filename="package://kuka_kr20_support/meshes/kuka_kr20_r1810_2/visual/base_link.stl" scale="0.001 0.001 0.001" />
+          <mesh filename="package://kuka_kr20_support/meshes/kr20_r1810_2/visual/base_link.stl" scale="0.001 0.001 0.001" />
         </geometry>
-        <xacro:material_kuka_pedestal />
+        <xacro:material_kuka_black />
       </visual>
       <collision>
         <origin xyz="0 0 0" rpy="0 0 0"/>
         <geometry>
-          <mesh filename="package://kuka_kr20_support/meshes/kuka_kr20_r1810_2/collision/base_link.stl" scale="0.001 0.001 0.001"/>
+          <mesh filename="package://kuka_kr20_support/meshes/kr20_r1810_2/collision/base_link.stl" scale="0.001 0.001 0.001" />
         </geometry>
       </collision>
     </link>
-    <!-- link 1 (A1) -->
     <link name="${prefix}link_1">
-      <inertial>
-        <origin xyz="0 0 0" rpy="0 0 0"/>
-        <mass value="2"/>
-        <inertia ixx="0.01" ixy="0" ixz="0" iyy="0.01" iyz="0" izz="0.01" />
-      </inertial>
       <visual>
         <origin xyz="0 0 0" rpy="0 0 0"/>
         <geometry>
-          <mesh filename="package://kuka_kr20_support/meshes/kuka_kr20_r1810_2/visual/link_1.stl" scale="0.001 0.001 0.001" />
+          <mesh filename="package://kuka_kr20_support/meshes/kr20_r1810_2/visual/link_1.stl" scale="0.001 0.001 0.001" />
         </geometry>
         <xacro:material_kuka_orange />
@@ -43,19 +29,13 @@
         <origin xyz="0 0 0" rpy="0 0 0"/>
         <geometry>
-          <mesh filename="package://kuka_kr20_support/meshes/kuka_kr20_r1810_2/collision/link_1.stl" scale="0.001 0.001 0.001"/>
+          <mesh filename="package://kuka_kr20_support/meshes/kr20_r1810_2/collision/link_1.stl" scale="0.001 0.001 0.001" />
         </geometry>
       </collision>
     </link>
-    <!-- link 2 -->
     <link name="${prefix}link_2">
-      <inertial>
-        <origin xyz="0 0 0" rpy="0 0 0"/>
-        <mass value="2"/>
-        <inertia ixx="0.01" ixy="0" ixz="0" iyy="0.01" iyz="0" izz="0.01" />
-      </inertial>
       <visual>
         <origin xyz="0 0 0" rpy="0 0 0"/>
         <geometry>
-          <mesh filename="package://kuka_kr20_support/meshes/kuka_kr20_r1810_2/visual/link_2.stl" scale="0.001 0.001 0.001"/>
+          <mesh filename="package://kuka_kr20_support/meshes/kr20_r1810_2/visual/link_2.stl" scale="0.001 0.001 0.001" />
         </geometry>
         <xacro:material_kuka_orange />
@@ -64,19 +44,13 @@
         <origin xyz="0 0 0" rpy="0 0 0"/>
         <geometry>
-          <mesh filename="package://kuka_kr20_support/meshes/kuka_kr20_r1810_2/collision/link_2.stl" scale="0.001 0.001 0.001"/>
+          <mesh filename="package://kuka_kr20_support/meshes/kr20_r1810_2/collision/link_2.stl" scale="0.001 0.001 0.001" />
         </geometry>
       </collision>
     </link>
-    <!-- link 3 -->
     <link name="${prefix}link_3">
-      <inertial>
-        <origin xyz="0 0 0" rpy="0 0 0"/>
-        <mass value="2"/>
-        <inertia ixx="0.01" ixy="0" ixz="0" iyy="0.01" iyz="0" izz="0.01" />
-      </inertial>
       <visual>
         <origin xyz="0 0 0" rpy="0 0 0"/>
         <geometry>
-          <mesh filename="package://kuka_kr20_support/meshes/kuka_kr20_r1810_2/visual/link_3.stl" scale="0.001 0.001 0.001"/>
+          <mesh filename="package://kuka_kr20_support/meshes/kr20_r1810_2/visual/link_3.stl" scale="0.001 0.001 0.001" />
         </geometry>
         <xacro:material_kuka_orange />
@@ -85,19 +59,13 @@
         <origin xyz="0 0 0" rpy="0 0 0"/>
         <geometry>
-          <mesh filename="package://kuka_kr20_support/meshes/kuka_kr20_r1810_2/collision/link_3.stl" scale="0.001 0.001 0.001"/>
+          <mesh filename="package://kuka_kr20_support/meshes/kr20_r1810_2/collision/link_3.stl" scale="0.001 0.001 0.001" />
         </geometry>
       </collision>
     </link>
-    <!-- link 4 -->
     <link name="${prefix}link_4">
-      <inertial>
-        <origin xyz="0 0 0" rpy="0 0 0"/>
-        <mass value="2"/>
-        <inertia ixx="0.01" ixy="0" ixz="0" iyy="0.01" iyz="0" izz="0.01" />
-      </inertial>
       <visual>
         <origin xyz="0 0 0" rpy="0 0 0"/>
         <geometry>
-          <mesh filename="package://kuka_kr20_support/meshes/kuka_kr20_r1810_2/visual/link_4.stl" scale="0.001 0.001 0.001"/>
+          <mesh filename="package://kuka_kr20_support/meshes/kr20_r1810_2/visual/link_4.stl" scale="0.001 0.001 0.001" />
         </geometry>
         <xacro:material_kuka_orange />
@@ -106,19 +74,13 @@
         <origin xyz="0 0 0" rpy="0 0 0"/>
         <geometry>
-          <mesh filename="package://kuka_kr20_support/meshes/kuka_kr20_r1810_2/collision/link_4.stl" scale="0.001 0.001 0.001"/>
+          <mesh filename="package://kuka_kr20_support/meshes/kr20_r1810_2/collision/link_4.stl" scale="0.001 0.001 0.001" />
         </geometry>
       </collision>
     </link>
-    <!-- link 5 -->
     <link name="${prefix}link_5">
-      <inertial>
-        <origin xyz="0 0 0" rpy="0 0 0"/>
-        <mass value="2"/>
-        <inertia ixx="0.01" ixy="0" ixz="0" iyy="0.01" iyz="0" izz="0.01" />
-      </inertial>
       <visual>
         <origin xyz="0 0 0" rpy="0 0 0"/>
         <geometry>
-          <mesh filename="package://kuka_kr20_support/meshes/kuka_kr20_r1810_2/visual/link_5.stl" scale="0.001 0.001 0.001"/>
+          <mesh filename="package://kuka_kr20_support/meshes/kr20_r1810_2/visual/link_5.stl" scale="0.001 0.001 0.001" />
         </geometry>
         <xacro:material_kuka_orange />
@@ -127,35 +89,23 @@
         <origin xyz="0 0 0" rpy="0 0 0"/>
         <geometry>
-          <mesh filename="package://kuka_kr20_support/meshes/kuka_kr20_r1810_2/collision/link_5.stl" scale="0.001 0.001 0.001"/>
+          <mesh filename="package://kuka_kr20_support/meshes/kr20_r1810_2/collision/link_5.stl" scale="0.001 0.001 0.001" />
         </geometry>
       </collision>
     </link>
-    <!-- link 6 -->
     <link name="${prefix}link_6">
-      <inertial>
-        <origin xyz="0 0 0" rpy="0 0 0"/>
-        <mass value="2"/>
-        <inertia ixx="0.01" ixy="0" ixz="0" iyy="0.01" iyz="0" izz="0.01" />
-      </inertial>
       <visual>
         <origin xyz="0 0 0" rpy="0 0 0"/>
         <geometry>
-          <mesh filename="package://kuka_kr20_support/meshes/kuka_kr20_r1810_2/visual/link_6.stl" scale="0.001 0.001 0.001"/>
+          <mesh filename="package://kuka_kr20_support/meshes/kr20_r1810_2/visual/link_6.stl" scale="0.001 0.001 0.001" />
         </geometry>
-        <xacro:material_kuka_pedestal />
+        <xacro:material_kuka_black />
       </visual>
       <collision>
         <origin xyz="0 0 0" rpy="0 0 0"/>
         <geometry>
-          <mesh filename="package://kuka_kr20_support/meshes/kuka_kr20_r1810_2/collision/link_6.stl" scale="0.001 0.001 0.001"/>
+          <mesh filename="package://kuka_kr20_support/meshes/kr20_r1810_2/collision/link_6.stl" scale="0.001 0.001 0.001" />
         </geometry>
       </collision>
     </link>
-    <!-- tool 0 -->
-    <!-- This frame corresponds to the $FLANGE coordinate system in KUKA KRC controllers. -->
-    <link name="${prefix}tool0"/>
-    <!-- END LINKS -->
-    <!-- JOINTS -->
-    <!-- joint 1 (A1) -->
     <joint name="${prefix}joint_a1" type="revolute">
       <origin xyz="0 0 0.520" rpy="0 0 0"/>
@@ -165,5 +115,4 @@
       <limit effort="0" lower="${radians(-185)}" upper="${radians(185)}" velocity="${radians(200)}"/>
     </joint>
-    <!-- joint 2 (A2) -->
     <joint name="${prefix}joint_a2" type="revolute">
       <origin xyz="0.160 0 0" rpy="0 0 0"/>
@@ -173,5 +122,4 @@
       <limit effort="0" lower="${radians(-185)}" upper="${radians(65)}" velocity="${radians(175)}"/>
     </joint>
-    <!-- joint 3 (A3) -->
     <joint name="${prefix}joint_a3" type="revolute">
       <origin xyz="0.780 0 0.0" rpy="0 0 0"/>
@@ -181,5 +129,4 @@
       <limit effort="0" lower="${radians(-138)}" upper="${radians(175)}" velocity="${radians(190)}"/>
     </joint>
-    <!-- joint 4 (A4) -->
     <joint name="${prefix}joint_a4" type="revolute">
       <origin xyz="0.0 0 0.150" rpy="0 0 0"/>
@@ -189,5 +136,4 @@
       <limit effort="0" lower="${radians(-350)}" upper="${radians(350)}" velocity="${radians(430)}"/>
     </joint>
-    <!-- joint 5 (A5) -->
     <joint name="${prefix}joint_a5" type="revolute">
       <origin xyz="0.860 0 0" rpy="0 0 0"/>
@@ -197,5 +143,4 @@
       <limit effort="0" lower="${radians(-130)}" upper="${radians(130)}" velocity="${radians(430)}"/>
     </joint>
-    <!-- joint 6 (A6) -->
     <joint name="${prefix}joint_a6" type="revolute">
       <origin xyz="0.153 0 0" rpy="0 0 0"/>
@@ -205,12 +150,5 @@
       <limit effort="0" lower="${radians(-350)}" upper="${radians(350)}" velocity="${radians(630)}"/>
     </joint>
-    <!-- tool frame - fixed frame -->
-    <joint name="${prefix}joint_a6-tool0" type="fixed">
-      <parent link="${prefix}link_6"/>
-      <child link="${prefix}tool0"/>
-      <origin xyz="0.0 0 0" rpy="0 ${radians(90)} 0"/>
-    </joint>
-    <!-- END JOINTS -->
-    <!-- ROS base_link to KUKA $ROBROOT coordinate system transform -->
+    <!-- ROS-Industrial 'base' frame: base_link to KUKA $ROBROOT coordinate system transform -->
     <link name="${prefix}base" />
     <joint name="${prefix}base_link-base" type="fixed">
@@ -219,4 +157,19 @@
       <child link="${prefix}base"/>
     </joint>
+    <!-- ROS-Industrial 'flange' frame: attachment point for EEF models -->
+    <link name="${prefix}flange" />
+    <joint name="${prefix}joint_6-flange" type="fixed">
+      <origin xyz="0 0 0" rpy="0 0 0" />
+      <parent link="${prefix}link_6" />
+      <child link="${prefix}flange" />
+    </joint>
+    <!-- ROS-Industrial 'tool0' frame: all-zeros tool frame -->
+    <!-- This frame corresponds to the $FLANGE coordinate system in KUKA KRC controllers. -->
+    <link name="${prefix}tool0"/>
+    <joint name="${prefix}joint_a6-tool0" type="fixed">
+      <parent link="${prefix}link_6"/>
+      <child link="${prefix}tool0"/>
+      <origin xyz="0 0 0" rpy="0 ${radians(90)} 0"/>
+    </joint>
   </xacro:macro>
 </robot>
